File: Spaceport/23-24/PCBs/Master Board/master-board/master-board.kicad_pcb (KiCad board)
At the start: 2 copper layers, 103.3 x 67.9 mm, 10 parts, among them J1 Screw_Terminal_01x02, J2 Conn_01x04_Pin, J3 Conn_01x03_Pin, J4 Conn_01x04_Pin, J5 Conn_01x04_Pin, J6 Conn_01x04_Pin

Commit message: generated gerbers
Parts:
- moved G*** 1.40 mm to (117.6, 125.0)
Other:
- board size 103.3 x 67.9 mm -> 98.7 x 67.9 mm
Changed lines of the file:
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@@
       (outputformat 1)
       (mirror false)
-      (drillshape 1)
+      (drillshape 0)
       (scaleselection 1)
-      (outputdirectory "")
+      (outputdirectory "gerbers/")
     )
   )
@@
   )
   (footprint "LOGO" (layer "F.Cu")
-    (at 116.2 125)
+    (at 117.6 125)
     (attr board_only exclude_from_pos_files exclude_from_bom)
     (fp_text reference "G***" (at 0 0) (layer "F.SilkS") hide
@@
         (effects (font (size 1 1) (thickness 0.15)))
     )
-    (fp_text value "Screw_Terminal_01x02" (at 1.6 6.805) (layer "F.Fab")
+    (fp_text value "Screw_Terminal_01x02" (at 1.6 6.805) (layer "F.Fab") hide
         (effects (font (size 1 1) (thickness 0.15)))
     )
@@
   (gr_arc (start 159.6 111.28) (mid 159.746447 110.926447) (end 160.1 110.78)
     (stroke (width 0.05) (type default)) (layer "F.SilkS"))
-  (gr_rect (start 86.8 59.95) (end 190.05 127.85)
+  (gr_rect (start 88.6 59.95) (end 187.25 127.85)
     (stroke (width 0.1) (type default)) (fill none) (layer "Edge.Cuts"))
   (gr_text "SCL\n" (at 118.8 108.6) (layer "F.SilkS")
@@
     (effects (font (size 1 1) (thickness 0.15)) (justify left bottom))
   )
-  (gr_text "TerpRockets Avionics" (at 88 126.6) (layer "F.SilkS")
+  (gr_text "TerpRockets Avionics" (at 89.4 126.6) (layer "F.SilkS")
     (effects (font (size 1.5 1.5) (thickness 0.3) bold) (justify left bottom))
   )
@@
         (xy 108.5 60.5)
         (xy 108.5 126)
-        (xy 187.6 126)
-        (xy 187.5 60.5)
+        (xy 186.6 126.4)
+        (xy 186.5 60.9)
       )
     )

Commit message: Updated master board
Parts:
- added H1: MountingHole, MountingHole:MountingHole_2.7mm_M2.5, F.Cu at (183.0, 127.8)
- added H2: MountingHole, MountingHole:MountingHole_2.7mm_M2.5, F.Cu at (183.0, 59.0)
- added H3: MountingHole, MountingHole:MountingHole_2.7mm_M2.5, F.Cu at (92.8, 127.8)
- added H4: MountingHole, MountingHole:MountingHole_2.7mm_M2.5, F.Cu at (92.8, 59.0)
- moved G*** 11.8 mm to (129.0, 128.0)
- moved J1 2.55 mm to (180.4, 117.6)
- moved J4 0.96 mm to (152.1, 80.4)
Routing:
- net Net-(J1-Pin_1): track 70.5 -> 69.6 mm
- net /3.3V: track 147.5 -> 146.7 mm
Other:
- board size 98.7 x 67.9 mm -> 98.5 x 76.2 mm
