File: Side_Projects/Live Video/PCBs/LVPD-board_v2/LVPD-board_v2.kicad_pcb (KiCad board)
At the start: 2 copper layers, 54.4 x 88.5 mm, 13 parts, among them J1 CNVT, J2 CTRL, J3 RPi, J4 Radio, J5 Radio

Commit message: PCB gerbers and LVPD fix
Routing:
- net GND: track 162.8 -> 163.6 mm
- net /VSIG: track 50.7 -> 51.4 mm
Changed lines of the file:
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@@
       (outputformat 1)
       (mirror false)
-      (drillshape 1)
+      (drillshape 0)
       (scaleselection 1)
-      (outputdirectory "")
+      (outputdirectory "../gerbers/LVPD_v2.0/")
     )
   )
@@
     (fp_line (start 7.45 3.4) (end 7.45 -2.35)
       (stroke (width 0.1) (type solid)) (layer "F.Fab"))
-    (pad "1" thru_hole roundrect (at 0 0 270) (size 1.7 1.95) (drill 0.95) (layers "*.Cu" "*.Mask") (roundrect_rratio 0.147059)
+    (pad "1" thru_hole roundrect (at 0 0 270) (size 1.7 1.95) (drill 0.95) (layers "*.Cu" "*.Mask") (roundrect_rratio 0.1470588235)
       (net 6 "/VSIG") (pinfunction "Pin_1") (pintype "passive"))
     (pad "2" thru_hole oval (at 2.5 0 270) (size 1.7 1.95) (drill 0.95) (layers "*.Cu" "*.Mask")
@@
     (fp_line (start 1 0.625) (end 1 -0.625)
       (stroke (width 0.1) (type solid)) (layer "B.Fab"))
-    (pad "1" smd roundrect (at -0.9125 0 90) (size 1.025 1.4) (layers "B.Cu" "B.Paste" "B.Mask") (roundrect_rratio 0.243902)
+    (pad "1" smd roundrect (at -0.9125 0 90) (size 1.025 1.4) (layers "B.Cu" "B.Paste" "B.Mask") (roundrect_rratio 0.243902439)
       (net 2 "GND") (pintype "passive"))
-    (pad "2" smd roundrect (at 0.9125 0 90) (size 1.025 1.4) (layers "B.Cu" "B.Paste" "B.Mask") (roundrect_rratio 0.243902)
+    (pad "2" smd roundrect (at 0.9125 0 90) (size 1.025 1.4) (layers "B.Cu" "B.Paste" "B.Mask") (roundrect_rratio 0.243902439)
       (net 4 "/EN") (pintype "passive"))
     (model "${KICAD6_3DMODEL_DIR}/Resistor_SMD.3dshapes/R_0805_2012Metric.wrl"
@@
   (segment (start 118.95 53.57) (end 118.89 53.57) (width 0.25) (layer "B.Cu") (net 1))
   (segment (start 150.46 65.46) (end 152 65.46) (width 1.5) (layer "B.Cu") (net 1))
-  (segment (start 103.5 84.6) (end 103.5 121) (width 1.5) (layer "F.Cu") (net 2))
   (segment (start 106.9 89.05) (end 111.34 93.49) (width 1.5) (layer "F.Cu") (net 2))
   (segment (start 151.655 62.575) (end 144.881268 62.575) (width 1.5) (layer "F.Cu") (net 2))
+  (segment (start 102.6 120.1) (end 105 122.5) (width 1.5) (layer "F.Cu") (net 2))
+  (segment (start 105 122.5) (end 106.025 122.5) (width 1.5) (layer "F.Cu") (net 2))
   (segment (start 103.5 63.5) (end 103.5 84.6) (width 1.5) (layer "F.Cu") (net 2))
   (segment (start 152 62.92) (end 151.655 62.575) (width 1.5) (layer "F.Cu") (net 2))
@@
   (segment (start 103.5 85.65) (end 106.9 89.05) (width 1.5) (layer "F.Cu") (net 2))
   (segment (start 144.881268 62.575) (end 143.456268 64) (width 1.5) (layer "F.Cu") (net 2))
+  (segment (start 103.5 84.6) (end 102.6 85.5) (width 1.5) (layer "F.Cu") (net 2))
   (segment (start 134.705787 63.98) (end 132.165787 61.44) (width 1.5) (layer "F.Cu") (net 2))
+  (segment (start 102.6 85.5) (end 102.6 120.1) (width 1.5) (layer "F.Cu") (net 2))
   (segment (start 136.14 64) (end 136.12 63.98) (width 1.5) (layer "F.Cu") (net 2))
   (segment (start 143.456268 64) (end 136.14 64) (width 1.5) (layer "F.Cu") (net 2))
@@
   (segment (start 136.12 63.98) (end 134.705787 63.98) (width 1.5) (layer "F.Cu") (net 2))
   (segment (start 106 61.74) (end 105.26 61.74) (width 1.5) (layer "F.Cu") (net 2))
-  (segment (start 103.5 121) (end 105 122.5) (width 1.5) (layer "F.Cu") (net 2))
-  (segment (start 105 122.5) (end 106.025 122.5) (width 1.5) (layer "F.Cu") (net 2))
   (segment (start 132.165787 61.44) (end 120.88 61.44) (width 1.5) (layer "F.Cu") (net 2))
   (segment (start 103.5 84.6) (end 103.5 85.65) (width 1.5) (layer "F.Cu") (net 2))
@@
   (segment (start 152 60.38) (end 140.5 60.38) (width 1.5) (layer "F.Cu") (net 5))
   (segment (start 106.025 117.5) (end 106 117.475) (width 0.25) (layer "F.Cu") (net 6))
-  (segment (start 106 66.82) (end 106 117.475) (width 0.25) (layer "B.Cu") (net 6))
-  (segment (start 106 117.475) (end 106.025 117.5) (width 0.25) (layer "B.Cu") (net 6))
+  (segment (start 105.2 67.62) (end 105.2 116.675) (width 0.25) (layer "B.Cu") (net 6))
+  (segment (start 105.2 116.675) (end 106.025 117.5) (width 0.25) (layer "B.Cu") (net 6))
+  (segment (start 106 66.82) (end 105.2 67.62) (width 0.25) (layer "B.Cu") (net 6))
   (segment (start 138 120.5) (end 138 91.26) (width 0.25) (layer "F.Cu") (net 7))
   (segment (start 138 91.26) (end 136.12 89.38) (width 0.25) (layer "F.Cu") (net 7))
