File: Spaceport/24-25/PCBs/Main Board/STLink.kicad_sch (KiCad schematic)
At the start: 43 parts, among them J1 USB_C_Receptacle_USB2.0_16P, J2 STLINK_SWD, Q1 Q_NPN_BCE, U1 USB6B1, U2 STM32F103CBTx, Y1 8Mhz

Commit message: Pasrt of main MCU designed
Connections:
- net RCC_IN is gone; now on net GND: C10.1, U2.5 (PD0), Y1.1
- net GND: no longer CR1.2 (GND)
- net USB_D+: no longer R10.2
- net USB_D-: now also R10.2
- net at R12.1: now also D2.1 (K); no longer D1.2 (A)
- net at R13.1: now also D1.2 (A); no longer D2.1 (K)
Other:
- moved on the sheet: C10, C11, C12, C13, C14, C15, C16, C2, C4, C6, C7, C9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
