File: Spaceport/23-24/PCBs/Unified Board/Unified_Board/Unified_Board.kicad_sch (KiCad schematic)
At the start: 54 parts, among them J1 Screw_Terminal_01x02, J2 Serial2 Breakout, J3 I2C Breakout, J4 Serial1 Breakout, U1 BNO055, U2 MAX-M10S, U3 DS3231M, Y1 32.768kHz

Commit message: Fixed unified board
Parts:
- removed BT2: 6.8mm_coin_cell_RTC, Battery:BatteryHolder_Keystone_2998_1x6.8mm, symbol Device:Battery_Cell
- removed C10, C8: 100nF, Capacitor_SMD:C_0805_2012Metric, symbol Device:C
- removed D2: RTC_LED, LED_SMD:LED_0805_2012Metric_Pad1.15x1.40mm_HandSolder, symbol Device:LED
- removed R10: 10kΩ, Resistor_SMD:R_0805_2012Metric, symbol Device:R
- removed R14: R, Resistor_SMD:R_0805_2012Metric, symbol Device:R
- removed U3: DS3231M, Package_SO:SOIC-16W_7.5x10.3mm_P1.27mm, symbol Timer_RTC:DS3231M
- added C4: 0.1uF, Capacitor_SMD:C_0805_2012Metric, symbol Device:C
- added J1: Screw_Terminal_01x02, TerminalBlock_4Ucon:TerminalBlock_4Ucon_1x02_P3.50mm_Vertical, symbol Connector:Screw_Terminal_01x02
- added J5: Conn_01x05_Pin, Connector_PinHeader_2.54mm:PinHeader_1x05_P2.54mm_Vertical, symbol Connector:Conn_01x05_Pin
- added J6: Conn_01x09_Pin, Connector_PinHeader_2.54mm:PinHeader_1x09_P2.54mm_Vertical, symbol Connector:Conn_01x09_Pin
Connections:
- net 3.3V: now also U2.7 (VCC_IO), U2.8 (VCC), C4.2, J6.1 (Pin_1)
- net GND: now also C7.1, U2.1 (GND), U2.10 (GND), U2.12 (GND), C4.1, J6.2 (Pin_2), J6.9 (Pin_9)
- net at C3.2, D6.1 (K), Teensy4.1.46 (GND): now also J1.2 (Pin_2); no longer J1.2 (Pin_2)
- net at Teensy4.1.24 (PWM): now also BZ1.1 (-)
- net Radio_CS: now reaches Teensy4.1.11 (CS)
- net Radio_CS: now also J6.8 (Pin_8)
- net Radio_MOSI: now reaches Teensy4.1.12 (MOSI)
- net Radio_MOSI: now also J6.7 (Pin_7)
- net Radio_MISO: now reaches Teensy4.1.13 (MISO)
- net Radio_MISO: now also J6.6 (Pin_6)
- net Radio_SCK: now reaches Teensy4.1.34 (SCK)
- net Radio_SCK: now also J6.5 (Pin_5)
- new net: J1.1 (Pin_1), J1.2 (Pin_2)
- no-connect marks 47 -> 40
Other:
- note added: "RFM69HCW"
- note removed: "DS3231"
- moved on the sheet: C7

Commit message: Updated unified board
Connections:
- net GND: no longer J6.9 (Pin_9)
- net Radio_INT: now reaches Teensy4.1.22 (GPIO)
- net Radio_INT: now also J6.4 (Pin_4)
- net Radio_RST: now reaches Teensy4.1.23 (GPIO)
- net Radio_RST: now also J6.9 (Pin_9)
- no-connect marks 40 -> 44
Changed lines of the file:
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@@
   (no_connect (at 34.29 76.2))
   (no_connect (at 57.15 88.9))
-  (no_connect (at 34.29 88.9))
   (no_connect (at 57.15 63.5))
   (no_connect (at 34.29 81.28))
+  (no_connect (at 227.33 115.57))
   (no_connect (at 34.29 58.42))
+  (no_connect (at 227.33 120.65))
   (no_connect (at 57.15 78.74))
+  (no_connect (at 227.33 113.03))
   (no_connect (at 34.29 71.12))
   (no_connect (at 34.29 40.64))
@@
   (no_connect (at 57.15 68.58))
   (no_connect (at 34.29 48.26))
+  (no_connect (at 190.5 115.57))
   (no_connect (at 193.04 66.04))
-  (no_connect (at 34.29 91.44))
   (no_connect (at 34.29 43.18))
   (no_connect (at 57.15 55.88))
   (no_connect (at 34.29 45.72))
+  (no_connect (at 227.33 110.49))
   (no_connect (at 57.15 73.66))
   (no_connect (at 57.15 45.72))
@@
   (no_connect (at 223.52 60.96))
   (no_connect (at 193.04 58.42))
+  (no_connect (at 227.33 118.11))
   (no_connect (at 34.29 50.8))
   (no_connect (at 34.29 83.82))
@@
     (stroke (width 0) (type default))
   )
+  (wire (pts (xy 31.75 88.9) (xy 34.29 88.9))
+    (stroke (width 0) (type default))
+  )
   (wire (pts (xy 76.2 30.48) (xy 76.2 35.56))
     (stroke (width 0) (type default))
@@
     (stroke (width 0) (type default))
   )
+  (wire (pts (xy 31.75 91.44) (xy 34.29 91.44))
+    (stroke (width 0) (type default))
+  )
   (wire (pts (xy 195.58 105.41) (xy 199.39 105.41))
     (stroke (width 0) (type default))
@@
     (stroke (width 0) (type default))
   )
+  (wire (pts (xy 190.5 118.11) (xy 198.12 118.11))
+    (stroke (width 0) (type default))
+  )
   (wire (pts (xy 130.81 52.07) (xy 130.81 63.5))
     (stroke (width 0) (type default))
@@
     (stroke (width 0) (type default))
   )
-  (wire (pts (xy 190.5 130.81) (xy 194.31 130.81))
-    (stroke (width 0) (type default))
-  )
   (wire (pts (xy 111.76 46.99) (xy 111.76 52.07))
     (stroke (width 0) (type default))
@@
   )
   (wire (pts (xy 153.67 99.06) (xy 151.13 99.06))
+    (stroke (width 0) (type default))
+  )
+  (wire (pts (xy 190.5 130.81) (xy 198.12 130.81))
     (stroke (width 0) (type default))
   )
@@
     (effects (font (size 1.27 1.27)) (justify right bottom))
   )
+  (label "Radio_INT" (at 31.75 88.9 180) (fields_autoplaced)
+    (effects (font (size 1.27 1.27)) (justify right bottom))
+  )
   (label "Radio_SCK" (at 69.85 66.04 0) (fields_autoplaced)
     (effects (font (size 1.27 1.27)) (justify left bottom))
@@
     (effects (font (size 1.27 1.27)) (justify left bottom))
   )
+  (label "Radio_RST" (at 31.75 91.44 180) (fields_autoplaced)
+    (effects (font (size 1.27 1.27)) (justify right bottom))
+  )
   (label "3.3V" (at 110.49 76.2 0) (fields_autoplaced)
+    (effects (font (size 1.27 1.27)) (justify left bottom))
+  )
+  (label "Radio_INT" (at 198.12 118.11 0) (fields_autoplaced)
     (effects (font (size 1.27 1.27)) (justify left bottom))
   )
@@
   )
   (label "3.3V" (at 257.81 116.84 0) (fields_autoplaced)
+    (effects (font (size 1.27 1.27)) (justify left bottom))
+  )
+  (label "Radio_RST" (at 198.12 130.81 0) (fields_autoplaced)
     (effects (font (size 1.27 1.27)) (justify left bottom))
   )
@@
         )
       )
-    )
-  )
-  (symbol (lib_id "power:GND") (at 194.31 130.81 90) (unit 1)
-    (in_bom yes) (on_board yes) (dnp no) (fields_autoplaced)
-    (property "Reference" "#PWR01" (at 200.66 130.81 0)
-      (effects (font (size 1.27 1.27)) hide)
-    )
-    (property "Value" "GND" (at 198.12 130.81 90)
-      (effects (font (size 1.27 1.27)) (justify right))
-    )
-    (property "Footprint" "" (at 194.31 130.81 0)
-      (effects (font (size 1.27 1.27)) hide)
-    )
-    (property "Datasheet" "" (at 194.31 130.81 0)
-      (effects (font (size 1.27 1.27)) hide)
-    )
-    (pin "1")
-    (instances
-      (project "master-board"
-        (path "/0377917c-9f6d-421e-bc69-b49bbfc3a6cf"
-          (reference "#PWR01") (unit 1)
-        )
-      )
-      (project "Unified_Board"
-        (path "/711155f6-b770-4d7a-a1c1-c9256b05a2ff"
-          (reference "#PWR024") (unit 1)
-        )
-      )

Commit message: Fixed unified board capacitors and LED wiring
Connections:
- net 3.3V: now also Alt2.5 (SDO)
- net BMP_I2C_ADDR: no longer names the net of Teensy4.1.27 (PWM)
- net BMP_I2C_ADDR: no longer Alt2.5 (SDO)
- no-connect marks 44 -> 45
Changed lines of the file:
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@@
   (junction (at 227.33 53.34) (diameter 0) (color 0 0 0 0)
+  )
+  (junction (at 130.81 63.5) (diameter 0) (color 0 0 0 0)
   )
   (junction (at 123.19 124.46) (diameter 0) (color 0 0 0 0)
@@
   (no_connect (at 190.5 115.57))
   (no_connect (at 193.04 66.04))
+  (no_connect (at 57.15 83.82))
   (no_connect (at 34.29 43.18))
   (no_connect (at 57.15 55.88))
@@
     (stroke (width 0) (type default))
   )
+  (wire (pts (xy 120.65 63.5) (xy 130.81 63.5))
+    (stroke (width 0) (type default))
+  )
   (wire (pts (xy 138.43 87.63) (xy 138.43 91.44))
     (stroke (width 0) (type default))
@@
     (stroke (width 0) (type default))
   )
-  (wire (pts (xy 120.65 57.15) (xy 120.65 49.53))
+  (wire (pts (xy 120.65 49.53) (xy 120.65 63.5))
     (stroke (width 0) (type default))
   )
@@
     (stroke (width 0) (type default))
   )
-  (wire (pts (xy 57.15 83.82) (xy 59.69 83.82))
-    (stroke (width 0) (type default))
-  )
   (wire (pts (xy 254 121.92) (xy 257.81 121.92))
     (stroke (width 0) (type default))
@@
     (stroke (width 0) (type default))
   )
-  (wire (pts (xy 104.14 57.15) (xy 120.65 57.15))
-    (stroke (width 0) (type default))
-  )
   (wire (pts (xy 132.08 33.02) (xy 135.89 33.02))
     (stroke (width 0) (type default))
@@
     (effects (font (size 1.27 1.27)) (justify left bottom))
   )
-  (label "BMP_I2C_ADDR" (at 59.69 83.82 0) (fields_autoplaced)
-    (effects (font (size 1.27 1.27)) (justify left bottom))
-  )
   (label "BACKUP" (at 274.32 63.5 0) (fields_autoplaced)
     (effects (font (size 1.27 1.27)) (justify left bottom))
@@
     (effects (font (size 1.27 1.27)) (justify left bottom))
   )
-  (label "BMP_I2C_ADDR" (at 104.14 57.15 0) (fields_autoplaced)
-    (effects (font (size 1.27 1.27)) (justify left bottom))
-  )
