File: Spaceport/24-25/PCBs/RF4463F30-test-board/RF4463F30-test-board.kicad_sch (KiCad schematic)
At the start: 4 parts

Commit message: added some secondary components
Parts:
- added BZ1: Buzzer, Avionics:Adafruit_5V_Buzzer, symbol Device:Buzzer
- added D1, D2, D3, D4: LED, LED_SMD:LED_0805_2012Metric, symbol Device:LED
- added H1, H2, H3: MountingHole, MountingHole:MountingHole_2.2mm_M2, symbol Mechanical:MountingHole
- added R1, R2, R3, R4: 10k, Resistor_SMD:R_0805_2012Metric, symbol Device:R
Connections:
- net 5V: now also D4.1 (K)
- net CS: now also D1.1 (K)
- net GND: now also BZ1.2 (-), R1.2, R2.2, R3.2, R4.2
- net IRQ: now also D2.1 (K)
- net SDN: now also D3.1 (K)
- net at Teensy4.1.32 (GPIO): now also BZ1.1 (+)
- new net: D3.2 (A), R3.1
- new net: D4.2 (A), R4.1
- new net: D1.2 (A), R1.1
- new net: D2.2 (A), R2.1
- no-connect marks 42 -> 41
Other:
- moved on the sheet: JPower1

Commit message: add CAD and update board with better dimensions
Parts:
- added H4: MountingHole, MountingHole:MountingHole_2.2mm_M2, symbol Mechanical:MountingHole
Connections:
- net CS: now also Teensy4.1.8 (TX2); no longer Teensy4.1.10 (CS)
- net GPIO0: now also Teensy4.1.9 (PWM); no longer Teensy4.1.6 (PWM)
- net GPIO1: now also Teensy4.1.10 (CS); no longer Teensy4.1.7 (RX2)
- net IRQ: now also Teensy4.1.7 (RX2); no longer Teensy4.1.9 (PWM)
- net SDN: now also Teensy4.1.6 (PWM); no longer Teensy4.1.8 (TX2)
- net at Teensy4.1.0 (RX1): now also BZ1.1 (+)
- net at Teensy4.1.32 (GPIO): no longer BZ1.1 (+)
Other:
- moved on the sheet: BZ1, H1, H2, H3
Changed lines of the file:
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@@
 	)
 	(no_connect
-		(at 59.69 54.61)
+		(at 59.69 110.49)
 	)
 	(no_connect
@@
 	(wire
 		(pts
+			(xy 53.34 57.15) (xy 55.88 57.15)
+		)
+		(stroke
+			(width 0)
+			(type default)
+		)
+	)
+	(wire
+		(pts
 			(xy 59.69 52.07) (xy 53.34 52.07)
 		)
@@
 	(wire
 		(pts
+			(xy 55.88 57.15) (xy 55.88 54.61)
+		)
+		(stroke
+			(width 0)
+			(type default)
+		)
+	)
+	(wire
+		(pts
 			(xy 128.27 111.76) (xy 133.35 111.76)
 		)
@@
 	(wire
 		(pts
+			(xy 55.88 54.61) (xy 59.69 54.61)
+		)
+		(stroke
+			(width 0)
+			(type default)
+		)
+	)
+	(wire
+		(pts
 			(xy 163.83 127) (xy 171.45 127)
 		)
@@
 	(wire
 		(pts
-			(xy 54.61 110.49) (xy 54.61 105.41)
-		)
-		(stroke
-			(width 0)
-			(type default)
-		)
-	)
-	(wire
-		(pts
 			(xy 59.69 69.85) (xy 52.07 69.85)
 		)
@@
 			(width 0)
 			(type default)
-		)
-	)
-	(label "GND"
-		(at 54.61 105.41 270)
-		(fields_autoplaced yes)
-		(effects
-			(font
-				(size 1.27 1.27)
-			)
-			(justify right bottom)
 		)
 	)
@@
 	)
 	(label "SDN"
-		(at 52.07 74.93 0)
+		(at 52.07 69.85 0)
 		(fields_autoplaced yes)
 		(effects
@@
 	)
 	(label "GPIO0"
-		(at 52.07 69.85 0)
+		(at 52.07 77.47 0)
 		(fields_autoplaced yes)
 		(effects
@@
 	)
 	(label "GPIO1"
-		(at 52.07 72.39 0)
+		(at 52.07 80.01 0)
 		(fields_autoplaced yes)
 		(effects
@@
 	)
 	(label "CS"
-		(at 52.07 80.01 0)
+		(at 52.07 74.93 0)
 		(fields_autoplaced yes)
 		(effects
@@
 	)
 	(label "IRQ"
-		(at 52.07 77.47 0)
+		(at 52.07 72.39 0)
 		(fields_autoplaced yes)
 		(effects
@@
 	(symbol
 		(lib_id "Mechanical:MountingHole")
+		(at 160.02 106.68 0)
+		(unit 1)
+		(exclude_from_sim yes)
+		(in_bom no)
+		(on_board yes)
+		(dnp no)
+		(fields_autoplaced yes)
+		(property "Reference" "H3"
+			(at 162.56 105.4099 0)
+			(effects
+				(font
+					(size 1.27 1.27)
+				)
+				(justify left)
+			)
+		)
+		(property "Value" "MountingHole"
+			(at 162.56 107.9499 0)
+			(effects
+				(font
+					(size 1.27 1.27)
+				)
+				(justify left)
+			)
+		)
+		(property "Footprint" "MountingHole:MountingHole_2.2mm_M2"
+			(at 160.02 106.68 0)
+			(effects
+				(font
+					(size 1.27 1.27)
+				)
+				(hide yes)
+			)
+		)
+		(property "Datasheet" "~"
+			(at 160.02 106.68 0)
+			(effects
+				(font
+					(size 1.27 1.27)
+				)
+				(hide yes)
+			)
+		)
+		(property "Description" "Mounting Hole without connection"
+			(at 160.02 106.68 0)
+			(effects
+				(font
+					(size 1.27 1.27)
+				)
+				(hide yes)
+			)
+		)
+		(instances
+			(project "RF4463F30-test-board"
+				(path "/10b1ca65-3bbd-4272-bddd-c70184b19a75"
+					(reference "H3")
+					(unit 1)
+				)
+			)
+		)
+	)
+	(symbol
+		(lib_id "Mechanical:MountingHole")
 		(at 160.02 111.76 0)
 		(unit 1)
@@
 		(dnp no)
 		(fields_autoplaced yes)
-		(property "Reference" "H3"
+		(property "Reference" "H4"
 			(at 162.56 110.4899 0)
 			(effects
@@
 			(project "RF4463F30-test-board"
 				(path "/10b1ca65-3bbd-4272-bddd-c70184b19a75"
-					(reference "H3")
+					(reference "H4")
 					(unit 1)
 				)
@@
 		(on_board yes)
 		(dnp no)
-		(fields_autoplaced yes)
 		(property "Reference" "JPower1"
 			(at 159.385 119.38 0)
@@
 	(symbol
 		(lib_id "Mechanical:MountingHole")
-		(at 160.02 105.41 0)
+		(at 160.02 101.6 0)
 		(unit 1)
 		(exclude_from_sim yes)
@@
 		(fields_autoplaced yes)
 		(property "Reference" "H2"
-			(at 162.56 104.1399 0)
+			(at 162.56 100.3299 0)
 			(effects
 				(font
@@
 		)
 		(property "Value" "MountingHole"
-			(at 162.56 106.6799 0)
+			(at 162.56 102.8699 0)
 			(effects
 				(font
@@
 		)
 		(property "Footprint" "MountingHole:MountingHole_2.2mm_M2"
-			(at 160.02 105.41 0)
+			(at 160.02 101.6 0)
 			(effects
 				(font
@@
 		)
 		(property "Datasheet" "~"
-			(at 160.02 105.41 0)
+			(at 160.02 101.6 0)
 			(effects
 				(font
@@
 		)
 		(property "Description" "Mounting Hole without connection"
-			(at 160.02 105.41 0)
+			(at 160.02 101.6 0)
 			(effects
 				(font
@@
 	(symbol
 		(lib_id "Mechanical:MountingHole")
-		(at 160.02 99.06 0)
+		(at 160.02 96.52 0)
 		(unit 1)
 		(exclude_from_sim yes)
@@
 		(fields_autoplaced yes)
 		(property "Reference" "H1"
+			(at 162.56 95.2499 0)
+			(effects
+				(font
+					(size 1.27 1.27)
+				)
+				(justify left)
+			)
+		)
+		(property "Value" "MountingHole"
 			(at 162.56 97.7899 0)
 			(effects
@@
 			)
 		)
-		(property "Value" "MountingHole"
-			(at 162.56 100.3299 0)
-			(effects
-				(font
-					(size 1.27 1.27)
-				)
-				(justify left)
-			)
-		)
 		(property "Footprint" "MountingHole:MountingHole_2.2mm_M2"
-			(at 160.02 99.06 0)
+			(at 160.02 96.52 0)
 			(effects
 				(font
@@
 		)
 		(property "Datasheet" "~"
-			(at 160.02 99.06 0)
+			(at 160.02 96.52 0)
 			(effects
 				(font
@@
 		)
 		(property "Description" "Mounting Hole without connection"
-			(at 160.02 99.06 0)
+			(at 160.02 96.52 0)
 			(effects
 				(font
@@
 	(symbol
 		(lib_id "Device:Buzzer")
-		(at 57.15 113.03 270)
+		(at 50.8 54.61 180)
 		(unit 1)
 		(exclude_from_sim no)
@@
 		(dnp no)
 		(property "Reference" "BZ1"
-			(at 60.706 115.316 90)
+			(at 48.514 58.166 90)
 			(effects
 				(font
@@
 		)
 		(property "Value" "Buzzer"
-			(at 60.706 117.856 90)
+			(at 45.974 58.166 90)
 			(effects
 				(font
@@
 		)
 		(property "Footprint" "Avionics:Adafruit_5V_Buzzer"
-			(at 59.69 112.395 90)
+			(at 51.435 57.15 90)
 			(effects
 				(font
@@
 		)
 		(property "Datasheet" "~"
-			(at 59.69 112.395 90)
+			(at 51.435 57.15 90)
 			(effects
 				(font
@@
 		)
 		(property "Description" "Buzzer, polarized"
-			(at 57.15 113.03 0)
-			(effects
-				(font
+			(at 50.8 54.61 0)
+			(effects
+				(font
