File: Spaceport/PCBs/Sensor Boards/SensorBoardPatch/SensorBoardNoMCU.kicad_pcb (KiCad board)
At the start: 2 copper layers, 52 x 44 mm, 28 parts, among them J1 I2C, U1 BMI088, U2 LIS3MDL, U3 MAX-M10S, U4 MS5611-01BA, U5 DPS310

Commit message: Update SensorBoardNoMCU.kicad_pcb
Routing:
- net GND: track 91.5 -> 97.8 mm, vias 16 -> 17
Changed lines of the file:
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@@
 		(sheetname "Root")
 		(sheetfile "SensorBoardNoMCU.kicad_sch")
+		(clearance 0.127)
 		(attr smd)
 		(fp_line
@@
 		)
 		(property "Value" "10n"
-			(at 0 1.68 360)
+			(at 0 1.68 0)
 			(layer "F.Fab")
 			(effects
@@
 		)
 		(fp_text user "${REFERENCE}"
-			(at 0 0 360)
+			(at 0 0 0)
 			(layer "F.Fab")
 			(effects
@@
 		(tags "capacitor")
 		(property "Reference" "C6"
-			(at 2.8 0 360)
+			(at 2.8 0 0)
 			(layer "F.SilkS")
 			(effects
@@
 		)
 		(property "Value" "100n"
-			(at 0 1.68 360)
+			(at 0 1.68 0)
 			(layer "F.Fab")
 			(effects
@@
 		)
 		(fp_text user "${REFERENCE}"
-			(at 0 0 360)
+			(at 0 0 0)
 			(layer "F.Fab")
 			(effects
@@
 		(tags "capacitor")
 		(property "Reference" "C4"
-			(at -0.7 1.75 360)
+			(at -0.7 1.75 0)
 			(layer "F.SilkS")
 			(effects
@@
 		)
 		(property "Value" "100n"
-			(at 0 1.68 360)
+			(at 0 1.68 0)
 			(layer "F.Fab")
 			(effects
@@
 		)
 		(fp_text user "${REFERENCE}"
-			(at 0 0 360)
+			(at 0 0 0)
 			(layer "F.Fab")
 			(effects
@@
 		(tags "capacitor")
 		(property "Reference" "C5"
-			(at 2.8 -0.125 360)
+			(at 2.8 -0.125 0)
 			(layer "F.SilkS")
 			(effects
@@
 		)
 		(property "Value" "100n"
-			(at 0 1.68 360)
+			(at 0 1.68 0)
 			(layer "F.Fab")
 			(effects
@@
 		)
 		(fp_text user "${REFERENCE}"
-			(at 0 0 360)
+			(at 0 0 0)
 			(layer "F.Fab")
 			(effects
@@
 		)
 		(property "Value" "1u"
-			(at 0 1.68 360)
+			(at 0 1.68 0)
 			(layer "F.Fab")
 			(effects
@@
 		)
 		(fp_text user "${REFERENCE}"
-			(at 0 0 360)
+			(at 0 0 0)
 			(layer "F.Fab")
 			(effects
@@
 		(tags "lga land grid array")
 		(property "Reference" "U2"
-			(at 0.1125 -2.375 180)
+			(at 0.1125 -2.375 360)
 			(layer "F.SilkS")
 			(effects
@@
 		(sheetname "Root")
 		(sheetfile "SensorBoardNoMCU.kicad_sch")
+		(clearance 0.127)
 		(attr smd)
 		(fp_line
@@
 	)
 	(segment
+		(start 111.225 67.725)
+		(end 111.25 67.75)
+		(width 0.2)
+		(layer "F.Cu")
+		(net 1)
+	)
+	(segment
+		(start 111.225 66)
+		(end 111.225 67.725)
+		(width 0.2)
+		(layer "F.Cu")
+		(net 1)
+	)
+	(segment
 		(start 117 71)
 		(end 116.5 71)
@@
 	)
 	(segment
+		(start 111.225 61.5)
+		(end 111.225 66)
+		(width 0.2)
+		(layer "F.Cu")
+		(net 1)
+	)
+	(segment
 		(start 115.55 86.175)
 		(end 114.75 86.175)
@@
 		(drill 0.3)
 		(layers "F.Cu" "B.Cu")
+		(net 1)
+	)
+	(via
+		(at 111.25 67.75)
+		(size 0.6)
+		(drill 0.3)
+		(layers "F.Cu" "B.Cu")
