File: Spaceport/PCBs/MCU Boards/Teensy MCU Board/mcu-board.kicad_pcb (KiCad board)
At the start: 2 copper layers, 48.3 x 84.5 mm, 21 parts, among them J1 Conn_01x04, J10 Conn_01x06, J2 Conn_01x04, J3 Conn_01x04, J4 Conn_01x04, J5 Conn_01x04, J6 Conn_01x04, J7 Conn_01x04, J8 Conn_01x06, J9 Conn_01x02

Commit message: Updated Teensy MCU Board to v1.1
Parts:
- added BZ1: Buzzer, Avionics:Adafruit_Buzzer, F.Cu at (182.5, 108.6)
- added D2: LED, LED_SMD:LED_0805_2012Metric_Pad1.15x1.40mm_HandSolder, F.Cu at (172.8, 111.0)
- added R6: 220Ω, Resistor_SMD:R_0805_2012Metric_Pad1.20x1.40mm_HandSolder, F.Cu at (172.8, 106.2)
- moved J7 28.5 mm to (154.8, 112.0)
- moved J6 1.28 mm to (154.9, 105.4)
Connections:
- Teensy4.2 pad 23: unconnected-(Teensy4.2-GPIO-Pad23) -> Net-(R6-Pad2)
- Teensy4.2 pad 24: unconnected-(Teensy4.2-PWM-Pad24) -> Net-(BZ1-+)
Routing:
- net GND: track 239.1 -> 293.2 mm
- net +3.3V: track 263.2 -> 211.6 mm
- net /RX8: track 15.7 -> 39.8 mm
- net /TX8: track 13.5 -> 36.2 mm
- net Net-(R6-Pad2): track 0.00 -> 16.7 mm, vias 0 -> 1
- net /SCK1: track 48.2 -> 60.5 mm
- net Net-(BZ1-+): track 0.00 -> 10.7 mm
- net /MOSI1: track 52.2 -> 62.7 mm
- net Net-(D2-A): track 0.00 -> 4.76 mm
- net /TX7: track 17.1 -> 15.8 mm
- net /RX7: track 25.2 -> 23.9 mm
Other:
- board size 48.3 x 84.5 mm -> 48.3 x 84.1 mm

Commit message: Trying to use KiCAD to update power controller
Parts:
- added J11: Screw_Terminal_01x02, Connector_JST:JST_EH_B2B-EH-A_1x02_P2.50mm_Vertical, B.Cu at (177.0, 45.0)
Connections:
- J9 pad 1: Net-(J9-Pin_1) -> Net-(J11-Pin_2)
- Teensy4.2 pad 47: Net-(J9-Pin_1) -> Net-(J11-Pin_1)
Routing:
- net Net-(J9-Pin_1): track 10.8 -> 0.00 mm
- net (no net): track 0.00 -> 10.8 mm
- net Net-(J11-Pin_2): track 0.00 -> 9.87 mm
- net Net-(J11-Pin_1): track 0.00 -> 5.16 mm

Commit message: Rearranged switch block & larger power traces
Parts:
- J11: footprint Connector_JST:JST_EH_B2B-EH-A_1x02_P2.50mm_Vertical -> TerminalBlock:TerminalBlock_Xinya_XY308-2.54-2P_1x02_P2.54mm_Horizontal; moved to F.Cu
- moved J11 10.8 mm to (173.0, 35.0), turned to 0 degrees
- moved D1 5.70 mm to (165.8, 34.5)
- moved R5 5.70 mm to (163.2, 34.5)
- moved J9 3.95 mm to (184.2, 34.3)
Routing:
- net (no net): track 10.8 -> 0.00 mm
- net GND: track 293.2 -> 303.7 mm
- net +3.3V: track 211.6 -> 216.7 mm
- net Net-(J11-Pin_1): track 5.16 -> 7.35 mm
- net Net-(J11-Pin_2): track 9.87 -> 10.5 mm
Other:
- board size 48.3 x 84.1 mm -> 48 x 84.1 mm
- board text added: "+"
- board text added: "-"
- board text removed: "POWER"
