File: Spaceport/PCBs/MCU Boards/Teensy MCU Board/mcu-board.kicad_sch (KiCad schematic)
At the start: 21 parts, among them J1 I2C0, J2 I2C2, J3 Switch, J4 5v, J6 UART1, J7 UART2, J8 UART2

Commit message: Revert "Merge branch 'main' of https://github.com/Terrapin-Rocket-Team/SRAD-Avionics"
This reverts commit e5f68e4e525f2a5ad7eebbc917cc2807b67ca5e1, reversing
changes made to 8a40e2e341d8980ca528983581171a8bd9cc0146.
Parts:
- BZ1: footprint Buzzer_Beeper:Buzzer_Murata_PKMCS0909E -> Buzzer_Beeper:Buzzer_12x9.5RM7.6
- J3: value Switch -> 5v
- J4: value 5v -> Switch
- Teensy4.1: value (none) -> ~
Connections:
- net GND: now also J4.1 (Pin_1); no longer J4.2 (Pin_2)
- net RX1: now also J6.2 (Pin_2); no longer J6.3 (Pin_3)
- net RX2: now also J7.2 (Pin_2); no longer J7.3 (Pin_3)
- net RX8: now also J8.2 (Pin_2); no longer J8.3 (Pin_3)
- net TX1: now also J6.3 (Pin_3); no longer J6.2 (Pin_2)
- net TX2: now also J7.3 (Pin_3); no longer J7.2 (Pin_2)
- net TX8: now also J8.3 (Pin_3); no longer J8.2 (Pin_2)
- net at J3.2 (Pin_2): now also J4.2 (Pin_2); no longer J4.1 (Pin_1)

Commit message: MCU Board Changes
Parts:
- J3: value 5v -> Switch
- J4: value Switch -> 5v
Connections:
- net GND: now also J4.2 (Pin_2); no longer J4.1 (Pin_1)
- net RX1: now also J6.3 (Pin_3); no longer J6.2 (Pin_2)
- net RX2: now also J7.3 (Pin_3); no longer J7.2 (Pin_2)
- net RX8: now also J8.3 (Pin_3); no longer J8.2 (Pin_2)
- net TX1: now also J6.2 (Pin_2); no longer J6.3 (Pin_3)
- net TX2: now also J7.2 (Pin_2); no longer J7.3 (Pin_3)
- net TX8: now also J8.2 (Pin_2); no longer J8.3 (Pin_3)
- net at J3.2 (Pin_2): now also J4.1 (Pin_1); no longer J4.2 (Pin_2)
Changed lines of the file:
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@@
 (kicad_sch
-	(version 20231120)
+	(version 20250114)
 	(generator "eeschema")
-	(generator_version "8.0")
+	(generator_version "9.0")
 	(paper "A4")
-	(junction
-		(at 175.26 64.77)
-		(diameter 0)
-		(color 0 0 0 0)
+	(text "I²C\nConnectors"
+		(exclude_from_sim no)
+		(at 69.85 38.862 0)
+		(effects
+			(font
+				(size 2.27 2.27)
+			)
+		)
+	)
+	(text "UART\nConnectors"
+		(exclude_from_sim no)
+		(at 69.85 90.932 0)
+		(effects
+			(font
+				(size 2.27 2.27)
+			)
+		)
 	)
 	(junction
@@
 		(color 0 0 0 0)
 	)
+	(junction
+		(at 180.34 67.31)
+		(diameter 0)
+		(color 0 0 0 0)
+	)
 	(no_connect
 		(at 138.43 92.71)
@@
 	(wire
 		(pts
-			(xy 177.8 60.96) (xy 177.8 67.31)
-		)
-		(stroke
-			(width 0)
-			(type default)
-		)
-	)
-	(wire
-		(pts
 			(xy 130.81 64.77) (xy 138.43 64.77)
 		)
@@
 	(wire
 		(pts
+			(xy 179.07 60.96) (xy 179.07 64.77)
+		)
+		(stroke
+			(width 0)
+			(type default)
+		)
+	)
+	(wire
+		(pts
 			(xy 161.29 118.11) (xy 168.91 118.11)
 		)
@@
 	(wire
 		(pts
-			(xy 177.8 67.31) (xy 180.34 67.31)
-		)
-		(stroke
-			(width 0)
-			(type default)
-		)
-	)
-	(wire
-		(pts
 			(xy 138.43 97.79) (xy 125.73 97.79)
 		)
@@
 	(wire
 		(pts
-			(xy 180.34 64.77) (xy 175.26 64.77)
+			(xy 39.37 55.88) (xy 44.45 55.88)
 		)
 		(stroke
@@
 	(wire
 		(pts
-			(xy 39.37 55.88) (xy 44.45 55.88)
+			(xy 50.8 110.49) (xy 55.88 110.49)
 		)
 		(stroke
@@
 	(wire
 		(pts
-			(xy 50.8 110.49) (xy 55.88 110.49)
+			(xy 175.26 62.23) (xy 175.26 58.42)
 		)
 		(stroke
@@
 	(wire
 		(pts
-			(xy 175.26 62.23) (xy 175.26 58.42)
+			(xy 180.34 64.77) (xy 179.07 64.77)
 		)
 		(stroke
@@
 	(wire
 		(pts
-			(xy 177.8 60.96) (xy 180.34 60.96)
+			(xy 179.07 60.96) (xy 180.34 60.96)
 		)
 		(stroke
@@
 	(wire
 		(pts
+			(xy 180.34 67.31) (xy 175.26 67.31)
+		)
+		(stroke
+			(width 0)
+			(type default)
+		)
+	)
+	(wire
+		(pts
 			(xy 85.09 134.62) (xy 90.17 134.62)
 		)
@@
 		)
 	)
-	(text "I²C\nConnectors"
-		(exclude_from_sim no)
-		(at 69.85 38.862 0)
-		(effects
-			(font
-				(size 2.27 2.27)
-			)
+	(wire
+		(pts
+			(xy 175.26 67.31) (xy 175.26 64.77)
 		)
-	)
-	(text "UART\nConnectors"
-		(exclude_from_sim no)
-		(at 69.85 90.932 0)
-		(effects
-			(font
-				(size 2.27 2.27)
-			)
+		(stroke
+			(width 0)
+			(type default)
 		)
 	)
@@
 	)
 	(label "RX8"
-		(at 90.17 129.54 180)
+		(at 90.17 132.08 180)
 		(effects
 			(font
@@
 	)
 	(label "TX2"
-		(at 90.17 113.03 180)
+		(at 90.17 110.49 180)
 		(effects
 			(font
@@
 	)
 	(label "RX2"
-		(at 90.17 110.49 180)
+		(at 90.17 113.03 180)
 		(effects
 			(font
@@
 	)
 	(label "TX8"
-		(at 90.17 132.08 180)
+		(at 90.17 129.54 180)
 		(effects
 			(font
@@
 	)
 	(label "RX1"
-		(at 55.88 110.49 180)
+		(at 55.88 113.03 180)
 		(effects
 			(font
@@
 	)
 	(label "TX1"
-		(at 55.88 113.03 180)
+		(at 55.88 110.49 180)
 		(effects
 			(font
@@
 			)
 		)
-		(property "Value" "Switch"
+		(property "Value" "5v"
 			(at 187.96 67.3099 0)
 			(effects
@@
 			)
 		)
-		(property "Value" "5v"
+		(property "Value" "Switch"
 			(at 187.96 60.9599 0)
 			(effects
@@
 		)
 		(property "Value" "+3.3V"
-			(at 175.26 69.85 0)
+			(at 170.942 73.66 0)
 			(effects
 				(font
@@
 	(symbol
 		(lib_id "power:GND")
-		(at 175.26 64.77 0)
+		(at 180.34 67.31 0)
 		(unit 1)
 		(exclude_from_sim no)
@@
 		(fields_autoplaced yes)
 		(property "Reference" "#PWR06"
-			(at 175.26 71.12 0)
+			(at 180.34 73.66 0)
 			(effects
 				(font
@@
 		)
 		(property "Value" "GND"
-			(at 175.26 69.85 0)
+			(at 180.34 72.39 0)
 			(effects
 				(font
@@
 		)
 		(property "Footprint" ""
-			(at 175.26 64.77 0)
+			(at 180.34 67.31 0)
 			(effects
 				(font
@@
 		)
 		(property "Datasheet" ""
-			(at 175.26 64.77 0)
+			(at 180.34 67.31 0)
 			(effects
 				(font
@@
 		)
 		(property "Description" "Power symbol creates a global label with name \"GND\" , ground"
-			(at 175.26 64.77 0)
+			(at 180.34 67.31 0)
 			(effects
 				(font
@@
 		)
 	)
+	(embedded_fonts no)
 )

Commit message: some very minor changes
Parts:
- BZ1: footprint Buzzer_Beeper:Buzzer_12x9.5RM7.6 -> Buzzer_Beeper:Buzzer_Murata_PKMCS0909E
- Teensy4.1: value ~ -> (none)
