File: Spaceport/PCBs/power-delivery-board/power-delivery-board/PCB.kicad_pcb (KiCad board)
At the start: 2 copper layers, 40 parts, among them J1 Conn_01x07_Pin, U1 ADP5033ACBZ-5-R7, U2 TPS610986DSER, U3 TPS610986DSER

Commit message: Housekeeping File Updates
- Removed extra PCB file that somehow got onto the repo
- Updated PCB file with footprints
Parts:
- moved C7 54.3 mm to (144.8, 106.8)
- moved COUT4 50.6 mm to (159.5, 100.8)
- moved J1 48.9 mm to (166.8, 87.2), turned to 180 degrees
- moved COUT2 48.5 mm to (158.9, 92.2)
- moved C2 47.9 mm to (133.2, 106.0)
- moved C6 44.4 mm to (133.8, 114.1)
- moved COUT1 44.0 mm to (154.8, 100.0), turned to 180 degrees
- moved CBAT1 43.9 mm to (144.2, 98.0)
- moved C5 43.6 mm to (137.7, 108.0)
- moved C3 42.9 mm to (139.8, 99.8)
- moved U2 41.5 mm to (155.0, 95.5)
- moved L4 40.7 mm to (150.4, 65.0)
- moved L3 39.6 mm to (154.0, 89.0)
- moved U3 38.0 mm to (151.2, 71.0)
- moved CIN2 37.9 mm to (156.8, 65.0)
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