File: Spaceport/PCBs/power-delivery-board/power-delivery-board/power-delivery-board.kicad_sch (KiCad schematic)
At the start: 26 parts, among them J1 Conn_01x03_Pin, U1 ADP5033ACBZ-5-R7, U2 TPS610986DSER, U3 TPS610986DSER

Commit message: Updated JST Pin
Parts:
- removed J1: Conn_01x03_Pin, symbol Connector:Conn_01x03_Pin
- added J2: Conn_01x07_Pin, symbol Connector:Conn_01x07_Pin
Connections:
- net VOUT1: now also J2.1 (Pin_1)
- net VOUT2: now also J2.2 (Pin_2)
- net VOUT3: now also J2.3 (Pin_3)
- net VOUT4: now also J2.4 (Pin_4)
- net VOUT5: now also J2.5 (Pin_5)
- net VOUT6: now also J2.6 (Pin_6)
- net VOUT7: now also J2.7 (Pin_7)
Other:
- note added: "SOURCE TWO"
- note added: "VOUT6 3.3V 350mA"
- note added: "VOUT7 3.3V 200mA"
- moved on the sheet: BAT1, CBAT, CBAT1, CIN, CIN1, COUT1, COUT2, COUT3, COUT4, L, L3, RIN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

Commit message: Added LEDS and Labeled VIN
Parts:
- added D1, D2, D3, D4, D5, D6: LED, symbol Device:LED
- added J1: Conn_01x06_Pin, symbol Connector:Conn_01x06_Pin
- added R1, R2, R3, R4, R5, R6: 10kΩ, symbol Device:R
Connections:
- net GND: now also R1.1, R2.1, R3.1, R4.1, R5.1, R6.1
- net VIN1: now also D6.1 (K), J1.1 (Pin_1)
- net VIN2: now also D5.1 (K), J1.2 (Pin_2)
- net VIN3: now also D4.1 (K), J1.3 (Pin_3)
- net VIN4: now also D3.1 (K), J1.4 (Pin_4); no longer CBAT.1, L.1
- net VIN5: now also CBAT.1, L.1, D2.1 (K), J1.5 (Pin_5); no longer CBAT1.1, L3.1
- new net: D1.2 (A), R1.2
- new net: D2.2 (A), R2.2
- new net: D3.2 (A), R3.2
- new net: D6.2 (A), R6.2
- new net: D5.2 (A), R5.2
- new net: D4.2 (A), R4.2
- new net VIN6: CBAT1.1, D1.1 (K), J1.6 (Pin_6), L3.1
Other:
- note added: "0.7V TO 4.5V"
- note added: "1.7V TO 5.5V"
- note added: "2.3V TO 5.5V"
- moved on the sheet: BAT1, C1, C2, C3, C4, C5, C7, CBAT, CBAT1, CIN, CIN1, COUT1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

Commit message: PCB Changes
Parts:
- removed J1: Conn_01x06_Pin, symbol Connector:Conn_01x06_Pin
- added BAT1, BAT2: 1048P, Avionics:BAT_1048P, symbol Avionics (1):1048P
- BAT3: renamed from BAT1; footprint (none) -> Avionics:BAT_1048P
- C1, C2, COUT1, COUT2, COUT3, COUT4: footprint (none) -> Capacitor_SMD:C_0805_2012Metric
- C3, C5: renamed from C7; footprint (none) -> Capacitor_SMD:C_0805_2012Metric
- C4: renamed from C5; footprint (none) -> Capacitor_SMD:C_0805_2012Metric
- C6: renamed from C4; footprint (none) -> Capacitor_SMD:C_0805_2012Metric
- C7: renamed from C3; footprint (none) -> Capacitor_SMD:C_0805_2012Metric
- CBAT1: renamed from CBAT; footprint (none) -> Capacitor_SMD:C_0805_2012Metric
- CBAT2: renamed from CBAT1; footprint (none) -> Capacitor_SMD:C_0805_2012Metric
- CIN1: renamed from CIN; footprint (none) -> Capacitor_SMD:C_0805_2012Metric
- CIN2: renamed from CIN1; footprint (none) -> Capacitor_SMD:C_0805_2012Metric
- D1, D2, D3, D4, D5, D6: footprint (none) -> LED_SMD:LED_0805_2012Metric
- J1: renamed from J2; footprint (none) -> Connector_PinHeader_1.00mm:PinHeader_1x07_P1.00mm_Vertical
- L1: renamed from L2; footprint (none) -> Inductor_SMD:L_0805_2012Metric
- L2: renamed from L1; footprint (none) -> Inductor_SMD:L_0805_2012Metric
- L3: renamed from L; footprint (none) -> Inductor_SMD:L_0805_2012Metric
- L4: renamed from L3; footprint (none) -> Inductor_SMD:L_0805_2012Metric
- R1, R2, R3, R4, R5, R6: footprint (none) -> Resistor_SMD:R_0805_2012Metric
- RIN1: renamed from RIN; footprint (none) -> Resistor_SMD:R_0805_2012Metric
- RIN2: renamed from RIN1; footprint (none) -> Resistor_SMD:R_0805_2012Metric
- U1: footprint CB_16_8_ADI -> Avionics:CB_16_8_ADI
- U2, U3: footprint DSE0006A -> Avionics:DSE0006A
Connections:
- net GND: now also BAT3.2 (-), BAT3.3 (-), BAT1.2 (-), BAT1.3 (-), BAT2.2 (-), BAT2.3 (-)
- net VIN1: no longer C1.1, U1.B3 (ENA), U1.B4 (ENB), U1.C1 (VIN1)
- net VIN2: now also BAT3.1 (+)
- net VIN3: now also BAT2.4 (+)
- net VIN4: now also BAT2.1 (+)
- net VIN5: now also BAT1.4 (+)
- net VIN6: now also BAT1.1 (+)
- net Battery IN: now reaches BAT3.4 (+)
- net Battery IN: now also C1.1, U1.B3 (ENA), U1.B4 (ENB), U1.C1 (VIN1)
Other:
- moved on the sheet: BAT3, D1, D2, D3, D4, D5, D6, J1, R1, R2, R3, R4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

Commit message: Housekeeping File Updates
- Removed extra PCB file that somehow got onto the repo
- Updated PCB file with footprints
Parts:
- removed BAT1, BAT2, BAT3: 1048P, Avionics:BAT_1048P, symbol Avionics (1):1048P
- added J2: Conn_01x12_Pin, symbol Connector:Conn_01x12_Pin
Connections:
- net Battery IN is gone; now on net VIN1: C1.1, U1.B3 (ENA), U1.B4 (ENB), U1.C1 (VIN1)

Commit message: Add USB and 5V / 3A Topology
Parts:
- removed J2: Conn_01x12_Pin, symbol Connector:Conn_01x12_Pin
- added C10, C11, C12, C13: C, symbol Device:C
- added C8: 1uF, Capacitor_SMD:C_0805_2012Metric, symbol Device:C
- added C9: 4.7uF, symbol Device:C
- added D7, D8: LED, symbol Device:LED
- added J2: Conn_02x06_Row_Letter_Last, symbol Connector_Generic:Conn_02x06_Row_Letter_Last
- added L5: 2.2uH, symbol Device:L
- added P1: USB_C_Plug_USB2.0, symbol Connector:USB_C_Plug_USB2.0
- added R10, R9: 10kΩ, Resistor_SMD:R_0805_2012Metric, symbol Device:R
- added R11: 187kΩ, symbol Device:R
- added R12: 1MΩ, symbol Device:R
- added R13: R, symbol Device:R
- added R7: 1kΩ, symbol Device:R
- added R8: 5kΩ, symbol Device:R
- added U4: USBLC6-2P6, Package_TO_SOT_SMD:SOT-666, symbol Power_Protection:USBLC6-2P6
- added U4: BQ25185DLHR, WSON10_DLH_TEX, symbol Avionics (1):BQ25185DLHR
- added U5: LT8609AEDDM-5#TRPBF, SON50P300X300X85-11N-D, symbol Avionics (1):LT8609AEDDM-5#TRPBF
Connections:
- net GND: now also C12.1, C13.2, C8.1, C9.2, J2.1b (Pin_1b), J2.2b (Pin_2b), J2.3b (Pin_3b), J2.4b (Pin_4b), J2.5b (Pin_5b), J2.6b (Pin_6b), P1.A1 (GND), P1.A12 (GND), P1.B1 (GND), P1.B12 (GND), R10.1, R11.1, R13.2, R7.2, R8.2, R9.1, U4.2 (GND), U4.4 (/CE), U4.5 (GND), U5.11 (GND)
- net VIN1: now also J2.1a (Pin_1a)
- net VIN2: now also J2.2a (Pin_2a)
- net VIN3: now also J2.3a (Pin_3a)
- net VIN4: now also J2.4a (Pin_4a)
- net VIN5: now also J2.5a (Pin_5a)
- net VIN6: now also J2.6a (Pin_6a)
- new net: D7.2 (A), R9.2
- new net: P1.A7 (D-), U4.1 (I/O1)
- new net: P1.A6 (D+), U4.3 (I/O2)
- new net: R13.1, U5.4 (RT)
- new net: C13.1, U5.3 (INTVCC)
- new net: R8.1, U4.7 (ILIM/VSET)
- new net: D8.2 (A), R10.2
- new net: C10.2, U5.1 (BST)
- new net: C10.1, L5.2, U5.2 (SW)
- new net: R7.1, U4.8 (ISET)
- new net BAT+: U4.2 (BAT)
- new net D+: U4.4 (I/O2)
- new net D-: U4.6 (I/O1)
- new net FB: C11.1, R11.2, R12.1, U5.6 (FB)
- new net STAT1: D7.1 (K), U4.9 (STAT1)
- new net STAT2: D8.1 (K), U4.3 (STAT2)
- new net VBUS: C8.2, P1.A4 (VBUS), P1.A9 (VBUS), P1.B4 (VBUS), P1.B9 (VBUS), U4.10 (IN), U4.5 (VBUS)
- new net VIN7: C9.1, U5.9 (VIN)
- new net VOUT8: C11.2, C12.2, L5.1, R12.2
- no-connect marks 3 -> 8
Other:
- note added: "6V TO 40V"
- note added: "INPUT / OUTPUT"
- note added: "SOURCE THREE"
- note added: "STATUS LEDs"
- note added: "VOUT 8 5V 3A"
- note removed: "Battery Supply Network"
- moved on the sheet: C1, C2, C3, C4, C5, C6, C7, CBAT1, CBAT2, CIN1, CIN2, COUT1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

Commit message: Schematic Updates. NOTE: ERC Fails
Parts:
- added J3: Screw_Terminal_01x02, symbol Connector:Screw_Terminal_01x02
Connections:
- net BAT+: now also J3.2 (Pin_2)
- new net VBAT: J3.1 (Pin_1)
- no-connect marks 8 -> 13
Other:
- note added: "USB-C CHARGING & DATA PASSTHROUGH"
- moved on the sheet: C8, D1, D2, D3, D4, D5, D6, D7, D8, J1, J2, P1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

Commit message: Assigned Footprints and Updated I/O Pins in Schematic
Parts:
- removed J1: Conn_01x07_Pin, Connector_PinHeader_1.00mm:PinHeader_1x07_P1.00mm_Vertical, symbol Connector:Conn_01x07_Pin
- removed J2: Conn_02x06_Row_Letter_Last, symbol Connector_Generic:Conn_02x06_Row_Letter_Last
- added D9: LED, LED_SMD:LED_0805_2012Metric, symbol Device:LED
- added J1: Conn_01x08_Pin, Connector_Pin:Pin_D1.0mm_L10.0mm, symbol Connector:Conn_01x08_Pin
- added J2: Conn_02x07_Row_Letter_Last, Connector_Pin:Pin_D1.0mm_L10.0mm, symbol Connector_Generic:Conn_02x07_Row_Letter_Last
- added R1: 10kΩ, Resistor_SMD:R_0805_2012Metric, symbol Device:R
- C10: renamed from C11; footprint (none) -> Capacitor_SMD:C_0805_2012Metric
- C11: renamed from C12; footprint (none) -> Capacitor_SMD:C_0805_2012Metric
- C12: renamed from C13; footprint (none) -> Capacitor_SMD:C_0805_2012Metric
- C8: renamed from C10; footprint (none) -> Capacitor_SMD:C_0805_2012Metric
- C9: footprint (none) -> Capacitor_SMD:C_0805_2012Metric
- D7, D8: footprint (none) -> LED_SMD:LED_0805_2012Metric
- J3: footprint (none) -> Connector_Phoenix_MSTB:PhoenixContact_MSTBA_2,5_2-G-5,08_1x02_P5.08mm_Horizontal
- L5, P1: footprint (none) -> Inductor_SMD:L_0805_2012Metric
- R10: renamed from R12; footprint (none) -> Resistor_SMD:R_0805_2012Metric
- R11: renamed from R13; footprint (none) -> Resistor_SMD:R_0805_2012Metric
- R12: renamed from R11; footprint (none) -> Resistor_SMD:R_0805_2012Metric
- R13: renamed from R8; footprint (none) -> Resistor_SMD:R_0805_2012Metric
- R14: renamed from R7; footprint (none) -> Resistor_SMD:R_0805_2012Metric
- U4: renamed from U5; footprint SON50P300X300X85-11N-D -> SRAD_Avionics:LT8609AEDDMs
- U6: renamed from U4; footprint WSON10_DLH_TEX -> SRAD_Avionics:BQ25185DLHR
- renumbered C3 to C1, C8 to C13, C1 to C2, C6 to C3, C2 to C4, C7 to C5, C5 to C6, C4 to C7, L3 to L1, L1 to L2, L4 to L3, L2 to L4, R1 to R2, R2 to R3, R3 to R4, R4 to R5, R5 to R6, R6 to R7, R9 to R8, R10 to R9, U2 to U1, U1 to U2, U4 to U5
Connections:
- net GND: now also J2.1b (Pin_1b), J2.2b (Pin_2b), J2.3b (Pin_3b), J2.4b (Pin_4b), J2.5b (Pin_5b), J2.6b (Pin_6b), J2.7b (Pin_7b), R1.1
- net STAT1: now also D8.1 (K); no longer D7.1 (K)
- net STAT2: now also D9.1 (K); no longer D8.1 (K)
- net VIN1: now also D7.1 (K), J2.1a (Pin_1a); no longer D6.1 (K)
- net VIN2: now also D6.1 (K), J2.2a (Pin_2a); no longer D5.1 (K)
- net VIN3: now also D5.1 (K), J2.3a (Pin_3a); no longer D4.1 (K)
- net VIN4: now also D4.1 (K), J2.4a (Pin_4a); no longer D3.1 (K)
- net VIN5: now also D3.1 (K), J2.5a (Pin_5a); no longer D2.1 (K)
- net VIN6: now also D2.1 (K), J2.6a (Pin_6a); no longer D1.1 (K)
- net VIN7: now also D1.1 (K), J2.7a (Pin_7a)
- net VOUT1: now also J1.1 (Pin_1)
- net VOUT2: now also J1.2 (Pin_2)
- net VOUT3: now also J1.3 (Pin_3)
- net VOUT4: now also J1.4 (Pin_4)
- net VOUT5: now also J1.5 (Pin_5)
- net VOUT6: now also J1.6 (Pin_6)
- net VOUT7: now also J1.7 (Pin_7)
- net VOUT8: now also J1.8 (Pin_8)
- net at D7.2 (A): now also R7.2; no longer R8.2
- net at R2.2: now also D2.2 (A); no longer D1.2 (A)
- net at R3.2: now also D3.2 (A); no longer D2.2 (A)
- net at R9.2: now also D9.2 (A); no longer D8.2 (A)
- net at R4.2: now also D4.2 (A); no longer D3.2 (A)
- net at D6.2 (A): now also R6.2; no longer R7.2
- net at D5.2 (A): now also R5.2; no longer R6.2
- new net: D1.2 (A), R1.2
- new net: D8.2 (A), R8.2
- no-connect marks 13 -> 14
Other:
- moved on the sheet: R2, R3, R4, R5, R6, R7, R8, R9

Commit message: Meeting
Connections:
- net GND: now also P1.S1 (SHIELD)
- no-connect marks 14 -> 13
Other:
- moved on the sheet: P1
Changed lines of the file:
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@@
 	)
 	(junction
+		(at 29.21 187.96)
+		(diameter 0)
+		(color 0 0 0 0)
+	)
+	(junction
 		(at 50.8 46.99)
 		(diameter 0)
@@
 	)
 	(no_connect
-		(at 21.2073 185.0423)
-	)
-	(no_connect
 		(at 97.79 157.48)
 	)
 	(no_connect
-		(at 44.0673 152.0223)
+		(at 44.45 153.035)
 	)
 	(no_connect
@@
 	)
 	(no_connect
-		(at 44.0673 154.5623)
+		(at 44.45 155.575)
 	)
 	(no_connect
@@
 	(wire
 		(pts
-			(xy 45.3373 164.7223) (xy 45.3373 163.4523)
+			(xy 45.3373 165.735) (xy 45.3373 163.4523)
 		)
 		(stroke
@@
 	(wire
 		(pts
-			(xy 45.3373 159.6423) (xy 45.3373 160.9123)
+			(xy 45.3373 160.655) (xy 45.3373 160.9123)
 		)
 		(stroke
@@
 	(wire
 		(pts
+			(xy 29.21 187.96) (xy 29.21 189.865)
+		)
+		(stroke
+			(width 0)
+			(type default)
+		)
+	)
+	(wire
+		(pts
 			(xy 208.28 34.29) (xy 208.28 39.37)
 		)
@@
 	(wire
 		(pts
-			(xy 44.0673 164.7223) (xy 45.3373 164.7223)
+			(xy 44.45 165.735) (xy 45.3373 165.735)
 		)
 		(stroke
@@
 	(wire
 		(pts
+			(xy 29.21 186.055) (xy 29.21 187.96)
+		)
+		(stroke
+			(width 0)
+			(type default)
+		)
+	)
+	(wire
+		(pts
 			(xy 190.5 123.19) (xy 190.5 140.97)
 		)
@@
 	(wire
 		(pts
+			(xy 44.45 147.955) (xy 49.53 147.955)
+		)
+		(stroke
+			(width 0)
+			(type default)
+		)
+	)
+	(wire
+		(pts
 			(xy 85.09 160.02) (xy 97.79 160.02)
 		)
@@
 	(wire
 		(pts
-			(xy 44.0673 159.6423) (xy 45.3373 159.6423)
+			(xy 44.45 160.655) (xy 45.3373 160.655)
 		)
 		(stroke
@@
 	(wire
 		(pts
+			(xy 21.59 186.055) (xy 21.59 187.96)
+		)
+		(stroke
+			(width 0)
+			(type default)
+		)
+	)
+	(wire
+		(pts
 			(xy 208.28 39.37) (xy 212.09 39.37)
 		)
@@
 	(wire
 		(pts
+			(xy 21.59 187.96) (xy 29.21 187.96)
+		)
+		(stroke
+			(width 0)
+			(type default)
+		)
+	)
+	(wire
+		(pts
 			(xy 209.55 130.81) (xy 209.55 140.97)
 		)
@@
 	)
 	(symbol
+		(lib_id "power:GND")
+		(at 29.21 189.865 0)
+		(unit 1)
+		(exclude_from_sim no)
+		(in_bom yes)
+		(on_board yes)
+		(dnp no)
+		(fields_autoplaced yes)
+		(property "Reference" "#PWR036"
+			(at 29.21 196.215 0)
+			(effects
+				(font
+					(size 1.27 1.27)
+				)
+				(hide yes)
+			)
+		)
+		(property "Value" "GND"
+			(at 29.21 194.3548 0)
+			(effects
+				(font
+					(size 1.27 1.27)
+				)
+			)
+		)
+		(property "Footprint" ""
+			(at 29.21 189.865 0)
+			(effects
+				(font
+					(size 1.27 1.27)
+				)
+				(hide yes)
+			)
+		)
+		(property "Datasheet" ""
+			(at 29.21 189.865 0)
+			(effects
+				(font
+					(size 1.27 1.27)
+				)
+				(hide yes)
+			)
+		)
+		(property "Description" "Power symbol creates a global label with name \"GND\" , ground"
+			(at 29.21 189.865 0)
+			(effects
+				(font
+					(size 1.27 1.27)
+				)
+				(hide yes)
+			)
+		)
+		(pin "1"
+		)
+		(instances
+			(project "power-delivery-board"
+				(path "/ede041fa-5c95-4d07-be56-df14cd7dcdb2"
+					(reference "#PWR036")
+					(unit 1)
+				)
+			)
+		)
+	)
+	(symbol
 		(lib_id "Device:C")
 		(at 256.54 129.54 0)
@@
 	(symbol
 		(lib_id "Connector:USB_C_Plug_USB2.0")
-		(at 28.8273 162.1823 0)
+		(at 29.21 163.195 0)
 		(unit 1)
 		(exclude_from_sim no)
@@
 		(dnp no)
 		(property "Reference" "P1"
-			(at 14.2669 162.4953 90)
+			(at 14.6496 163.508 90)
 			(effects
 				(font
@@
 		)
 		(property "Value" "USB_C_Plug_USB2.0"
-			(at 16.8069 162.4953 90)
+			(at 17.1896 163.508 90)
 			(effects
 				(font
@@
 		)
 		(property "Footprint" "Inductor_SMD:L_0805_2012Metric"
-			(at 32.6373 162.1823 0)
+			(at 33.02 163.195 0)
 			(effects
 				(font
@@
 		)
 		(property "Datasheet" "https://www.usb.org/sites/default/files/documents/usb_type-c.zip"
-			(at 32.6373 162.1823 0)
+			(at 33.02 163.195 0)
 			(effects
 				(font
@@
 		)
 		(property "Description" "USB 2.0-only Type-C Plug connector"
-			(at 28.8273 162.1823 0)
+			(at 29.21 163.195 0)
 			(effects
 				(font
@@
 	)
 	(symbol
-		(lib_id "power:VBUS")
-		(at 44.0673 146.9423 270)
+		(lib_id "Device:L")
+		(at 195.58 123.19 90)
 		(unit 1)
 		(exclude_from_sim no)
@@
 		(dnp no)
 		(fields_autoplaced yes)
-		(property "Reference" "#PWR026"
-			(at 40.2573 146.9423 0)
+		(property "Reference" "L5"
+			(at 195.58 118.11 90)
 			(effects
 				(font
 					(size 1.27 1.27)
 				)
-				(hide yes)
 			)
 		)
-		(property "Value" "VBUS"
-			(at 47.8773 146.9422 90)
+		(property "Value" "2.2uH"
+			(at 195.58 120.65 90)
 			(effects
 				(font
 					(size 1.27 1.27)
 				)
-				(justify left)
 			)
 		)
-		(property "Footprint" ""
-			(at 44.0673 146.9423 0)
+		(property "Footprint" "Inductor_SMD:L_0805_2012Metric"
+			(at 195.58 123.19 0)
 			(effects
 				(font
@@
 			)
 		)
-		(property "Datasheet" ""
-			(at 44.0673 146.9423 0)
+		(property "Datasheet" "~"
+			(at 195.58 123.19 0)
 			(effects
 				(font
@@
 			)
 		)
-		(property "Description" "Power symbol creates a global label with name \"VBUS\""
-			(at 44.0673 146.9423 0)
+		(property "Description" "Inductor"
+			(at 195.58 123.19 0)
 			(effects
 				(font
@@
 			)
 		)
+		(pin "2"
+		)
 		(pin "1"
 		)
@@
 			(project ""
 				(path "/ede041fa-5c95-4d07-be56-df14cd7dcdb2"
-					(reference "#PWR026")
+					(reference "L5")
 					(unit 1)
 				)
@@
 	)
 	(symbol
-		(lib_id "Device:L")
-		(at 195.58 123.19 90)
+		(lib_id "power:VBUS")
+		(at 49.53 147.955 270)
 		(unit 1)
 		(exclude_from_sim no)
@@
 		(dnp no)
 		(fields_autoplaced yes)
-		(property "Reference" "L5"
-			(at 195.58 118.11 90)
+		(property "Reference" "#PWR026"
+			(at 45.72 147.955 0)
 			(effects
 				(font
 					(size 1.27 1.27)
 				)
+				(hide yes)
 			)
 		)
-		(property "Value" "2.2uH"
-			(at 195.58 120.65 90)
+		(property "Value" "VBUS"
+			(at 53.34 147.9549 90)
 			(effects
 				(font
 					(size 1.27 1.27)
 				)
+				(justify left)
 			)
 		)
-		(property "Footprint" "Inductor_SMD:L_0805_2012Metric"
-			(at 195.58 123.19 0)
+		(property "Footprint" ""
+			(at 49.53 147.955 0)
 			(effects
 				(font
@@
 			)
 		)
-		(property "Datasheet" "~"
-			(at 195.58 123.19 0)
+		(property "Datasheet" ""
+			(at 49.53 147.955 0)
 			(effects
 				(font
@@
 			)
 		)
-		(property "Description" "Inductor"
-			(at 195.58 123.19 0)
+		(property "Description" "Power symbol creates a global label with name \"VBUS\""
+			(at 49.53 147.955 0)
 			(effects
 				(font
@@
 			)
 		)
-		(pin "2"
-		)
 		(pin "1"
 		)
 		(instances
-			(project ""
+			(project "power-delivery-board"
 				(path "/ede041fa-5c95-4d07-be56-df14cd7dcdb2"
-					(reference "L5")
+					(reference "#PWR026")
 					(unit 1)
 				)
@@
 					(unit 1)
 				)
-			)
-		)
-	)
-	(symbol
-		(lib_id "power:GND")
-		(at 28.8273 185.0423 0)
-		(unit 1)
-		(exclude_from_sim no)
-		(in_bom yes)
-		(on_board yes)
-		(dnp no)
-		(fields_autoplaced yes)
-		(property "Reference" "#PWR036"
-			(at 28.8273 191.3923 0)
-			(effects
-				(font
-					(size 1.27 1.27)
-				)
-				(hide yes)
-			)
-		)
-		(property "Value" "GND"
-			(at 28.8273 189.5321 0)
-			(effects
-				(font
-					(size 1.27 1.27)
-				)
-			)
-		)
-		(property "Footprint" ""
-			(at 28.8273 185.0423 0)
-			(effects
-				(font
-					(size 1.27 1.27)
-				)
-				(hide yes)
-			)
-		)
-		(property "Datasheet" ""
-			(at 28.8273 185.0423 0)
-			(effects
-				(font
-					(size 1.27 1.27)
-				)
-				(hide yes)
-			)
-		)
-		(property "Description" "Power symbol creates a global label with name \"GND\" , ground"
-			(at 28.8273 185.0423 0)
-			(effects
-				(font
-					(size 1.27 1.27)
-				)
-				(hide yes)
-			)
-		)
-		(pin "1"
-		)
-		(instances
-			(project ""
-				(path "/ede041fa-5c95-4d07-be56-df14cd7dcdb2"
-					(reference "#PWR036")
-					(unit 1)
-				)
