File: Spaceport/PCBs/low_power_module/low_power_module.kicad_pcb (KiCad board)
At the start: 2 copper layers, 40 x 70 mm, 11 parts, among them J1 Conn_Coaxial, U1 Si4463

Commit message: TCXO and Decoupling Caps Added
TCXO
- A 30MHz TCXO was added:
https://www.digikey.com/en/products/detail/raltron-electronics/RTX-104CHZ1-S-32-000-TR/14558648?s=N4IgjCBcoOwdIDGUBmBDANgZwKYBoQB7KAbRAGZywAmANmpAF0CAHAFyhAGU2AnASwB2AcxABfAmAAc5KKGSR02fEVIgALGAAM9Wk1YdI3PkNESQ1AKyyECpbgLFIZGpb3MQ7TjwEjxBajBLLTkkVEwHVWcKLQACAFkACQAvfU9DEABVQX42AHkUeJw0LABXXhxxcwZogBUAYQANPKYxIA

- 10nF Decoupling capacitors were added to VCC

- PCB Layout not updated
Parts:
- moved XO 15.6 mm to (148.8, 82.8), turned to -90 degrees
- moved R1 11.7 mm to (158.8, 71.8), turned to 90 degrees
- moved RFS1 10.1 mm to (159.7, 81.4)
- moved U1 0.78 mm to (152.1, 89.4)
- renumbered XO-1 to XO
Routing:
- net GND: track 0.00 -> 20.8 mm, vias 0 -> 7
- net +3.3V: track 0.00 -> 2.12 mm

Commit message: Added Teensy 4.1 to Schematic
PCB Layout NOT Complete
Parts:
- removed C1, C2: 4.3pF, Capacitor_SMD:C_0805_2012Metric
- removed C3: 56pF, Capacitor_SMD:C_0805_2012Metric
- removed J1: Conn_Coaxial, Connector_Coaxial:SMA_Amphenol_132289_EdgeMount
- removed L1: 8.2nH, Inductor_SMD:L_0805_2012Metric
- removed L2: L, Inductor_SMD:L_0805_2012Metric
- removed R1: R, Resistor_SMD:R_0805_2012Metric
- removed R2: R, Inductor_SMD:L_0805_2012Metric
- removed RFS1: CG2409M2, RF:CG2409M2-C4
- removed U1: Si4463, Package_DFN_QFN:QFN-20-1EP_4x4mm_P0.5mm_EP2.6x2.6mm_ThermalVias
- removed XO: DSC1001CI5-030.0000, XO:CDFN4_3P2X2P5_MCH
Routing:
- net GND: track 20.8 -> 7.00 mm, vias 7 -> 0
- net +3.3V: track 2.12 -> 0.00 mm
Other:
- board outline removed

Commit message: minor schematic fixes and first pass at layout
Also fixed .gitignore
Parts:
- added C0: C, Capacitor_SMD:C_0805_2012Metric_Pad1.18x1.45mm_HandSolder, F.Cu at (118.8, 102.8)
- added C8: 1uF, Capacitor_SMD:C_0805_2012Metric_Pad1.18x1.45mm_HandSolder, F.Cu at (112.6, 88.0)
- added C9: 1uF, Capacitor_SMD:C_0805_2012Metric_Pad1.18x1.45mm_HandSolder, F.Cu at (118.6, 88.0)
- added CB0: 10nF, Capacitor_SMD:C_0805_2012Metric_Pad1.18x1.45mm_HandSolder, F.Cu at (128.7, 96.8)
- added CB1: C, Capacitor_SMD:C_0805_2012Metric_Pad1.18x1.45mm_HandSolder, F.Cu at (114.5, 93.4)
- added CB2: C, Capacitor_SMD:C_0805_2012Metric_Pad1.18x1.45mm_HandSolder, F.Cu at (116.5, 93.4)
- added CB3: C, Capacitor_SMD:C_0805_2012Metric_Pad1.18x1.45mm_HandSolder, F.Cu at (115.6, 86.4)
- added CD0: 10uF, Capacitor_SMD:C_0805_2012Metric_Pad1.18x1.45mm_HandSolder, F.Cu at (127.2, 107.0)
- added CD1: 10uF, Capacitor_SMD:C_0805_2012Metric_Pad1.18x1.45mm_HandSolder, F.Cu at (127.2, 105.0)
- added CD2: 10uF, Capacitor_SMD:C_0805_2012Metric_Pad1.18x1.45mm_HandSolder, F.Cu at (133.8, 93.8)
- added CM1: C, Capacitor_SMD:C_0805_2012Metric_Pad1.18x1.45mm_HandSolder, F.Cu at (110.7, 98.8)
- added CM2: C, Capacitor_SMD:C_0805_2012Metric_Pad1.18x1.45mm_HandSolder, F.Cu at (115.8, 82.2)
- added CM3: C, Capacitor_SMD:C_0805_2012Metric_Pad1.18x1.45mm_HandSolder, F.Cu at (121.9, 84.2)
- added CM4: C, Capacitor_SMD:C_0805_2012Metric_Pad1.18x1.45mm_HandSolder, F.Cu at (111.8, 101.7)
- added CR1: 2.2pF, Capacitor_SMD:C_0805_2012Metric_Pad1.18x1.45mm_HandSolder, F.Cu at (119.7, 100.8)
- added CR2: 2.2pF, Capacitor_SMD:C_0805_2012Metric_Pad1.18x1.45mm_HandSolder, F.Cu at (122.8, 96.2)
- added D1: LED, LED_SMD:LED_0805_2012Metric_Pad1.15x1.40mm_HandSolder, F.Cu at (175.0, 82.4)
- added D2: LED, LED_SMD:LED_0805_2012Metric_Pad1.15x1.40mm_HandSolder, F.Cu at (175.0, 85.3)
- added D3: LED, LED_SMD:LED_0805_2012Metric_Pad1.15x1.40mm_HandSolder, F.Cu at (175.0, 88.2)
- added D4: LED, LED_SMD:LED_0805_2012Metric_Pad1.15x1.40mm_HandSolder, F.Cu at (175.0, 91.2)
- added H1: MountingHole, MountingHole:MountingHole_2.2mm_M2, F.Cu at (160.0, 83.8)
- added H2: MountingHole, MountingHole:MountingHole_2.2mm_M2, F.Cu at (160.0, 89.7)
- added H3: MountingHole, MountingHole:MountingHole_2.2mm_M2, F.Cu at (160.0, 95.7)
- added H4: MountingHole, MountingHole:MountingHole_2.2mm_M2, F.Cu at (160.0, 101.6)
- added J1: SMA, adafruit:SMA_EDGELAUNCH, F.Cu at (122.0, 77.7)
- added J2: Conn_01x06_Pin, Connector_PinHeader_2.54mm:PinHeader_1x06_P2.54mm_Vertical, F.Cu at (165.8, 95.8)
- added J3: Conn_01x06_Pin, Connector_PinHeader_2.54mm:PinHeader_1x06_P2.54mm_Vertical, F.Cu at (169.9, 83.1)
- added L0: L, Inductor_SMD:L_0805_2012Metric_Pad1.15x1.40mm_HandSolder, F.Cu at (114.7, 102.8)
- added LChoke1: L, Inductor_SMD:L_0805_2012Metric_Pad1.15x1.40mm_HandSolder, F.Cu at (121.8, 103.8)
- added LM1: L, Inductor_SMD:L_0805_2012Metric_Pad1.15x1.40mm_HandSolder, F.Cu at (109.8, 101.8)
- added LM2: L, Inductor_SMD:L_0805_2012Metric_Pad1.15x1.40mm_HandSolder, F.Cu at (109.8, 95.8)
- added LM3: L, Inductor_SMD:L_0805_2012Metric_Pad1.15x1.40mm_HandSolder, F.Cu at (118.9, 83.2)
- added LR1: 62nH, Inductor_SMD:L_0805_2012Metric_Pad1.15x1.40mm_HandSolder, F.Cu at (122.8, 100.0)
- added LR2: 56nH, Inductor_SMD:L_0805_2012Metric_Pad1.15x1.40mm_HandSolder, F.Cu at (120.8, 96.2)
- added R3: 1k, Resistor_SMD:R_0805_2012Metric_Pad1.20x1.40mm_HandSolder, F.Cu at (178.8, 82.3)
- added R4: 1k, Resistor_SMD:R_0805_2012Metric_Pad1.20x1.40mm_HandSolder, F.Cu at (178.8, 85.3)
- added R5: 1k, Resistor_SMD:R_0805_2012Metric_Pad1.20x1.40mm_HandSolder, F.Cu at (178.8, 88.2)
- added R6: 1k, Resistor_SMD:R_0805_2012Metric_Pad1.20x1.40mm_HandSolder, F.Cu at (178.8, 91.2)
- added RFS1: CG2409M2, Avionics:CG2409M2, F.Cu at (115.6, 89.9)
- added TCXO2: TG2520SMN, Avionics:TG2520SMN, F.Cu at (130.8, 94.2)
- added U1: Si4463, Package_DFN_QFN:QFN-20-1EP_4x4mm_P0.5mm_EP2.6x2.6mm_ThermalVias, F.Cu at (126.8, 100.8)
Routing:
- net SDN: track 0.00 -> 14.0 mm
- net GPIO3: track 0.00 -> 12.9 mm
- net GPIO2: track 0.00 -> 12.9 mm
- net GPIO0: track 0.00 -> 8.67 mm
- net GPIO1: track 0.00 -> 7.83 mm
- net IRQ: track 0.00 -> 7.26 mm
- net SCLK: track 0.00 -> 7.20 mm
- net MISO: track 0.00 -> 7.13 mm
- net MOSI: track 0.00 -> 7.07 mm
- net GND: track 7.00 -> 0.00 mm
- net CS: track 0.00 -> 7.00 mm
- added copper zone on F.Cu, net +3.3V
- added copper zone on F.Cu, net GND
- removed copper zone on B.Cu, net GND
Other:
- board outline added: 37.5 x 32 mm

Commit message: tweak PA component values
Parts:
- removed J2, J3: Conn_01x06_Pin, Connector_PinHeader_2.54mm:PinHeader_1x06_P2.54mm_Vertical
- C0: value C -> 9.1pF
- CB1, CB2, CB3: value C -> 1u
- CM1: value C -> 4.7pF
- CM2, CM3: value C -> 22pF
- CM4: value C -> 15pF
- CR1: value 2.2pF -> 4.7pF
- L0: value L -> 33nH
- LChoke1: value L -> 220nH
- LM1, LM2: value L -> 56nH
- LM3: value L -> 10nH

Commit message: update filters
Routing:
- net GPIO3: track 12.9 -> 20.9 mm
- net SDN: track 14.0 -> 6.52 mm
Changed lines of the file:
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@@
 	)
 	(segment
-		(start 125.75 93.684314)
-		(end 131.217157 88.217157)
+		(start 125.75 98.065686)
+		(end 125.75 93.352943)
+		(width 0.2)
+		(layer "F.Cu")
+		(net 11)
+	)
+	(segment
+		(start 122.147057 89.75)
+		(end 114.265164 89.75)
+		(width 0.2)
+		(layer "F.Cu")
+		(net 11)
+	)
+	(segment
+		(start 113.65 89.134836)
+		(end 113.65 88.00455)
 		(width 0.2)
 		(layer "F.Cu")
@@
 	(segment
 		(start 125.75 98.9)
-		(end 125.75 93.684314)
+		(end 125.332843 98.482843)
+		(width 0.2)
+		(layer "F.Cu")
+		(net 11)
+	)
+	(segment
+		(start 114.265164 89.75)
+		(end 113.65 89.134836)
+		(width 0.2)
+		(layer "F.Cu")
+		(net 11)
+	)
+	(segment
+		(start 125.75 93.352943)
+		(end 122.147057 89.75)
+		(width 0.2)
+		(layer "F.Cu")
+		(net 11)
+	)
+	(segment
+		(start 125.332843 98.482843)
+		(end 125.75 98.065686)
 		(width 0.2)
 		(layer "F.Cu")
@@
 		(width 0.2)
 		(layer "F.Cu")
-		(net 23)
-	)
-	(segment
-		(start 125.35 93.518628)
-		(end 130.618629 88.25)
-		(width 0.2)
-		(layer "F.Cu")

Commit message: Edited Trace Width on 50Ω microstrip and Changed Layout with New Filter
Parts:
- removed LM2: 56nH, Inductor_SMD:L_0805_2012Metric_Pad1.15x1.40mm_HandSolder
- added CM5: 22pF, Capacitor_SMD:C_0805_2012Metric_Pad1.18x1.45mm_HandSolder, F.Cu at (109.8, 96.0)
- added Teensy4.1: ~, SRAD_Avionics:Teensy_4.1, F.Cu at (147.1, 99.9)
- CM1: value 4.7pF -> 22pF
- LM1: value 56nH -> 10nH
- moved R3 65.1 mm to (121.8, 113.9)
- moved D1 65.1 mm to (118.0, 113.9)
- moved D2 65.1 mm to (118.0, 116.8)
- moved D3 65.1 mm to (118.0, 119.8)
- moved D4 65.1 mm to (118.0, 122.8)
- moved R4 65.1 mm to (121.8, 116.8)
- moved R5 65.1 mm to (121.8, 119.8)
- moved R6 65.1 mm to (121.8, 122.8)
- moved H3 60.3 mm to (111.8, 131.8)
- moved H1 50.2 mm to (111.8, 69.8)
- moved H4 30.3 mm to (162.8, 131.8)
- moved H2 20.1 mm to (162.8, 69.8)
- moved J1 12.0 mm to (122.0, 65.7)
- moved TCXO2 4.12 mm to (131.8, 98.2)
- moved CD2 2.47 mm to (132.2, 95.8), turned to 180 degrees
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Connections:
- CM4 pad 1: Net-(CM4-Pad1) -> Net-(CM1-Pad1)
- L0 pad 2: Net-(CM4-Pad1) -> Net-(CM1-Pad1)
- LM1 pad 1: Net-(CM4-Pad1) -> Net-(CM1-Pad1)
- LM1 pad 2: Net-(CM1-Pad1) -> RF2
Routing:
- net GPIO3: track 20.9 -> 0.00 mm
- net GPIO2: track 12.9 -> 0.00 mm
- net GPIO0: track 8.67 -> 0.00 mm
- net GPIO1: track 7.83 -> 0.00 mm
- net IRQ: track 7.26 -> 0.00 mm
- net SCLK: track 7.20 -> 0.00 mm
- net MISO: track 7.13 -> 0.00 mm
- net MOSI: track 7.07 -> 0.00 mm
- net CS: track 7.00 -> 0.00 mm
- net SDN: track 6.52 -> 0.00 mm
Other:
- board size 37.5 x 32 mm -> 57.2 x 69 mm

Commit message: More PCB Routing Completed
Parts:
- moved R5 29.0 mm to (124.8, 90.9), turned to 90 degrees
- moved D3 24.7 mm to (124.8, 96.1), turned to 90 degrees
- moved R4 20.2 mm to (135.2, 101.8)
- moved D2 20.0 mm to (131.2, 101.8)
- moved R3 19.5 mm to (135.2, 99.8)
- moved D1 19.4 mm to (131.2, 99.8)
- moved D4 14.5 mm to (121.8, 108.8), turned to -90 degrees
- moved R6 10.0 mm to (121.8, 112.8), turned to -90 degrees
- moved TCXO 5.60 mm to (127.8, 94.3), turned to -90 degrees
- moved H1 5.50 mm to (106.2, 69.8)
- moved H3 5.50 mm to (106.2, 131.8)
- moved CD2 2.46 mm to (130.2, 94.3), turned to -90 degrees
- moved CM1 1.75 mm to (108.8, 99.0)
- moved CM5 1.41 mm to (108.8, 97.0), turned to 0 degrees
- moved Teensy4.1 0.89 mm to (148.0, 99.8)
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- renumbered TCXO2 to TCXO
Connections:
- CB1 pad 2: RF1 -> RF2
- CB2 pad 1: RF2 -> RF1
Routing:
- net Net-(J1-In): track 0.00 -> 15.5 mm
- net Net-(CM1-Pad1): track 0.00 -> 9.18 mm
- net RF2: track 0.00 -> 7.51 mm
- net +3.3V: track 0.00 -> 7.47 mm
- net TX: track 0.00 -> 5.59 mm
- net RXp: track 0.00 -> 4.34 mm
- net Net-(CB3-Pad2): track 0.00 -> 4.32 mm
- net RXn: track 0.00 -> 4.25 mm
- net RF1: track 0.00 -> 3.91 mm
- net Net-(D3-A): track 0.00 -> 3.12 mm
- net SDN: track 0.00 -> 2.76 mm
- net Net-(RFS1-RF1): track 0.00 -> 2.38 mm
- net XO_IN: track 0.00 -> 2.30 mm
- net Net-(RFS1-RF2): track 0.00 -> 2.25 mm
- net Net-(C0-Pad2): track 0.00 -> 2.00 mm
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Other:
- board size 57.2 x 69 mm -> 62.2 x 69 mm

Commit message: Routed more. Added ground plane. DC power and GND pins remain.
Parts:
- moved D1 1.38 mm to (132.5, 99.2)
- moved R3 1.38 mm to (136.5, 99.2)
- moved CD0 1.25 mm to (127.2, 108.2)
- moved CD1 1.25 mm to (127.2, 106.2)
- moved D2 0.96 mm to (131.5, 102.8)
- moved R4 0.96 mm to (135.5, 102.8)
Routing:
- net SCLK: track 0.00 -> 29.3 mm
- net SDN: track 2.76 -> 20.2 mm
- net MISO: track 0.00 -> 12.8 mm
- net MOSI: track 0.00 -> 12.0 mm
- net +3.3V: track 7.47 -> 12.9 mm
- net RXn: track 4.25 -> 7.75 mm
- net CS: track 1.55 -> 3.04 mm
- net IRQ: track 1.55 -> 2.18 mm
- added copper zone on B.Cu, net GND
