File: Spaceport/PCBs/MCU Boards/Teensy MCU Board v2.0 - compact/mcu-board v2.kicad_pcb (KiCad board)
At the start: 2 copper layers, 30.8 x 62 mm, 16 parts, among them J11 Screw_Terminal_01x02, J2 Conn_01x04, J4 Conn_01x04, J9 Conn_01x02

Commit message: generated gerbers
Parts:
- R5, R6: value 220Ω -> 1kΩ
- moved H1 0.60 mm to (117.3, 46.0)
- moved H2 0.60 mm to (117.3, 100.8)
- moved R5 0.20 mm to (118.3, 82.0)
- moved D1 0.12 mm to (118.4, 77.2)
Routing:
- net GND: track 18.6 -> 3.55 mm, vias 0 -> 2
Changed lines of the file:
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@@
 			(outputformat 1)
 			(mirror no)
-			(drillshape 1)
+			(drillshape 0)
 			(scaleselection 1)
-			(outputdirectory "")
+			(outputdirectory "../../Gerbers/Teensy-MCU-Board-v2.0/")
 		)
 	)
@@
 	(footprint "MountingHole:MountingHole_3.2mm_M3"
 		(layer "F.Cu")
-		(at 116.75 46)
+		(at 117.348 46)
 		(descr "Mounting Hole 3.2mm, no annular, M3")
 		(tags "mounting hole 3.2mm no annular m3")
@@
 	(footprint "LED_SMD:LED_0805_2012Metric_Pad1.15x1.40mm_HandSolder"
 		(layer "F.Cu")
-		(at 118.525 77.25)
+		(at 118.4 77.25)
 		(descr "LED SMD 0805 (2012 Metric), square (rectangular) end terminal, IPC_7351 nominal, (Body size source: https://docs.google.com/spreadsheets/d/1BsfQQcO9C6DZCsRaXUlFlo91Tg2WpOkGARC1WS5S8t0/edit?usp=sharing), generated with kicad-footprint-generator")
 		(tags "LED handsolder")
@@
 			)
 		)
-		(property "Value" "220Ω"
+		(property "Value" "1kΩ"
 			(at 0 1.5 90)
 			(layer "F.SilkS")
@@
 	(footprint "Resistor_SMD:R_0805_2012Metric_Pad1.20x1.40mm_HandSolder"
 		(layer "F.Cu")
-		(at 118.5 82)
+		(at 118.3 82)
 		(descr "Resistor SMD 0805 (2012 Metric), square (rectangular) end terminal, IPC_7351 nominal with elongated pad for handsoldering. (Body size source: IPC-SM-782 page 72, https://www.pcb-3d.com/wordpress/wp-content/uploads/ipc-sm-782a_amendment_1_and_2.pdf), generated with kicad-footprint-generator")
 		(tags "resistor handsolder")
@@
 			)
 		)
-		(property "Value" "220Ω"
+		(property "Value" "1kΩ"
 			(at 0 1.65 0)
 			(layer "F.SilkS")
@@
 	(footprint "MountingHole:MountingHole_3.2mm_M3"
 		(layer "F.Cu")
-		(at 116.75 100.75)
+		(at 117.348 100.75)
 		(descr "Mounting Hole 3.2mm, no annular, M3")
 		(tags "mounting hole 3.2mm no annular m3")
@@
 	)
 	(segment
-		(start 110.75 99.025)
-		(end 110.75 99)
+		(start 111 99.025)
+		(end 111.471 99.025)
 		(width 0.2)
 		(layer "F.Cu")
@@
 	)
 	(segment
-		(start 111 99.025)
-		(end 118.75 91.275)
+		(start 110.75 99.025)
+		(end 110.75 99)
 		(width 0.2)
 		(layer "F.Cu")
@@
 	)
 	(segment
-		(start 111.75 74)
-		(end 112 74)
+		(start 117.375 77.25)
+		(end 115.858 77.25)
 		(width 0.2)
 		(layer "F.Cu")
@@
 	)
 	(segment
-		(start 118.75 91.275)
-		(end 118.75 90.75)
+		(start 111.471 99.025)
+		(end 112.522 100.076)
 		(width 0.2)
 		(layer "F.Cu")
@@
 	)
 	(segment
-		(start 115.25 77.25)
-		(end 117.5 77.25)
+		(start 115.858 77.25)
+		(end 115.824 77.216)
 		(width 0.2)
 		(layer "F.Cu")
 		(net 2)
 	)
-	(segment
-		(start 112 74)
-		(end 115.25 77.25)
-		(width 0.2)
-		(layer "F.Cu")
+	(via
+		(at 112.522 100.076)
+		(size 0.6)
+		(drill 0.3)
+		(layers "F.Cu" "B.Cu")
+		(net 2)
+	)
+	(via
+		(at 115.824 77.216)
+		(size 0.6)
+		(drill 0.3)
+		(layers "F.Cu" "B.Cu")
 		(net 2)
 	)
@@
 	)
 	(segment
-		(start 117.5 82)
-		(end 117.25 82)
-		(width 0.2)
-		(layer "F.Cu")
-		(net 7)
-	)
-	(segment
 		(start 120.6 67.35)
 		(end 120.6 71.65)
@@
 	)
 	(segment
-		(start 117.5 82)
-		(end 118.75 83.25)
-		(width 0.2)
+		(start 116.75 81.5)
+		(end 118.5 83.25)
+		(width 0.5)
 		(layer "F.Cu")
 		(net 7)
 	)
 	(segment
-		(start 120.65 82.85)
-		(end 120.65 73.9)
-		(width 0.2)
+		(start 111.75 81.5)
+		(end 116.75 81.5)
+		(width 0.5)
 		(layer "F.Cu")
 		(net 7)
 	)
 	(segment
-		(start 113 59.75)
-		(end 120.6 67.35)
-		(width 0.3)
+		(start 120.5 83)
+		(end 120.5 73.75)
+		(width 0.5)
 		(layer "F.Cu")
 		(net 7)
 	)
 	(segment
-		(start 118.75 83.25)
-		(end 120.25 83.25)
-		(width 0.2)
-		(layer "F.Cu")
-		(net 7)
-	)
-	(segment
-		(start 117.25 82)
-		(end 116.75 81.5)
-		(width 0.2)
+		(start 113 59.75)
+		(end 120.6 67.35)
+		(width 0.3)
 		(layer "F.Cu")
 		(net 7)
@@
 		(start 117.5 68.25)
 		(end 119.5 70.25)
-		(width 0.2)
+		(width 0.5)
 		(layer "F.Cu")
 		(net 7)
@@
 		(start 112.25 59.75)
 		(end 112.25 54.12)
-		(width 0.3)
+		(width 0.5)
 		(layer "F.Cu")
 		(net 7)
@@
 	(segment
 		(start 120.25 83.25)
-		(end 120.65 82.85)
-		(width 0.2)
+		(end 120.5 83)
+		(width 0.5)
+		(layer "F.Cu")
+		(net 7)
+	)
+	(segment
+		(start 120.5 73.75)
+		(end 119.5 72.75)
+		(width 0.5)
 		(layer "F.Cu")
 		(net 7)
@@
 		(start 112.25 54.12)
 		(end 107.378125 49.248125)
-		(width 0.3)
+		(width 0.5)
 		(layer "F.Cu")
 		(net 7)
@@
 		(start 119.5 70.25)
 		(end 119.5 72.75)
-		(width 0.2)
+		(width 0.5)
 		(layer "F.Cu")
 		(net 7)
@@
 	)
 	(segment
-		(start 120.65 73.9)
-		(end 119.5 72.75)
-		(width 0.2)
-		(layer "F.Cu")
-		(net 7)
-	)
-	(segment
-		(start 116.75 81.5)
-		(end 111.75 81.5)
-		(width 0.2)
+		(start 118.5 83.25)
+		(end 120.25 83.25)
+		(width 0.5)
 		(layer "F.Cu")
 		(net 7)
@@
 		(start 115.25 51.75)
 		(end 114.5 51.75)
-		(width 0.4)
+		(width 0.5)
 		(layer "F.Cu")
 		(net 10)
@@
 		(start 118.25 62.75)
 		(end 120 61)
-		(width 0.4)
+		(width 0.5)
 		(layer "F.Cu")
 		(net 10)
@@
 		(start 120 56.5)
 		(end 115.25 51.75)
-		(width 0.4)
+		(width 0.5)
 		(layer "F.Cu")
 		(net 10)
@@
 		(start 120 61)
 		(end 120 56.5)
-		(width 0.4)
+		(width 0.5)
 		(layer "F.Cu")
 		(net 10)
@@
 		(start 109.75 46.54)
 		(end 107.378125 44.168125)
-		(width 0.45)
+		(width 0.5)
 		(layer "F.Cu")
 		(net 11)
@@
 		(start 114.5 54.29)
 		(end 109.75 49.54)
-		(width 0.45)
+		(width 0.5)
 		(layer "F.Cu")
 		(net 11)
@@
 		(start 109.75 49.54)
 		(end 109.75 46.54)
-		(width 0.45)
+		(width 0.5)
 		(layer "F.Cu")
 		(net 11)
