File: Spaceport/PCBs/MCU Boards/ESP32_BluetoothModule_TerrapinRockets/ESP32_BluetoothModule_TerrapinRockets.kicad_pcb (KiCad board)
At the start: 2 copper layers, 50.5 x 55 mm, 10 parts, among them J1 Conn_01x06, U1 ESP32-WROOM-32D

Commit message: JTAG Connection
Need this connection to program ESP- Check you tube video I sent to Varun
Parts:
- added J2: Conn_01x04, Connector_JST:JST_EH_B4B-EH-A_1x04_P2.50mm_Vertical, F.Cu at (78.0, 114.5)
- added R2: 100, Resistor_SMD:R_0402_1005Metric_Pad0.72x0.64mm_HandSolder, F.Cu at (83.6, 122.0)
- added R3: 100, Resistor_SMD:R_0402_1005Metric_Pad0.72x0.64mm_HandSolder, F.Cu at (83.6, 120.0)
- added R4: 100, Resistor_SMD:R_0402_1005Metric_Pad0.72x0.64mm_HandSolder, F.Cu at (83.6, 118.0)
- added R5: 100, Resistor_SMD:R_0402_1005Metric_Pad0.72x0.64mm_HandSolder, F.Cu at (83.6, 116.0)
- moved C1 27.5 mm to (116.0, 119.0), turned to 90 degrees
- moved C2 25.3 mm to (115.5, 115.5), turned to 90 degrees
- moved R1 24.6 mm to (115.5, 112.9), turned to 90 degrees
- moved C3 23.0 mm to (116.0, 122.6), turned to 90 degrees
Connections:
- U1 pad 13: unconnected-(U1-IO14-Pad13) -> Net-(U1-IO14)
- U1 pad 14: unconnected-(U1-IO12-Pad14) -> Net-(U1-IO12)
- U1 pad 16: unconnected-(U1-IO13-Pad16) -> Net-(U1-IO13)
- U1 pad 23: unconnected-(U1-IO15-Pad23) -> Net-(U1-IO15)
Routing:
- net Net-(U1-IO15): track 0.00 -> 26.0 mm, vias 0 -> 2
- net Net-(U1-IO13): track 0.00 -> 23.0 mm, vias 0 -> 2
- net Net-(J2-Pin_1): track 0.00 -> 12.8 mm
- net GND: track 79.6 -> 92.0 mm, vias 0 -> 1
- net +3.3V: track 52.3 -> 41.2 mm, vias 1 -> 2
- net Net-(J2-Pin_4): track 0.00 -> 9.77 mm, vias 0 -> 1
- net /EN: track 43.2 -> 51.6 mm
- net Net-(U1-IO12): track 0.00 -> 8.22 mm
- net Net-(J2-Pin_2): track 0.00 -> 8.20 mm
- net Net-(J2-Pin_3): track 0.00 -> 6.82 mm, vias 0 -> 1
- net /TX: track 8.73 -> 13.6 mm, vias 0 -> 1
- net Net-(U1-IO14): track 0.00 -> 4.49 mm

Commit message: . Added JTAG Pin connection
Parts:
- removed J2: Conn_01x04, Connector_JST:JST_EH_B4B-EH-A_1x04_P2.50mm_Vertical
- added J3: Conn_01x06, Connector_JST:JST_EH_B6B-EH-A_1x06_P2.50mm_Vertical, F.Cu at (79.0, 124.5)
Routing:
- net +3.3V: track 41.2 -> 63.6 mm, vias 2 -> 1
- net GND: track 92.0 -> 102.6 mm, vias 1 -> 0
- net Net-(U1-IO13): track 23.0 -> 14.7 mm
- net Net-(J3-Pin_2): track 12.8 -> 7.48 mm, vias 0 -> 1
- net /TX: track 13.6 -> 8.72 mm, vias 1 -> 0
- net Net-(J3-Pin_5): track 9.77 -> 5.82 mm, vias 1 -> 0
- net Net-(J3-Pin_3): track 8.20 -> 5.55 mm
- net Net-(U1-IO15): track 26.0 -> 28.0 mm
- net /EN: track 51.6 -> 53.1 mm, vias 1 -> 2
- net Net-(J3-Pin_4): track 6.82 -> 5.61 mm, vias 1 -> 0

Commit message: updated schematic
Other:
- board size 50.5 x 55 mm -> 50.5 x 58 mm
Changed lines of the file:
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@@
 	(gr_rect
 		(start 70 78)
-		(end 120.5 133)
+		(end 120.5 136)
 		(stroke
 			(width 0.05)

Commit message: modified schematic
Parts:
- C2, C3: footprint Capacitor_SMD:C_0402_1005Metric_Pad0.74x0.62mm_HandSolder -> Capacitor_SMD:C_0603_1608Metric_Pad1.08x0.95mm_HandSolder
- R1, R2, R3, R4, R5: footprint Resistor_SMD:R_0402_1005Metric_Pad0.72x0.64mm_HandSolder -> Resistor_SMD:R_0805_2012Metric_Pad1.20x1.40mm_HandSolder
- moved H3 75.4 mm to (133.0, 129.0)
- moved R5 40.4 mm to (122.5, 127.0), turned to 0 degrees
- moved H2 36.9 mm to (140.5, 110.5)
- moved J3 34.5 mm to (113.0, 130.5), turned to 0 degrees
- moved R4 33.6 mm to (116.0, 127.0)
- moved H4 32.5 mm to (106.0, 129.0)
- moved H1 25.5 mm to (100.0, 110.5)
- moved J1 24.9 mm to (132.5, 122.0)
- moved U1 23.9 mm to (119.2, 115.2)
- moved R2 23.7 mm to (107.0, 118.0), turned to 0 degrees
- moved R3 23.4 mm to (107.0, 120.5), turned to 0 degrees
- moved C1 14.6 mm to (107.0, 107.5), turned to 180 degrees
- moved C3 12.2 mm to (108.5, 113.0), turned to -90 degrees
- moved C2 10.4 mm to (107.0, 109.5), turned to 180 degrees
- moved R1 9.50 mm to (106.0, 113.0)
Connections:
- J1 pad 3: /TX -> /RX
- J1 pad 4: /RX -> /TX
- U1 pad 34: /TX -> /RX
- U1 pad 35: /RX -> /TX
Routing:
- net GND: track 102.6 -> 29.1 mm, vias 0 -> 4
- net Net-(U1-IO15): track 28.0 -> 2.38 mm, vias 2 -> 0
- net /EN: track 53.1 -> 32.7 mm, vias 2 -> 1
- net Net-(U1-IO13): track 14.7 -> 2.38 mm, vias 2 -> 0
- net Net-(J3-Pin_3): track 5.55 -> 16.4 mm
- net Net-(J3-Pin_2): track 7.48 -> 18.1 mm, vias 1 -> 0
- net +3.3V: track 63.6 -> 58.9 mm, vias 1 -> 0
- net Net-(U1-IO12): track 8.18 -> 4.54 mm
- net /TX: track 8.72 -> 6.05 mm
- net /IO0: track 13.9 -> 15.9 mm
- net Net-(J3-Pin_5): track 5.82 -> 4.12 mm
- net Net-(U1-IO14): track 4.64 -> 5.53 mm
- net Net-(J3-Pin_4): track 5.61 -> 4.95 mm
- added copper zone on B.Cu, net GND
Other:
- board size 50.5 x 58 mm -> 47.5 x 28.5 mm

Commit message: updated to esp32-s3
Parts:
- removed H1, H2: MountingHole, MountingHole:MountingHole_3.2mm_M3
- removed U1: ESP32-WROOM-32D, RF_Module:ESP32-WROOM-32D
- added J2: Conn_01x04, Connector_JST:JST_EH_B4B-EH-A_1x04_P2.50mm_Vertical, F.Cu at (132.0, 117.0)
- added U2: ESP32-S3-WROOM-1, RF_Module:ESP32-S3-WROOM-1, F.Cu at (119.8, 112.0)
- J1: value Conn_01x06 -> Conn_01x02; footprint Connector_JST:JST_EH_B6B-EH-A_1x06_P2.50mm_Vertical -> Connector_JST:JST_EH_B2B-EH-A_1x02_P2.50mm_Vertical
- moved J1 25.1 mm to (107.5, 120.0), turned to -90 degrees
- moved R5 19.3 mm to (107.0, 115.5)
- moved R3 14.5 mm to (120.0, 127.0)
- moved R2 12.7 mm to (116.0, 127.0)
- moved R4 8.00 mm to (124.0, 127.0)
- moved H3 1.12 mm to (132.0, 129.5)
- moved H4 0.71 mm to (106.5, 129.5)
- moved C3 0.50 mm to (108.5, 112.5)
- moved R1 0.50 mm to (106.0, 112.5)
Connections:
- J1 pad 1: GND -> /EN
- J1 pad 2: /EN -> /IO0
- R2 pad 2: Net-(U1-IO14) -> /IO12
- R3 pad 2: Net-(U1-IO12) -> /IO13
- R4 pad 2: Net-(U1-IO13) -> /IO14
- R5 pad 2: Net-(U1-IO15) -> /IO15
Routing:
- net Net-(J3-Pin_5): track 4.12 -> 27.6 mm, vias 0 -> 1
- net GND: track 29.1 -> 7.96 mm, vias 4 -> 5
- net /EN: track 32.7 -> 15.8 mm, vias 1 -> 0
- net Net-(J3-Pin_2): track 18.1 -> 3.71 mm
- net Net-(J3-Pin_3): track 16.4 -> 3.91 mm
- net /IO0: track 15.9 -> 25.3 mm, vias 0 -> 1
- net Net-(U1-IO14): track 5.53 -> 0.00 mm
- net Net-(U1-IO12): track 4.54 -> 0.00 mm
- net /IO12: track 0.00 -> 3.38 mm
- net /IO14: track 0.00 -> 3.06 mm
- net /IO15: track 0.00 -> 3.05 mm
- net /IO13: track 0.00 -> 2.75 mm
- net /RX: track 7.13 -> 4.61 mm
- net Net-(U1-IO15): track 2.38 -> 0.00 mm
- net Net-(U1-IO13): track 2.38 -> 0.00 mm
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Other:
- board size 47.5 x 28.5 mm -> 31 x 28.5 mm
- board text added: "3.3V"
- board text added: "EN"
- board text added: "GND"
- board text added: "IO0"
- board text added: "RX"
- board text added: "TRT AVIONICS BT v1.0"
- board text added: "TX"
