File: Spaceport/PCBs/MCU Boards/ESP32_BluetoothModule_TerrapinRockets/ESP32_BluetoothModule_TerrapinRockets.kicad_sch (KiCad schematic)
At the start: 10 parts, among them J1 Conn_01x06, U1 ESP32-WROOM-32D

Commit message: JTAG Connection
Need this connection to program ESP- Check you tube video I sent to Varun
Parts:
- added J2: Conn_01x04, Connector_JST:JST_EH_B4B-EH-A_1x04_P2.50mm_Vertical, symbol Connector_Generic:Conn_01x04
- added R2, R3, R4, R5: 100, Resistor_SMD:R_0402_1005Metric_Pad0.72x0.64mm_HandSolder, symbol Device:R
Connections:
- net at U1.13 (IO14): now also R2.2
- net at U1.14 (IO12): now also R3.2
- net at U1.16 (IO13): now also R4.2
- net at U1.23 (IO15): now also R5.2
- new net: J2.1 (Pin_1), R2.1
- new net: J2.2 (Pin_2), R3.1
- new net: J2.3 (Pin_3), R4.1
- new net: J2.4 (Pin_4), R5.1
- no-connect marks 30 -> 26

Commit message: . Added JTAG Pin connection
Parts:
- removed J2: Conn_01x04, Connector_JST:JST_EH_B4B-EH-A_1x04_P2.50mm_Vertical, symbol Connector_Generic:Conn_01x04
- added J3: Conn_01x06, Connector_JST:JST_EH_B6B-EH-A_1x06_P2.50mm_Vertical, symbol Connector_Generic:Conn_01x06
Connections:
- net +3.3V: now also J3.1 (Pin_1)
- net GND: now also J3.6 (Pin_6)
- net at R2.1: now also J3.2 (Pin_2)
- net at R3.1: now also J3.3 (Pin_3)
- net at R4.1: now also J3.4 (Pin_4)
- net at R5.1: now also J3.5 (Pin_5)

Commit message: updated schematic
Connections:
- net RX: now also J1.3 (Pin_3), U1.34 (RXD0/IO3); no longer J1.4 (Pin_4), U1.35 (TXD0/IO1)
- net TX: now also J1.4 (Pin_4), U1.35 (TXD0/IO1); no longer J1.3 (Pin_3), U1.34 (RXD0/IO3)
Changed lines of the file:
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@@
 		)
 	)
-	(label "RX"
+	(label "TX"
 		(at 240.03 127 0)
 		(effects
@@
 		)
 	)
-	(label "TX"
+	(label "RX"
 		(at 240.03 129.54 0)
 		(effects

Commit message: modified schematic
Parts:
- C2, C3: footprint Capacitor_SMD:C_0402_1005Metric_Pad0.74x0.62mm_HandSolder -> Capacitor_SMD:C_0603_1608Metric_Pad1.08x0.95mm_HandSolder
- R1, R2, R3, R4, R5: footprint Resistor_SMD:R_0402_1005Metric_Pad0.72x0.64mm_HandSolder -> Resistor_SMD:R_0805_2012Metric_Pad1.20x1.40mm_HandSolder
Changed lines of the file:
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@@
 			)
 		)
-		(property "Footprint" "Capacitor_SMD:C_0402_1005Metric_Pad0.74x0.62mm_HandSolder"
+		(property "Footprint" "Capacitor_SMD:C_0603_1608Metric_Pad1.08x0.95mm_HandSolder"
 			(at 108.9152 95.25 0)
 			(effects
@@
 			)
 		)
-		(property "Footprint" "Resistor_SMD:R_0402_1005Metric_Pad0.72x0.64mm_HandSolder"
+		(property "Footprint" "Resistor_SMD:R_0805_2012Metric_Pad1.20x1.40mm_HandSolder"
 			(at 106.172 76.2 90)
 			(effects
@@
 			)
 		)
-		(property "Footprint" "Capacitor_SMD:C_0402_1005Metric_Pad0.74x0.62mm_HandSolder"
+		(property "Footprint" "Capacitor_SMD:C_0603_1608Metric_Pad1.08x0.95mm_HandSolder"
 			(at 131.7752 54.61 0)
 			(effects
@@
 			)
 		)
-		(property "Footprint" "Resistor_SMD:R_0402_1005Metric_Pad0.72x0.64mm_HandSolder"
+		(property "Footprint" "Resistor_SMD:R_0805_2012Metric_Pad1.20x1.40mm_HandSolder"
 			(at 187.452 54.61 90)
 			(effects
@@
 			)
 		)
-		(property "Footprint" "Resistor_SMD:R_0402_1005Metric_Pad0.72x0.64mm_HandSolder"
+		(property "Footprint" "Resistor_SMD:R_0805_2012Metric_Pad1.20x1.40mm_HandSolder"
 			(at 179.832 54.61 90)
 			(effects
@@
 			)
 		)
-		(property "Footprint" "Resistor_SMD:R_0402_1005Metric_Pad0.72x0.64mm_HandSolder"
+		(property "Footprint" "Resistor_SMD:R_0805_2012Metric_Pad1.20x1.40mm_HandSolder"
 			(at 195.072 54.61 90)
 			(effects
@@
 			)
 		)
-		(property "Footprint" "Resistor_SMD:R_0402_1005Metric_Pad0.72x0.64mm_HandSolder"
+		(property "Footprint" "Resistor_SMD:R_0805_2012Metric_Pad1.20x1.40mm_HandSolder"
 			(at 202.692 54.61 90)
 			(effects

Commit message: updated to esp32-s3
Parts:
- removed H1, H2: MountingHole, MountingHole:MountingHole_3.2mm_M3, symbol Mechanical:MountingHole
- removed J1: Conn_01x06, Connector_JST:JST_EH_B6B-EH-A_1x06_P2.50mm_Vertical, symbol Connector_Generic:Conn_01x06
- removed U1: ESP32-WROOM-32D, RF_Module:ESP32-WROOM-32D, symbol RF_Module:ESP32-WROOM-32D
- added J1: Conn_01x02, Connector_JST:JST_EH_B2B-EH-A_1x02_P2.50mm_Vertical, symbol Connector_Generic:Conn_01x02
- added J2: Conn_01x04, Connector_JST:JST_EH_B4B-EH-A_1x04_P2.50mm_Vertical, symbol Connector_Generic:Conn_01x04
- added U2: ESP32-S3-WROOM-1, RF_Module:ESP32-S3-WROOM-1, symbol RF_Module:ESP32-S3-WROOM-1
Connections:
- net +3.3V: now also J2.4 (Pin_4), U2.2 (3V3)
- net EN: now also J1.1 (Pin_1), U2.3 (EN)
- net GND: now also J2.1 (Pin_1), U2.1 (GND), U2.40 (GND), U2.41 (GND)
- net IO0: now also J1.2 (Pin_2), U2.27 (IO0)
- net RX: now also J2.2 (Pin_2), U2.36 (RXD0)
- net TX: now also J2.3 (Pin_3), U2.37 (TXD0)
- net IO12: now reaches R2.2
- net IO12: now also U2.20 (IO12)
- net IO13: now reaches R3.2
- net IO13: now also U2.21 (IO13)
- net IO14: now reaches R4.2
- net IO14: now also U2.22 (IO14)
- net IO15: now reaches R5.2
- net IO15: now also U2.8 (IO15)
- no-connect marks 26 -> 1
Other:
- note added: "JTAG"
