File: Spaceport/PCBs/high-power-module/high-power-module.kicad_pcb (KiCad board)
At the start: 4 copper layers, 37.4 x 37.6 mm, 77 parts, among them J1 Conn_01x06_Pin, J2 SMA, J3 Conn_01x06_Pin, J4 Conn_01x02_Pin, U1 Si4463, U2 SN74LV1T08QDBVRQ1, U3 TPS62177DQCR

Commit message: add screw holes to HPM paste layer
Parts:
- moved H2 0.40 mm to (158.9, 73.5)
- moved H3 0.40 mm to (158.9, 97.5)
- moved H1 0.30 mm to (127.9, 73.5)
- moved H4 0.30 mm to (127.9, 97.5)
Changed lines of the file:
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@@
 	(footprint "MountingHole:MountingHole_3.2mm_M3"
 		(layer "F.Cu")
-		(at 128.2 97.5)
+		(at 127.9 97.5)
 		(descr "Mounting Hole 3.2mm, no annular, M3")
 		(tags "mounting hole 3.2mm no annular m3")
@@
 			(size 3.2 3.2)
 			(drill 3.2)
-			(layers "*.Cu" "*.Mask")
+			(layers "F&B.Cu" "*.Paste" "*.Mask")
 		)
 	)
@@
 	(footprint "MountingHole:MountingHole_3.2mm_M3"
 		(layer "F.Cu")
-		(at 128.2 73.5)
+		(at 127.9 73.5)
 		(descr "Mounting Hole 3.2mm, no annular, M3")
 		(tags "mounting hole 3.2mm no annular m3")
@@
 			(size 3.2 3.2)
 			(drill 3.2)
-			(layers "*.Cu" "*.Mask")
+			(layers "F&B.Cu" "*.Paste" "*.Mask")
 		)
 	)
@@
 	(footprint "MountingHole:MountingHole_3.2mm_M3"
 		(layer "F.Cu")
-		(at 158.5 73.5)
+		(at 158.9 73.5)
 		(descr "Mounting Hole 3.2mm, no annular, M3")
 		(tags "mounting hole 3.2mm no annular m3")
@@
 			(size 3.2 3.2)
 			(drill 3.2)
-			(layers "*.Cu" "*.Mask")
+			(layers "F&B.Cu" "*.Paste" "*.Mask")
 		)
 	)
 	(footprint "MountingHole:MountingHole_3.2mm_M3"
 		(layer "F.Cu")
-		(at 158.5 97.5)
+		(at 158.9 97.5)
 		(descr "Mounting Hole 3.2mm, no annular, M3")
 		(tags "mounting hole 3.2mm no annular m3")
@@
 			(size 3.2 3.2)
 			(drill 3.2)
-			(layers "*.Cu" "*.Mask")
+			(layers "F&B.Cu" "*.Paste" "*.Mask")
 		)
 	)

Commit message: update HPM based on sims
Parts:
- removed C1: 1u, Capacitor_SMD:C_0805_2012Metric_Pad1.18x1.45mm_HandSolder
- removed L4: 33nH, Inductor_SMD:L_0805_2012Metric_Pad1.15x1.40mm_HandSolder
- added CM6: 22pF, Capacitor_SMD:C_0805_2012Metric_Pad1.18x1.45mm_HandSolder, F.Cu at (139.7, 86.5)
- added CM7: 22pF, Capacitor_SMD:C_0805_2012Metric_Pad1.18x1.45mm_HandSolder, F.Cu at (139.7, 84.5)
- added CM8: 22pF, Capacitor_SMD:C_0805_2012Metric_Pad1.18x1.45mm_HandSolder, F.Cu at (130.7, 82.3)
- added CM9: 22pF, Capacitor_SMD:C_0805_2012Metric_Pad1.18x1.45mm_HandSolder, F.Cu at (134.7, 85.4)
- added L0: 15nH, Inductor_SMD:L_0805_2012Metric_Pad1.15x1.40mm_HandSolder, F.Cu at (139.8, 95.7)
- added LM4: 18nH, Inductor_SMD:L_0805_2012Metric_Pad1.15x1.40mm_HandSolder, F.Cu at (137.7, 93.8)
- added LM5: 11nH, Inductor_SMD:L_0805_2012Metric_Pad1.15x1.40mm_HandSolder, F.Cu at (142.5, 85.5)
- added LM6: 11nH, Inductor_SMD:L_0805_2012Metric_Pad1.15x1.40mm_HandSolder, F.Cu at (132.7, 83.4)
- C2: value 39p -> 36pF
- C3: value 100p -> 100pF
- C4: value 0.1u -> 0.1uF
- C5: value 10u -> 10uF
- C6: value 22p -> 39pF
- CB1, CB2, CB4: value 1u -> 1uF
- CM3: value 15pF -> 6.2pF
- L1: value 3.6n -> 3.3nH
- L2: value 56n -> 56nH
- L3: value 5.6n -> 3.0nH
- LM1, LM2: value 10nH -> 11nH
- R10, R11, R12, R4, R5, R6, R7, R8, R9: value 1k -> 2k
- R3: value 68n -> 68nH
- moved CM2 4.93 mm to (142.7, 76.5), turned to -90 degrees
- moved CM5 4.43 mm to (132.9, 96.6), turned to -90 degrees
- moved CM3 4.29 mm to (136.0, 95.8), turned to 180 degrees
- moved CB2 3.61 mm to (141.7, 82.5)
- moved C2 3.12 mm to (130.0, 91.9), turned to 0 degrees
- moved L1 3.07 mm to (132.9, 91.0), turned to -90 degrees
- moved CM1 2.96 mm to (135.9, 75.5)
- moved LM2 2.84 mm to (133.9, 93.8)
- moved CM4 2.77 mm to (134.9, 91.0)
- moved CB1 2.72 mm to (135.6, 82.5)
- moved C9 2.38 mm to (140.7, 79.4)
- moved C8 2.31 mm to (136.5, 79.4)
- moved RFS1 2.30 mm to (138.6, 81.9)
- moved CB4 2.27 mm to (138.6, 78.4)
- moved LM1 1.59 mm to (139.6, 75.5), turned to 0 degrees
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- renumbered C10 to C0
Connections:
- net PAout renamed Net-(L2-Pad2)
- C2 pad 1: GND -> PAin
- C2 pad 2: Net-(C1-Pad1) -> Net-(C2-Pad2)
- C6 pad 2: RF2 -> Net-(C6-Pad2)
- CD2 pad 1: GND -> +3.3V
- CD2 pad 2: +3.3V -> GND
- CD3 pad 1: GND -> +3.3V
- CD3 pad 2: +3.3V -> GND
- CM3 pad 2: GND -> Net-(CM3-Pad2)
- CM4 pad 1: Net-(CM3-Pad1) -> Net-(CM3-Pad2)
- CM5 pad 1: Net-(C1-Pad2) -> Net-(C2-Pad2)
- CR2 pad 2: RF1 -> Net-(CM6-Pad1)
- L1 pad 1: Net-(C1-Pad1) -> GND
- L1 pad 2: PAin -> Net-(C2-Pad2)
- L3 pad 2: RF2 -> Net-(C6-Pad2)
- LM2 pad 1: Net-(CM3-Pad1) -> Net-(CM3-Pad2)
- LM2 pad 2: Net-(C1-Pad2) -> Net-(C2-Pad2)
- LR2 pad 2: RF1 -> Net-(CM6-Pad1)
Routing:
- net Net-(C6-Pad2): track 0.00 -> 6.07 mm
- net Net-(C2-Pad2): track 0.00 -> 5.58 mm
- net Net-(CM3-Pad2): track 0.00 -> 5.58 mm
- net Net-(CM6-Pad1): track 0.00 -> 5.50 mm
- net GND: track 70.5 -> 74.8 mm, vias 34 -> 39
- net Net-(C1-Pad2): track 4.08 -> 0.00 mm
- net Net-(C1-Pad1): track 3.72 -> 0.00 mm
- net Net-(CM3-Pad1): track 5.48 -> 1.80 mm
- net GPIO2: track 47.6 -> 49.9 mm
- net GPIO3: track 67.7 -> 68.9 mm

Commit message: forgot to connect TCXO
Routing:
- net XO_IN: track 0.00 -> 1.68 mm
- net Net-(TCXO1-OUTPUT): track 0.00 -> 1.60 mm
Changed lines of the file:
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@@
 		(tags "capacitor handsolder")
 		(property "Reference" "CM6"
-			(at 1.3625 -1.68 360)
+			(at 1.3625 -1.68 0)
 			(layer "F.SilkS")
 			(effects
@@
 		)
 		(property "Value" "22pF"
-			(at 0 1.68 360)
+			(at 0 1.68 0)
 			(layer "F.Fab")
 			(hide yes)
@@
 		)
 		(fp_text user "${REFERENCE}"
-			(at 0 0 360)
+			(at 0 0 0)
 			(layer "F.Fab")
 			(effects
@@
 		(tags "inductor handsolder")
 		(property "Reference" "LM4"
-			(at -0.825 1.6 360)
+			(at -0.825 1.6 0)
 			(layer "F.SilkS")
 			(effects
@@
 		)
 		(property "Value" "18nH"
-			(at 0 1.65 360)
+			(at 0 1.65 0)
 			(layer "F.Fab")
 			(hide yes)
@@
 		)
 		(fp_text user "${REFERENCE}"
-			(at 0 0 360)
+			(at 0 0 0)
 			(layer "F.Fab")
 			(effects
@@
 		(tags "capacitor handsolder")
 		(property "Reference" "CM3"
-			(at 0 -1.5 360)
+			(at 0 -1.5 0)
 			(layer "F.SilkS")
 			(effects
@@
 		)
 		(property "Value" "6.2pF"
-			(at 0 1.68 360)
+			(at 0 1.68 0)
 			(layer "F.Fab")
 			(hide yes)
@@
 		)
 		(fp_text user "${REFERENCE}"
-			(at 0 0 360)
+			(at 0 0 0)
 			(layer "F.Fab")
 			(effects
@@
 		)
 		(property "Value" "22pF"
-			(at 0 1.68 360)
+			(at 0 1.68 0)
 			(layer "F.Fab")
 			(hide yes)
@@
 		)
 		(fp_text user "${REFERENCE}"
-			(at 0 0 360)
+			(at 0 0 0)
 			(layer "F.Fab")
 			(effects
@@
 		(tags "inductor handsolder")
 		(property "Reference" "L0"
-			(at 0 -1.4 360)
+			(at 0 -1.4 0)
 			(layer "F.SilkS")
 			(effects
@@
 		)
 		(property "Value" "15nH"
-			(at 0 1.65 360)
+			(at 0 1.65 0)
 			(layer "F.Fab")
 			(hide yes)
@@
 		)
 		(fp_text user "${REFERENCE}"
-			(at 0 0 360)
+			(at 0 0 0)
 			(layer "F.Fab")
 			(effects
@@
 		(tags "capacitor handsolder")
 		(property "Reference" "C2"
-			(at -2.7625 0 360)
+			(at -2.7625 0 0)
 			(layer "F.SilkS")
 			(effects
@@
 		)
 		(property "Value" "36pF"
-			(at 0 1.68 360)
+			(at 0 1.68 0)
 			(layer "F.Fab")
 			(hide yes)
@@
 		)
 		(fp_text user "${REFERENCE}"
-			(at 0 0 360)
+			(at 0 0 0)
 			(layer "F.Fab")
 			(effects
@@
 		(tags "capacitor handsolder")
 		(property "Reference" "CD3"
-			(at 3.2625 0 360)
+			(at 3.2625 0 0)
 			(layer "F.SilkS")
 			(effects
@@
 		)
 		(property "Value" "10uF"
-			(at 0 1.68 360)
+			(at 0 1.68 0)
 			(layer "F.Fab")
 			(hide yes)
@@
 		)
 		(fp_text user "${REFERENCE}"
-			(at 0 0 360)
+			(at 0 0 0)
 			(layer "F.Fab")
 			(effects
@@
 		(tags "capacitor handsolder")
 		(property "Reference" "CD2"
-			(at 3.2625 0 360)
+			(at 3.2625 0 0)
 			(layer "F.SilkS")
 			(effects
@@
 		)
 		(property "Value" "10uF"
-			(at 0 1.68 360)
+			(at 0 1.68 0)
 			(layer "F.Fab")
 			(hide yes)
@@
 		)
 		(fp_text user "${REFERENCE}"
-			(at 0 0 360)
+			(at 0 0 0)
 			(layer "F.Fab")
 			(effects
@@
 		(tags "capacitor handsolder")
 		(property "Reference" "CB2"
-			(at -3.3375 -0.7 360)
+			(at -3.3375 -0.7 0)
 			(layer "F.SilkS")
 			(effects
@@
 		)
 		(property "Value" "1uF"
-			(at 0 1.68 360)
+			(at 0 1.68 0)
 			(layer "F.Fab")
 			(hide yes)
@@
 		)
 		(fp_text user "${REFERENCE}"
-			(at 0 0 360)
+			(at 0 0 0)
 			(layer "F.Fab")
 			(effects
@@
 		)
 		(property "Value" "11nH"
-			(at 0 1.65 360)
+			(at 0 1.65 0)
 			(layer "F.Fab")
 			(hide yes)
@@
 		)
 		(fp_text user "${REFERENCE}"
-			(at 0 0 360)
+			(at 0 0 0)
 			(layer "F.Fab")
 			(effects
@@
 	)
 	(segment
+		(start 150.7 89.6)
+		(end 150.7 88)
+		(width 0.1524)
+		(layer "F.Cu")
+		(net 14)
+	)
+	(segment
+		(start 148.7 89.675)
+		(end 148.625 89.6)
+		(width 0.1524)
+		(layer "F.Cu")
+		(net 15)
+	)
+	(segment
+		(start 148.7 91.25)
+		(end 148.7 89.675)
+		(width 0.1524)
+		(layer "F.Cu")
+		(net 15)
+	)
+	(segment

Commit message: add AND gate decoupling cap
Parts:
- added CB5: 0.1uF, Capacitor_SMD:C_0805_2012Metric_Pad1.18x1.45mm_HandSolder, B.Cu at (140.6, 90.4)
Routing:
- net +5V: track 111.0 -> 112.8 mm
- net GND: track 74.8 -> 76.2 mm, vias 39 -> 40
