File: Spaceport/PCBs/high-power-module/high-power-module.kicad_sch (KiCad schematic)
At the start: 63 parts, among them J1 Conn_01x06_Pin, J2 SMA, J3 Conn_01x06_Pin, U1 Si4463, U2 SN74LVC1G00DBV

Commit message: Initial complete high power module
Parts:
- added CIN1: 2.2uF, Capacitor_SMD:C_0805_2012Metric, symbol Device:C
- added COUT1: 22uF, Capacitor_SMD:C_0805_2012Metric, symbol Device:C
- added H1, H2, H3, H4: MountingHole, MountingHole:MountingHole_3.2mm_M3, symbol Mechanical:MountingHole
- added J4: Conn_01x02_Pin, Connector_PinHeader_2.54mm:PinHeader_1x02_P2.54mm_Vertical, symbol Connector:Conn_01x02_Pin
- added L5: 10nH, Inductor_SMD:L_0805_2012Metric, symbol Device:L
- added R13: 215, Resistor_SMD:R_0805_2012Metric_Pad1.20x1.40mm_HandSolder, symbol Device:R
- added R15: 10k, Resistor_SMD:R_0805_2012Metric_Pad1.20x1.40mm_HandSolder, symbol Device:R
- added R16: 100k, Resistor_SMD:R_0805_2012Metric, symbol Device:R
- added R17: 0, Resistor_SMD:R_0805_2012Metric, symbol Device:R
- added U3: TPS62177DQCR, Avionics:TPS62177DQCR, symbol Avionics:TPS62177DQCR
- J1, J3: footprint Connector_PinHeader_2.54mm:PinHeader_1x06_P2.54mm_Vertical -> Connector_JST:JST_XH_B6B-XH-A_1x06_P2.50mm_Vertical
- R10, R11, R12, R4, R5, R6, R7, R8, R9: value 1k -> 2k
- R14: footprint Resistor_SMD:R_0805_2012Metric_Pad1.20x1.40mm_HandSolder -> Resistor_SMD:R_0805_2012Metric
- R2: value 240 -> 100k
- U2: value SN74LVC1G00DBV -> SN74LV1T08QDBVRQ1
- renumbered VCC1 to 3V3, VCC2 to 5V1
Connections:
- net +3.3V: now also 3V3.2 (A), R17.2; no longer 3V3.1 (K)
- net +5V: now also 5V1.2 (A), J1.6 (Pin_6), CIN1.2, U3.2 (VIN), U3.3 (EN); no longer 5V1.1 (K), J1.1 (Pin_1), R14.1
- net CS: now also CS1.2 (A), J1.1 (Pin_1); no longer CS1.1 (K), J1.6 (Pin_6)
- net GND: now also J1.5 (Pin_5), R2.1, CIN1.1, COUT1.2, J4.1 (Pin_1), R15.1, U3.1 (PGND), U3.11 (EXP), U3.6 (AGND), U3.P1 (EXP__1), U3.P2 (EXP__2), U3.P3 (EXP__3); no longer J1.2 (Pin_2)
- net GPIO0: now also GPIO0.2 (A), J3.5 (Pin_5); no longer GPIO0.1 (K), J3.1 (Pin_1)
- net GPIO1: now also GPIO1.2 (A), J3.4 (Pin_4); no longer GPIO1.1 (K), J3.2 (Pin_2)
- net GPIO2: now also GPIO2.2 (A); no longer GPIO2.1 (K)
- net GPIO3: now also GPIO3.2 (A), J3.2 (Pin_2), R15.2; no longer GPIO3.1 (K), J3.4 (Pin_4)
- net IRQ: now also IRQ1.2 (A), J3.6 (Pin_6); no longer IRQ1.1 (K), J3.5 (Pin_5)
- net MISO: now also J1.3 (Pin_3); no longer J1.5 (Pin_5)
- net MOSI: now also J1.2 (Pin_2); no longer J1.4 (Pin_4)
- net SCLK: now also J1.4 (Pin_4); no longer J1.3 (Pin_3)
- net SDN: now also J3.1 (Pin_1), SDN1.2 (A); no longer J3.6 (Pin_6), SDN1.1 (K)
- net at R6.1: now also GPIO2.1 (K); no longer GPIO2.2 (A)
- net at R12.1: now also 3V3.1 (K); no longer 3V3.2 (A)
- net at R2.2, U2.4: now also R13.2
- net at R7.1: now also GPIO1.1 (K); no longer GPIO1.2 (A)
- net at R10.1: now also IRQ1.1 (K); no longer IRQ1.2 (A)
- net at R9.1: now also CS1.1 (K); no longer CS1.2 (A)
- net at R11.1: now also SDN1.1 (K); no longer SDN1.2 (A)
- net AND: now reaches C4.2, D1.2 (K), R3.1
- net AND: now also R13.1; no longer R2.1
- net at R5.1: now also GPIO3.1 (K); no longer GPIO3.2 (A)
- net at R4.1: now also 5V1.1 (K); no longer 5V1.2 (A)
- net at R8.1: now also GPIO0.1 (K); no longer GPIO0.2 (A)
- new net: L5.1, U3.9 (SW)
- new net: COUT1.1, L5.2, R16.2, R17.1, U3.10 (VOS)
- new net: R16.1, U3.7 (PG)
- new net: J4.2 (Pin_2), R14.1
- no-connect marks 2 -> 5
Other:
- note added: "AND Gate"
- note added: "NOTE: GPIO3 HIGH TX GPIO2 HIGH RX"
- note added: "Power Conversion"
- note added: "VIN 4.75V TO 28V"
- note added: "VOUT 3.3V 500mA"
- note removed: "Power Conversion? TODO"
- moved on the sheet: 3V3, 5V1, CB3, CD1, CS1, GPIO0, GPIO1, GPIO2, GPIO3, IRQ1, J1, J3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

Commit message: update HPM based on sims
Parts:
- removed C1: 1u, Capacitor_SMD:C_0805_2012Metric_Pad1.18x1.45mm_HandSolder, symbol Device:C
- removed L4: 33nH, Inductor_SMD:L_0805_2012Metric_Pad1.15x1.40mm_HandSolder, symbol Device:L
- added CM6, CM7, CM8, CM9: 22pF, Capacitor_SMD:C_0805_2012Metric_Pad1.18x1.45mm_HandSolder, symbol Device:C
- added L0: 15nH, Inductor_SMD:L_0805_2012Metric_Pad1.15x1.40mm_HandSolder, symbol Device:L
- added LM4: 18nH, Inductor_SMD:L_0805_2012Metric_Pad1.15x1.40mm_HandSolder, symbol Device:L
- added LM5, LM6: 11nH, Inductor_SMD:L_0805_2012Metric_Pad1.15x1.40mm_HandSolder, symbol Device:L
- C2: value 39p -> 36pF
- C3: value 100p -> 100pF
- C4: value 0.1u -> 0.1uF
- C5: value 10u -> 10uF
- C6: value 22p -> 39pF
- CB1, CB2, CB4: value 1u -> 1uF
- CM3: value 15pF -> 6.2pF
- L1: value 3.6n -> 3.3nH
- L2: value 56n -> 56nH
- L3: value 5.6n -> 3.0nH
- LM1, LM2: value 10nH -> 11nH
- R3: value 68n -> 68nH
- renumbered C10 to C0
Connections:
- net +3.3V: now also CD2.1, CD3.1; no longer CD2.2, CD3.2
- net GND: now also CD2.2, CD3.2, L1.1, CM6.2, CM7.2, CM8.2, CM9.2, LM4.1; no longer C2.1, CD2.1, CD3.1, CM3.2
- net PAin: now also C2.1; no longer L1.2
- net RF1: now also CM7.1, LM5.2; no longer CR2.2, LR2.2
- net RF2: now also CM9.1, LM6.2; no longer C6.2, L3.2
- net at CM4.1, LM2.1: now also CM3.2, LM4.2; no longer CM3.1
- net at C0.2: now also L0.1
- net at C2.2: now also CM5.1, L1.2, LM2.2; no longer L1.1
- net PAout: no longer names the net of L2.2, L3.1, PA1.14 (RFout), PA1.15 (RFout), PA1.16 (RFout)
- new net: CM3.1, L0.2
- new net: CM6.1, CR2.2, LM5.1, LR2.2
- new net: C6.2, CM8.1, L3.2, LM6.1
Other:
- note added: "50Ohm match 434 MHz"
- note added: "Input DC block and PA match"
- note added: "PA stage"
- note removed: "50Ohm match for 434 MHz"
- note removed: "Input DC block and 50Ohm match"
- moved on the sheet: 3V3, 5V1, C0, C2, C3, C4, C5, C6, C8, C9, CB1, CB2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

Commit message: add AND gate decoupling cap
Parts:
- added CB5: 0.1uF, Capacitor_SMD:C_0805_2012Metric_Pad1.18x1.45mm_HandSolder, symbol Device:C
Connections:
- net +5V: now also CB5.1
- net GND: now also CB5.2
Changed lines of the file:
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@@
 	)
 	(junction
-		(at 250.19 76.2)
+		(at 175.26 121.92)
 		(diameter 0)
 		(color 0 0 0 0)
 	)
 	(junction
-		(at 175.26 121.92)
+		(at 250.19 76.2)
 		(diameter 0)
 		(color 0 0 0 0)
@@
 	)
 	(junction
+		(at 250.19 60.96)
+		(diameter 0)
+		(color 0 0 0 0)
+	)
+	(junction
 		(at 210.82 161.29)
 		(diameter 0)
@@
 	(symbol
 		(lib_id "power:+5V")
-		(at 250.19 76.2 180)
+		(at 250.19 60.96 0)
 		(unit 1)
 		(exclude_from_sim no)
@@
 		(on_board yes)
 		(dnp no)
-		(fields_autoplaced yes)
 		(property "Reference" "#PWR032"
-			(at 250.19 72.39 0)
+			(at 250.19 64.77 0)
 			(effects
 				(font
@@
 		)
 		(property "Value" "+5V"
-			(at 250.19 81.28 0)
+			(at 247.904 57.404 0)
 			(effects
 				(font
 					(size 1.27 1.27)
 				)
+				(justify left)
 			)
 		)
 		(property "Footprint" ""
-			(at 250.19 76.2 0)
+			(at 250.19 60.96 0)
 			(effects
 				(font
@@
 		)
 		(property "Datasheet" ""
-			(at 250.19 76.2 0)
+			(at 250.19 60.96 0)
 			(effects
 				(font
@@
 		)
 		(property "Description" "Power symbol creates a global label with name \"+5V\""
-			(at 250.19 76.2 0)
+			(at 250.19 60.96 0)
 			(effects
 				(font
@@
 	)
 	(symbol
+		(lib_id "Device:C")
+		(at 250.19 80.01 0)
+		(unit 1)
+		(exclude_from_sim no)
+		(in_bom yes)
+		(on_board yes)
+		(dnp no)
+		(property "Reference" "CB5"
+			(at 246.38 79.248 0)
+			(effects
+				(font
+					(size 1.27 1.27)
+				)
+			)
+		)
+		(property "Value" "0.1uF"
+			(at 246.38 81.788 0)
+			(effects
+				(font
+					(size 1.27 1.27)
+				)
+			)
+		)
+		(property "Footprint" "Capacitor_SMD:C_0805_2012Metric_Pad1.18x1.45mm_HandSolder"
+			(at 251.1552 83.82 0)
+			(effects
+				(font
+					(size 1.27 1.27)
+				)
+				(hide yes)
+			)
+		)
+		(property "Datasheet" "~"
+			(at 250.19 80.01 0)
+			(effects
+				(font
+					(size 1.27 1.27)
+				)
+				(hide yes)
+			)
+		)
+		(property "Description" "Unpolarized capacitor"
+			(at 250.19 80.01 0)
+			(effects
+				(font
+					(size 1.27 1.27)
+				)
+				(hide yes)
+			)
+		)
+		(pin "2"
+		)
+		(pin "1"
+		)
+		(instances
+			(project "high-power-module"
+				(path "/fd00db32-824a-4d36-8ae2-c391ba092059"
+					(reference "CB5")
+					(unit 1)
+				)
+			)
+		)
+	)
+	(symbol
 		(lib_id "power:GND")
 		(at 153.67 88.9 0)
@@
 					(unit 1)
 				)
+			)
+		)
+	)
+	(symbol
+		(lib_id "power:GND")
+		(at 250.19 83.82 0)
+		(unit 1)
+		(exclude_from_sim no)
+		(in_bom yes)
+		(on_board yes)
+		(dnp no)
+		(fields_autoplaced yes)
+		(property "Reference" "#PWR044"
+			(at 250.19 90.17 0)
+			(effects
+				(font
+					(size 1.27 1.27)
+				)
+				(hide yes)
+			)
+		)
+		(property "Value" "GND"
+			(at 250.19 88.9 0)
+			(effects
+				(font
+					(size 1.27 1.27)
+				)
+			)
+		)
+		(property "Footprint" ""
+			(at 250.19 83.82 0)
+			(effects
+				(font
+					(size 1.27 1.27)
+				)
+				(hide yes)
+			)
+		)
+		(property "Datasheet" ""
+			(at 250.19 83.82 0)
+			(effects
+				(font
+					(size 1.27 1.27)
+				)
+				(hide yes)
+			)
+		)
+		(property "Description" "Power symbol creates a global label with name \"GND\" , ground"
+			(at 250.19 83.82 0)
+			(effects
+				(font
+					(size 1.27 1.27)
+				)
+				(hide yes)
+			)
+		)
+		(pin "1"
+		)
+		(instances
+			(project "high-power-module"
+				(path "/fd00db32-824a-4d36-8ae2-c391ba092059"
+					(reference "#PWR044")
+					(unit 1)
+				)

Commit message: update HPM to v2
Parts:
- removed CIN1: 2.2uF, Capacitor_SMD:C_0805_2012Metric, symbol Device:C
- removed COUT1: 22uF, Capacitor_SMD:C_0805_2012Metric, symbol Device:C
- removed CS1, GPIO0, GPIO1, SDN1: LED, LED_SMD:LED_0805_2012Metric_Pad1.15x1.40mm_HandSolder, symbol Device:LED
- removed J4: Conn_01x02_Pin, Connector_PinHeader_2.54mm:PinHeader_1x02_P2.54mm_Vertical, symbol Connector:Conn_01x02_Pin
- removed L5: 10nH, Inductor_SMD:L_0805_2012Metric, symbol Device:L
- removed R11, R7, R8, R9: 2k, Resistor_SMD:R_0805_2012Metric_Pad1.20x1.40mm_HandSolder, symbol Device:R
- removed U3: TPS62177DQCR, Avionics:TPS62177DQCR, symbol Avionics:TPS62177DQCR
- added C1, C7: 1uF, Capacitor_SMD:C_0805_2012Metric_Pad1.18x1.45mm_HandSolder, symbol Device:C
- added CD4: 4.7u, Capacitor_SMD:C_0805_2012Metric_Pad1.18x1.45mm_HandSolder, symbol Device:C
- added CD5, CD6: 10n, Capacitor_SMD:C_0603_1608Metric_Pad1.08x0.95mm_HandSolder, symbol Device:C
- added J5: Conn_01x04_Pin, Connector_PinHeader_2.54mm:PinHeader_2x02_P2.54mm_Vertical, symbol Connector:Conn_01x04_Pin
- added J7: UART, Connector_JST:JST_XH_S4B-XH-A_1x04_P2.50mm_Horizontal, symbol Connector_Generic:Conn_01x04
- added Q1, Q2, Q3: PMOS, Avionics:AONS21309C, symbol Simulation_SPICE:PMOS
- added U3: MCP1703AT-3302E/MB, Avionics:SOT-89_3MC_MCH, symbol Avionics:MCP1703AT-3302E_MB
- added U4, U5: ~, Avionics:DIO_UDZSTE_ROM, symbol Avionics:UDZVTE-175.1B
- added U6: STM32F103C8Tx, Package_QFP:LQFP-48_7x7mm_P0.5mm, symbol MCU_ST_STM32F1:STM32F103C8Tx
- D1: value D_Zener_Dual_CommonAnode_KKA -> SM05T1G
- J1, J3: footprint Connector_JST:JST_XH_B6B-XH-A_1x06_P2.50mm_Vertical -> Connector_JST:JST_XH_S6B-XH-A_1x06_P2.50mm_Horizontal
- LM1, LM2, LM5, LM6: footprint Inductor_SMD:L_0805_2012Metric_Pad1.15x1.40mm_HandSolder -> Inductor_SMD:L_0603_1608Metric_Pad1.05x0.95mm_HandSolder
- LM4: footprint Inductor_SMD:L_0805_2012Metric_Pad1.15x1.40mm_HandSolder -> Inductor_SMD:L_0805_2012Metric_Pad1.05x1.20mm_HandSolder
- R10, R12, R4, R5, R6: value 2k -> 5.1k; footprint Resistor_SMD:R_0805_2012Metric_Pad1.20x1.40mm_HandSolder -> Resistor_SMD:R_0402_1005Metric_Pad0.72x0.64mm_HandSolder
- R14: value 0 -> 10k; footprint Resistor_SMD:R_0805_2012Metric -> Resistor_SMD:R_0805_2012Metric_Pad1.20x1.40mm_HandSolder
- R16: value 100k -> 10k; footprint Resistor_SMD:R_0805_2012Metric -> Resistor_SMD:R_0805_2012Metric_Pad1.20x1.40mm_HandSolder
- R17: value 0 -> 100M; footprint Resistor_SMD:R_0805_2012Metric -> Resistor_SMD:R_0805_2012Metric_Pad1.20x1.40mm_HandSolder
- U1: footprint Package_DFN_QFN:QFN-20-1EP_4x4mm_P0.5mm_EP2.6x2.6mm_ThermalVias -> Avionics:Si4463
- renumbered 5V1 to 5V0
Connections:
- net +3.3V: now also C1.2, CD4.1, CD5.1, CD6.1, U3.3, U6.1 (VBAT), U6.24 (VDD), U6.36 (VDD), U6.48 (VDD), U6.9 (VDDA); no longer R14.2, R17.2
- net +5V: now also C7.1, Q3.1 (D), U3.2; no longer J1.6 (Pin_6)
- net CS: now also U6.13 (PA3)
- net GND: now also R14.2, R16.1, C1.1, C7.2, CD4.2, CD5.2, CD6.2, J5.3 (Pin_3), J7.4 (Pin_4), U3.1, U4.2 (A), U6.23 (VSS), U6.35 (VSS), U6.47 (VSS), U6.8 (VSSA); no longer TCXO1.1 (NC), TCXO1.2 (GND), U1.18 (GND)
- net GPIO0: now also U6.18 (PB0)
- net GPIO1: now also U6.19 (PB1)
- net GPIO2: now also U6.20 (PB2)
- net GPIO3: now also U6.21 (PB10)
- net IRQ: now also U6.14 (PA4)
- net MISO: now also U6.16 (PA6)
- net MOSI: now also U6.17 (PA7)
- net SCLK: now also U6.15 (PA5)
- net SDN: now also U6.22 (PB11)
- net TX: now also J7.2 (Pin_2), U6.30 (PA9)
- net at R16.2: now also Q2.1 (D), Q3.2 (G); no longer R17.1
- net at R14.1: now also Q1.2 (G), U5.2 (A)
- new net: Q1.3 (S), Q2.3 (S), Q3.3 (S), R17.1, U5.1 (K)
- new net: Q2.2 (G), R17.2, U4.1 (K)
- new net GNDX: TCXO1.1 (NC), TCXO1.2 (GND), U1.18 (GND)
- new net NRST: J5.1 (Pin_1), U6.7 (NRST)
- new net RX: J7.3 (Pin_3), U6.31 (PA10)
- new net SWCLK: J5.4 (Pin_4), U6.37 (PA14)
- new net SWDIO: J5.2 (Pin_2), U6.34 (PA13)
- new net VIN: J1.6 (Pin_6), J7.1 (Pin_1), Q1.1 (D)
- no-connect marks 5 -> 26
Other:
- note added: "Circuit Protection"
- note added: "L2 >100 Ohm @ 434 Mhz Note: I(L2) > 1A"
- note added: "STM32"
- note added: "TCXO GND connected only to RF IC GNDX (pin 18)"
- note added: "VIN 2.7V to 16V"
- note added: "VOUT 3.3V 250mA"
- note removed: "L2 >100 Ohm @ 434 Mhz"
- note removed: "VIN 4.75V TO 28V"
- note removed: "VOUT 3.3V 500mA"
- moved on the sheet: GPIO2, GPIO3, IRQ1, R10, R5, R6

Commit message: HPM v2 finishing touches
Parts:
- added R7: 10k, Resistor_SMD:R_0805_2012Metric_Pad1.20x1.40mm_HandSolder, symbol Device:R
Connections:
- net +3.3V: now also R7.1
- net AND: now also R2.2, U2.4; no longer C4.2, D1.2 (K), R3.1
- net SDN: now also R7.2
- new net: C4.2, D1.2 (K), R13.2, R3.1
Other:
- moved on the sheet: C0, C1, C2, C3, C4, C5, C6, C7, C8, C9, CB1, CB2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

Commit message: add teardrops and VIN filter
Parts:
- added C10: 10uF, Capacitor_SMD:C_0805_2012Metric_Pad1.18x1.45mm_HandSolder, symbol Device:C
- added FB1: Wurth 7427931, Avionics:W7427931, symbol Device:FerriteBead
Connections:
- net GND: now also C10.2; no longer CD1.2
- net GNDX: now also CD1.2
- net TX: no longer J7.2 (Pin_2), U6.30 (PA9)
- net VIN: now also FB1.1; no longer Q1.1 (D)
- net RX renamed SRX
- new net: C10.1, FB1.2, Q1.1 (D)
- new net STX: J7.2 (Pin_2), U6.30 (PA9)

Commit message: HPM v2 rf layout improvements
Connections:
- net RXn: now also CR2.1, LR1.2; no longer CR1.2, LR1.1, LR2.1
- net RXp: now also CR1.2, LR1.1, LR2.1; no longer CR2.1, LR1.2
