File: Spaceport/PCBs/new-pa-test-board/new-pa-test-board.kicad_sch (KiCad schematic)
At the start: 14 parts, among them J1 Conn_Coaxial, J2 Conn_Coaxial, J3 Conn_01x03_Pin, J4 Conn_01x03_Pin, Q1 AFT05MS004NT1

Commit message: new pa board finishing updates
Parts:
- added R2: R, Resistor_SMD:R_0805_2012Metric_Pad1.20x1.40mm_HandSolder, symbol Device:R
- C1, C2, C7, C8: footprint (none) -> Capacitor_SMD:C_0805_2012Metric_Pad1.18x1.45mm_HandSolder
- FB2: footprint (none) -> Inductor_SMD:L_1806_4516Metric_Pad1.45x1.90mm_HandSolder
- J1, J2: footprint (none) -> adafruit:SMA_EDGELAUNCH
- J3, J4: footprint (none) -> Connector_PinHeader_2.54mm:PinHeader_1x03_P2.54mm_Vertical
- L1, L2, L3: footprint (none) -> Inductor_SMD:L_0805_2012Metric_Pad1.05x1.20mm_HandSolder
- Q1: footprint (none) -> Avionics:AFT05MS004NT1
- R1: footprint (none) -> Resistor_SMD:R_0805_2012Metric_Pad1.20x1.40mm_HandSolder
Connections:
- net VBIAS: now also J4.2 (Pin_2), R2.1; no longer J3.3 (Pin_3)
- net at C1.2, Q1.2 (G), R1.2: no longer J4.2 (Pin_2)
- no-connect marks 0 -> 2

Commit message: small new pa board updates and gerbers
Parts:
- C1, C2, C8: footprint Capacitor_SMD:C_0805_2012Metric_Pad1.18x1.45mm_HandSolder -> Capacitor_SMD:C_0603_1608Metric
- C7: footprint Capacitor_SMD:C_0805_2012Metric_Pad1.18x1.45mm_HandSolder -> Capacitor_SMD:C_0805_2012Metric
- J1, J2: footprint adafruit:SMA_EDGELAUNCH -> Adafruit:SMA_EDGELAUNCH
- L1, L2: footprint Inductor_SMD:L_0805_2012Metric_Pad1.05x1.20mm_HandSolder -> Inductor_SMD:L_0603_1608Metric
- L3: value 16.6nH -> 18nH; footprint Inductor_SMD:L_0805_2012Metric_Pad1.05x1.20mm_HandSolder -> Inductor_SMD:L_0805_2012Metric
Changed lines of the file:
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@@
 			)
 		)
-		(property "Footprint" "adafruit:SMA_EDGELAUNCH"
+		(property "Footprint" "Adafruit:SMA_EDGELAUNCH"
 			(at 171.45 91.44 0)
 			(effects
@@
 			)
 		)
-		(property "Footprint" "adafruit:SMA_EDGELAUNCH"
+		(property "Footprint" "Adafruit:SMA_EDGELAUNCH"
 			(at 101.6 92.71 0)
 			(effects
@@
 			)
 		)
-		(property "Footprint" "Capacitor_SMD:C_0805_2012Metric_Pad1.18x1.45mm_HandSolder"
+		(property "Footprint" "Capacitor_SMD:C_0603_1608Metric"
 			(at 119.38 91.7448 0)
 			(effects
@@
 			)
 		)
-		(property "Footprint" "Inductor_SMD:L_0805_2012Metric_Pad1.05x1.20mm_HandSolder"
+		(property "Footprint" "Inductor_SMD:L_0603_1608Metric"
 			(at 160.02 97.79 0)
 			(effects
@@
 			)
 		)
-		(property "Footprint" "Inductor_SMD:L_0805_2012Metric_Pad1.05x1.20mm_HandSolder"
+		(property "Footprint" "Inductor_SMD:L_0603_1608Metric"
 			(at 106.68 97.79 0)
 			(effects
@@
 			)
 		)
-		(property "Footprint" "Capacitor_SMD:C_0805_2012Metric_Pad1.18x1.45mm_HandSolder"
+		(property "Footprint" "Capacitor_SMD:C_0805_2012Metric"
 			(at 163.5252 73.66 0)
 			(effects
@@
 			)
 		)
-		(property "Value" "16.6nH"
+		(property "Value" "18nH"
 			(at 143.51 85.0899 0)
 			(effects
@@
 			)
 		)
-		(property "Footprint" "Inductor_SMD:L_0805_2012Metric_Pad1.05x1.20mm_HandSolder"
+		(property "Footprint" "Inductor_SMD:L_0805_2012Metric"
 			(at 142.24 83.82 0)
 			(effects
@@
 			)
 		)
-		(property "Footprint" "Capacitor_SMD:C_0805_2012Metric_Pad1.18x1.45mm_HandSolder"
+		(property "Footprint" "Capacitor_SMD:C_0603_1608Metric"
 			(at 153.3652 73.66 0)
 			(effects
@@
 			)
 		)
-		(property "Footprint" "Capacitor_SMD:C_0805_2012Metric_Pad1.18x1.45mm_HandSolder"
+		(property "Footprint" "Capacitor_SMD:C_0603_1608Metric"
 			(at 156.21 90.4748 0)
 			(effects
