File: Apollo/example_for_L1_cert_team/lokesh/lokesh_l1flc/lokesh_l1flc.kicad_sch (KiCad schematic)
At the start: 0 parts

Commit message: add teensy symbol
Parts:
- added Teensy4.1: ~, symbol mylibrary:Teensy4.1
Changed lines of the file:
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@@
 	(generator_version "9.0")
 	(paper "A4")
+	(symbol
+		(lib_id "mylibrary:Teensy4.1")
+		(at 116.84 85.09 0)
+		(unit 1)
+		(exclude_from_sim no)
+		(in_bom yes)
+		(on_board yes)
+		(dnp no)
+		(fields_autoplaced yes)
+		(property "Reference" "Teensy4.1"
+			(at 116.84 49.53 0)
+			(effects
+				(font
+					(size 1.27 1.27)
+				)
+			)
+		)
+		(property "Value" "~"
+			(at 116.84 52.07 0)
+			(effects
+				(font
+					(size 1.27 1.27)
+				)
+			)
+		)
+		(property "Footprint" ""
+			(at 116.84 85.09 0)
+			(effects
+				(font
+					(size 1.27 1.27)
+				)
+				(hide yes)
+			)
+		)
+		(property "Datasheet" ""
+			(at 116.84 85.09 0)
+			(effects
+				(font
+					(size 1.27 1.27)
+				)
+				(hide yes)
+			)
+		)
+		(property "Description" ""
+			(at 116.84 85.09 0)
+			(effects
+				(font
+					(size 1.27 1.27)
+				)
+				(hide yes)
+			)
+		)
+		(pin "5"
+		)
+		(pin "30"
+		)
+		(pin "10"
+		)
+		(pin "29"
+		)
+		(pin "G1"
+		)
+		(pin "23"
+		)
+		(pin "21"
+		)
+		(pin "6"
+		)
+		(pin "0"
+		)
+		(pin "1"
+		)
+		(pin "2"
+		)
+		(pin "12"
+		)
+		(pin "3V"
+		)
+		(pin "26"
+		)
+		(pin "4"
+		)
+		(pin "25"
+		)
+		(pin "G"
+		)
+		(pin "3"
+		)
+		(pin "24"
+		)
+		(pin "7"
+		)
+		(pin "11"
+		)
+		(pin "9"
+		)
+		(pin "28"
+		)
+		(pin "27"
+		)
+		(pin "8"
+		)
+		(pin "31"
+		)
+		(pin "32"
+		)
+		(pin "5V"
+		)
+		(pin "3V1"
+		)
+		(pin "22"
+		)
+		(pin "18"
+		)
+		(pin "39"
+		)
+		(pin "16"
+		)
+		(pin "38"
+		)
+		(pin "36"
+		)
+		(pin "35"
+		)
+		(pin "33"
+		)
+		(pin "G2"
+		)
+		(pin "17"
+		)
+		(pin "40"
+		)
+		(pin "20"
+		)
+		(pin "19"
+		)
+		(pin "15"
+		)
+		(pin "14"
+		)
+		(pin "13"
+		)
+		(pin "41"
+		)
+		(pin "37"
+		)
+		(pin "34"
+		)
+		(instances
+			(project ""
+				(path "/29675cad-ec68-4c6c-98a3-8f281860e1fa"
+					(reference "Teensy4.1")
+					(unit 1)
+				)
+			)
+		)
+	)
 	(sheet_instances
 		(path "/"
