File: Apollo/project_folder/Jack_Yeulenski_Flight_Computer/Barometer.kicad_sch (KiCad schematic)
At the start: 1 part

Commit message: Finished updating sensors and main sheet, waiting on Drew review
Connections:
- net +3V3: now also A1.6 (CS)
- net GND: now also A1.3 (RES)
- no-connect marks 0 -> 2
Other:
- note added: "Accurate within .702 ft"
- note added: "The 7-bit slave address (SAD) associated to the LPS22DF is 101110xb. The SDO/SA0 pin can be used to modify the less significant bit of the device address. If the SA0 pin is connected to the voltage supply, LSb is 1 (7-bit address 1011101b=5Dh), otherwise if the SA0 pin is connected to ground, the LSb value is 0 (7-bit address 1011100b=5Ch)"
- note added: "This has been checked over and should be good"
Changed lines of the file:
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@@
 	(generator_version "9.0")
 	(paper "A4")
+	(text "The 7-bit slave address (SAD) associated to the LPS22DF is 101110xb. The SDO/SA0 pin can be used to modify\nthe less significant bit of the device address. If the SA0 pin is connected to the voltage supply, LSb is 1 (7-bit\naddress 1011101b=5Dh), otherwise if the SA0 pin is connected to ground, the LSb value is 0 (7-bit address\n1011100b=5Ch)\n"
+		(exclude_from_sim no)
+		(at 108.204 54.356 0)
+		(effects
+			(font
+				(size 1.27 1.27)
+			)
+		)
+	)
+	(text "This has been checked over and should be good"
+		(exclude_from_sim no)
+		(at 81.026 85.852 0)
+		(effects
+			(font
+				(size 1.27 1.27)
+			)
+		)
+	)
+	(text "Accurate within .702 ft"
+		(exclude_from_sim no)
+		(at 83.566 94.488 0)
+		(effects
+			(font
+				(size 1.27 1.27)
+			)
+		)
+	)
 	(junction
 		(at 160.02 107.95)
@@
 	)
 	(junction
+		(at 160.02 105.41)
+		(diameter 0)
+		(color 0 0 0 0)
+	)
+	(junction
+		(at 160.02 72.39)
+		(diameter 0)
+		(color 0 0 0 0)
+	)
+	(junction
 		(at 160.02 82.55)
 		(diameter 0)
 		(color 0 0 0 0)
 	)
+	(no_connect
+		(at 160.02 95.25)
+	)
+	(no_connect
+		(at 119.38 95.25)
+	)
 	(wire
 		(pts
@@
 	(wire
 		(pts
+			(xy 160.02 72.39) (xy 160.02 82.55)
+		)
+		(stroke
+			(width 0)
+			(type default)
+		)
+	)
+	(wire
+		(pts
+			(xy 160.02 71.12) (xy 160.02 72.39)
+		)
+		(stroke
+			(width 0)
+			(type default)
+		)
+	)
+	(wire
+		(pts
 			(xy 160.02 82.55) (xy 160.02 85.09)
+		)
+		(stroke
+			(width 0)
+			(type default)
+		)
+	)
+	(wire
+		(pts
+			(xy 119.38 72.39) (xy 160.02 72.39)
+		)
+		(stroke
+			(width 0)
+			(type default)
+		)
+	)
+	(wire
+		(pts
+			(xy 160.02 100.33) (xy 160.02 105.41)
+		)
+		(stroke
+			(width 0)
+			(type default)
+		)
+	)
+	(wire
+		(pts
+			(xy 119.38 90.17) (xy 119.38 72.39)
 		)
 		(stroke
@@
 	(symbol
 		(lib_id "power:+3V3")
-		(at 160.02 82.55 0)
+		(at 160.02 71.12 0)
 		(unit 1)
 		(exclude_from_sim no)
@@
 		(fields_autoplaced yes)
 		(property "Reference" "#PWR04"
-			(at 160.02 86.36 0)
+			(at 160.02 74.93 0)
 			(effects
 				(font
@@
 		)
 		(property "Value" "+3V3"
-			(at 160.02 77.47 0)
+			(at 160.02 66.04 0)
 			(effects
 				(font
@@
 		)
 		(property "Footprint" ""
-			(at 160.02 82.55 0)
+			(at 160.02 71.12 0)
 			(effects
 				(font
@@
 		)
 		(property "Datasheet" ""
-			(at 160.02 82.55 0)
+			(at 160.02 71.12 0)
 			(effects
 				(font
@@
 		)
 		(property "Description" "Power symbol creates a global label with name \"+3V3\""
-			(at 160.02 82.55 0)
-			(effects
-				(font
+			(at 160.02 71.12 0)
+			(effects
+				(font

Commit message: Fixed mistakes Drew Found
Parts:
- added C4, C5: 100nF, symbol Device:C
Connections:
- net +3V3: now also C4.2, C5.1
- net GND: now also A1.5 (SDO/SA0), C4.1, C5.2
- no-connect marks 2 -> 1
Other:
- note added: "The 7-bit slave address (SAD) associated to the LPS22DF is 101110xb. The SDO/SA0 pin can be used to modify the less significant bit of the device address. If the SA0 pin is connected to the voltage supply, LSb is 1 (7-bit address 1011101b=5Dh), otherwise if the SA0 pin is connected to ground, the LSb value is 0 (7-bit address 1011100b=5Ch) currently connected to ground so address: 1011100b=5Ch"
- note removed: "The 7-bit slave address (SAD) associated to the LPS22DF is 101110xb. The SDO/SA0 pin can be used to modify the less significant bit of the device address. If the SA0 pin is connected to the voltage supply, LSb is 1 (7-bit address 1011101b=5Dh), otherwise if the SA0 pin is connected to ground, the LSb value is 0 (7-bit address 1011100b=5Ch)"
Changed lines of the file:
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@@
 	(generator_version "9.0")
 	(paper "A4")
-	(text "The 7-bit slave address (SAD) associated to the LPS22DF is 101110xb. The SDO/SA0 pin can be used to modify\nthe less significant bit of the device address. If the SA0 pin is connected to the voltage supply, LSb is 1 (7-bit\naddress 1011101b=5Dh), otherwise if the SA0 pin is connected to ground, the LSb value is 0 (7-bit address\n1011100b=5Ch)\n"
+	(text "The 7-bit slave address (SAD) associated to the LPS22DF is 101110xb. The SDO/SA0 pin can be used to modify\nthe less significant bit of the device address. If the SA0 pin is connected to the voltage supply, LSb is 1 (7-bit\naddress 1011101b=5Dh), otherwise if the SA0 pin is connected to ground, the LSb value is 0 (7-bit address\n1011100b=5Ch)\n\ncurrently connected to ground so address: 1011100b=5Ch"
 		(exclude_from_sim no)
 		(at 108.204 54.356 0)
@@
 	)
 	(junction
+		(at 160.02 77.47)
+		(diameter 0)
+		(color 0 0 0 0)
+	)
+	(junction
+		(at 148.59 72.39)
+		(diameter 0)
+		(color 0 0 0 0)
+	)
+	(junction
 		(at 160.02 72.39)
 		(diameter 0)
@@
 	)
 	(junction
+		(at 167.64 77.47)
+		(diameter 0)
+		(color 0 0 0 0)
+	)
+	(junction
+		(at 160.02 100.33)
+		(diameter 0)
+		(color 0 0 0 0)
+	)
+	(junction
 		(at 160.02 82.55)
 		(diameter 0)
 		(color 0 0 0 0)
-	)
-	(no_connect
-		(at 160.02 95.25)
 	)
 	(no_connect
@@
 	(wire
 		(pts
+			(xy 167.64 107.95) (xy 160.02 107.95)
+		)
+		(stroke
+			(width 0)
+			(type default)
+		)
+	)
+	(wire
+		(pts
+			(xy 167.64 77.47) (xy 167.64 107.95)
+		)
+		(stroke
+			(width 0)
+			(type default)
+		)
+	)
+	(wire
+		(pts
+			(xy 160.02 77.47) (xy 160.02 82.55)
+		)
+		(stroke
+			(width 0)
+			(type default)
+		)
+	)
+	(wire
+		(pts
 			(xy 160.02 105.41) (xy 160.02 107.95)
 		)
@@
 	(wire
 		(pts
-			(xy 160.02 72.39) (xy 160.02 82.55)
+			(xy 160.02 72.39) (xy 160.02 77.47)
 		)
 		(stroke
@@
 	(wire
 		(pts
+			(xy 167.64 64.77) (xy 167.64 77.47)
+		)
+		(stroke
+			(width 0)
+			(type default)
+		)
+	)
+	(wire
+		(pts
 			(xy 160.02 82.55) (xy 160.02 85.09)
 		)
@@
 	(wire
 		(pts
-			(xy 119.38 72.39) (xy 160.02 72.39)
+			(xy 160.02 95.25) (xy 160.02 100.33)
+		)
+		(stroke
+			(width 0)
+			(type default)
+		)
+	)
+	(wire
+		(pts
+			(xy 148.59 64.77) (xy 167.64 64.77)
+		)
+		(stroke
+			(width 0)
+			(type default)
+		)
+	)
+	(wire
+		(pts
+			(xy 119.38 72.39) (xy 148.59 72.39)
+		)
+		(stroke
+			(width 0)
+			(type default)
+		)
+	)
+	(wire
+		(pts
+			(xy 148.59 72.39) (xy 160.02 72.39)
 		)
 		(stroke
@@
 					(unit 1)
 				)
+			)
+		)
+	)
+	(symbol
+		(lib_id "Device:C")
+		(at 148.59 68.58 180)
+		(unit 1)
+		(exclude_from_sim no)
+		(in_bom yes)
+		(on_board yes)
+		(dnp no)
+		(fields_autoplaced yes)
+		(property "Reference" "C5"
+			(at 152.4 67.3099 0)
+			(effects
+				(font
+					(size 1.27 1.27)
+				)
+				(justify right)
+			)
+		)
+		(property "Value" "100nF"
+			(at 152.4 69.8499 0)
+			(effects
+				(font
+					(size 1.27 1.27)
+				)
+				(justify right)
+			)
+		)
+		(property "Footprint" ""
+			(at 147.6248 64.77 0)
+			(effects
+				(font
+					(size 1.27 1.27)
+				)
+				(hide yes)
+			)
+		)
+		(property "Datasheet" "~"
+			(at 148.59 68.58 0)
+			(effects
+				(font
+					(size 1.27 1.27)
+				)
+				(hide yes)
+			)
+		)
+		(property "Description" "Unpolarized capacitor"
+			(at 148.59 68.58 0)
+			(effects
+				(font
+					(size 1.27 1.27)
+				)
+				(hide yes)
+			)
+		)
+		(pin "2"
+		)
+		(pin "1"
+		)
+		(instances
+			(project ""
+				(path "/0e457dee-ab7a-4947-acac-685db257dbd9/90dbbe8f-d831-457a-80e5-86785cc75e56"
+					(reference "C5")
+					(unit 1)
+				)
+			)
+		)
+	)
+	(symbol
+		(lib_id "Device:C")
+		(at 163.83 77.47 270)
+		(unit 1)
+		(exclude_from_sim no)
+		(in_bom yes)
+		(on_board yes)
+		(dnp no)
+		(fields_autoplaced yes)
+		(property "Reference" "C4"
+			(at 163.83 69.85 90)
+			(effects
+				(font
+					(size 1.27 1.27)
+				)
+			)
+		)
+		(property "Value" "100nF"
+			(at 163.83 72.39 90)
+			(effects
+				(font
+					(size 1.27 1.27)
+				)
+			)
+		)
+		(property "Footprint" ""
+			(at 160.02 78.4352 0)
+			(effects
+				(font
+					(size 1.27 1.27)
+				)
+				(hide yes)
+			)
+		)
+		(property "Datasheet" "~"
+			(at 163.83 77.47 0)
+			(effects
+				(font
+					(size 1.27 1.27)
+				)
+				(hide yes)
+			)
+		)
+		(property "Description" "Unpolarized capacitor"
+			(at 163.83 77.47 0)
+			(effects
+				(font
+					(size 1.27 1.27)
+				)
+				(hide yes)
+			)
+		)
+		(pin "2"
+		)
+		(pin "1"
+		)
+		(instances
+			(project ""
+				(path "/0e457dee-ab7a-4947-acac-685db257dbd9/90dbbe8f-d831-457a-80e5-86785cc75e56"
+					(reference "C4")
+					(unit 1)
+				)

Commit message: Added footprints to all components and started PCB
Parts:
- C4, C5: footprint (none) -> Capacitor_SMD:C_0805_2012Metric
Changed lines of the file:
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@@
 			)
 		)
-		(property "Footprint" ""
+		(property "Footprint" "Capacitor_SMD:C_0805_2012Metric"
 			(at 147.6248 64.77 0)
 			(effects
@@
 			)
 		)
-		(property "Footprint" ""
+		(property "Footprint" "Capacitor_SMD:C_0805_2012Metric"
 			(at 160.02 78.4352 0)
 			(effects

Commit message: designed PCB
Parts:
- A1: footprint LPS22DFTR:XDCR_LPS22DFTR -> Package_LGA:ST_HLGA-10_2x2mm_P0.5mm_LayoutBorder3x2y
- renumbered C5 to C1, C4 to C2
Changed lines of the file:
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@@
 			)
 		)
-		(property "Footprint" "LPS22DFTR:XDCR_LPS22DFTR"
+		(property "Footprint" "Package_LGA:ST_HLGA-10_2x2mm_P0.5mm_LayoutBorder3x2y"
 			(at 139.7 95.25 0)
 			(effects
@@
 		(dnp no)
 		(fields_autoplaced yes)
-		(property "Reference" "#PWR03"
+		(property "Reference" "#PWR016"
 			(at 160.02 114.3 0)
 			(effects
@@
 			(project ""
 				(path "/0e457dee-ab7a-4947-acac-685db257dbd9/90dbbe8f-d831-457a-80e5-86785cc75e56"
-					(reference "#PWR03")
+					(reference "#PWR016")
 					(unit 1)
 				)
@@
 		(dnp no)
 		(fields_autoplaced yes)
-		(property "Reference" "#PWR04"
+		(property "Reference" "#PWR015"
 			(at 160.02 74.93 0)
 			(effects
@@
 			(project ""
 				(path "/0e457dee-ab7a-4947-acac-685db257dbd9/90dbbe8f-d831-457a-80e5-86785cc75e56"
-					(reference "#PWR04")
+					(reference "#PWR015")
 					(unit 1)
 				)
@@
 		(dnp no)
 		(fields_autoplaced yes)
-		(property "Reference" "C5"
+		(property "Reference" "C1"
 			(at 152.4 67.3099 0)
 			(effects
@@
 			(project ""
 				(path "/0e457dee-ab7a-4947-acac-685db257dbd9/90dbbe8f-d831-457a-80e5-86785cc75e56"
-					(reference "C5")
+					(reference "C1")
 					(unit 1)
 				)
@@
 		(dnp no)
 		(fields_autoplaced yes)
-		(property "Reference" "C4"
+		(property "Reference" "C2"
 			(at 163.83 69.85 90)
 			(effects
@@
 			(project ""
 				(path "/0e457dee-ab7a-4947-acac-685db257dbd9/90dbbe8f-d831-457a-80e5-86785cc75e56"
-					(reference "C4")
-					(unit 1)
-				)
+					(reference "C2")
+					(unit 1)
+				)
