File: Apollo/project_folder/Jack_Yeulenski_Flight_Computer/Jack_Yeulenski_Flight_Computer.kicad_sch (KiCad schematic)
At the start: 0 parts

Commit message: idk, I dont know
Parts:
- added Teensy4.1: ~, my footprint library:teensy, symbol New_Library:Teensy4.1
Connections:
- new net +3.3V: Teensy4.1.3V1 (3.3V)
- new net GND: Teensy4.1.G1 (GND)
- new net SCL: Teensy4.1.19 (SCL)
- new net SDA: Teensy4.1.18 (SDA)

Commit message: Placed sensors
Parts:
- added J1: Conn_01x04, symbol Connector_Generic:Conn_01x04
- added U1: BNO055, BNO055:LGA28R50P4X10_380X520X100, symbol SRAD:BNO055
Other:
- added sheet Barometer (Barometer.kicad_sch)
- moved on the sheet: Teensy4.1

Commit message: Just moved stuff around (hierarchal sheets)
Parts:
- removed U1: BNO055, BNO055:LGA28R50P4X10_380X520X100, symbol SRAD:BNO055
Other:
- added sheet IMU (IMU.kicad_sch)
Changed lines of the file:
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@@
-	)
-	(symbol
-		(lib_id "SRAD:BNO055")
-		(at 215.9 113.03 0)
-		(unit 1)
-		(exclude_from_sim no)
-		(in_bom yes)
-		(on_board yes)
-		(dnp no)
-		(fields_autoplaced yes)
-		(property "Reference" "U1"
-			(at 215.9 92.71 0)
-			(effects
-				(font
-					(size 1.27 1.27)
-				)
-			)
-		)
-		(property "Value" "BNO055"
-			(at 215.9 95.25 0)
-			(effects
-				(font
-					(size 1.27 1.27)
-				)
-			)
-		)
-		(property "Footprint" "BNO055:LGA28R50P4X10_380X520X100"
-			(at 215.9 113.03 0)
-			(effects
-				(font
-					(size 1.27 1.27)
-				)
-				(justify bottom)
-				(hide yes)
-			)
-		)
-		(property "Datasheet" ""
-			(at 215.9 113.03 0)
-			(effects
-				(font
-					(size 1.27 1.27)
-				)
-				(hide yes)
-			)
-		)
-		(property "Description" ""
-			(at 215.9 113.03 0)
-			(effects
-				(font
-					(size 1.27 1.27)
-				)
-				(hide yes)
-			)
-		)
-		(property "MANUFACTURER" "BOSCH"
-			(at 215.9 113.03 0)
-			(effects
-				(font
-					(size 1.27 1.27)
-				)
-				(justify bottom)
-				(hide yes)
-			)
-		)
-		(pin "17"
-		)
-		(pin "27"
-		)
-		(pin "4"
-		)
-		(pin "28"
-		)
-		(pin "5"
-		)
-		(pin "20"
-		)
-		(pin "19"
-		)
-		(pin "11"
-		)
-		(pin "18"
-		)
-		(pin "6"
-		)
-		(pin "9"
-		)
-		(pin "3"
-		)
-		(pin "26"
-		)
-		(pin "14"
-		)
-		(pin "10"
-		)
-		(pin "15"
-		)
-		(pin "16"
-		)
-		(pin "2"
-		)
-		(pin "25"
-		)
-		(instances
-			(project ""
-				(path "/0e457dee-ab7a-4947-acac-685db257dbd9"
-					(reference "U1")
-					(unit 1)
-				)
-			)
-		)
 	)
 	(symbol
@@
 	)
 	(sheet
-		(at 181.61 24.13)
-		(size 66.04 44.45)
+		(at 27.94 97.79)
+		(size 43.18 40.64)
 		(exclude_from_sim no)
 		(in_bom yes)
@@
 		)
 		(property "Sheetname" "Barometer"
-			(at 181.61 23.4184 0)
+			(at 27.94 97.0784 0)
 			(effects
 				(font
@@
 		)
 		(property "Sheetfile" "Barometer.kicad_sch"
-			(at 181.61 69.1646 0)
+			(at 27.94 139.0146 0)
 			(effects
 				(font
@@
 				)
 			)
+		)
+	)
+	(sheet
+		(at 27.94 146.05)
+		(size 43.18 39.37)
+		(exclude_from_sim no)
+		(in_bom yes)
+		(on_board yes)
+		(dnp no)
+		(fields_autoplaced yes)
+		(stroke
+			(width 0.1524)
+			(type solid)
+		)
+		(fill
+			(color 0 0 0 0.0000)
+		)
+		(property "Sheetname" "IMU"
+			(at 27.94 145.3384 0)
+			(effects
+				(font
+					(size 1.27 1.27)
+				)
+				(justify left bottom)
+			)
+		)
+		(property "Sheetfile" "IMU.kicad_sch"
+			(at 27.94 186.0046 0)
+			(effects
+				(font
+					(size 1.27 1.27)
+				)
+				(justify left top)
+			)
+		)
+		(instances
+			(project "Jack_Yeulenski_Flight_Computer"
+				(path "/0e457dee-ab7a-4947-acac-685db257dbd9"
+					(page "3")
+				)
+			)

Commit message: Finished updating sensors and main sheet, waiting on Drew review
Parts:
- added BZ1: Buzzer, symbol Device:Buzzer
- added D1, D2, D3: LED, symbol Device:LED
- added J2: UART Radio Connector, symbol Connector_Generic:Conn_01x04
- added J3: BAT, symbol Connector_Generic:Conn_01x02
- added J4: SW, symbol Connector_Generic:Conn_01x02
- added R1, R2, R3: 560, symbol Device:R
- added R4: 78k7, symbol Device:R
- added R6: 100k, symbol Device:R
- added Rpull1, Rpull2: 5k1, symbol Device:R
- J1: value Conn_01x04 -> I2C GPS Connector
Connections:
- net GND: now also J1.4 (Pin_4), BZ1.2 (-), J2.4 (Pin_4), J3.2 (Pin_2), R1.2, R2.2, R3.2, R6.1
- net SCL: now also J1.3 (Pin_3), Rpull1.1
- net SDA: now also J1.2 (Pin_2), Rpull2.1
- net RX: now reaches Teensy4.1.0 (RX1)
- net RX: now also J2.3 (Pin_3)
- net TX: now reaches Teensy4.1.1 (TX1)
- net TX: now also J2.2 (Pin_2)
- net at Teensy4.1.14 (A0): now also R4.1, R6.2
- net at Teensy4.1.31 (GPIO): now also D3.2 (A)
- net at Teensy4.1.32 (GPIO): now also D2.2 (A)
- net at Teensy4.1.33 (PWM): now also BZ1.1 (+)
- net at Teensy4.1.5V (VIN): now also J4.1 (Pin_1)
- net +3V3: now reaches J1.1 (Pin_1)
- net +3V3: now also D1.2 (A), J2.1 (Pin_1), Rpull1.2, Rpull2.2
- new net: D2.1 (K), R2.1
- new net: J3.1 (Pin_1), J4.2 (Pin_2), R4.2
- new net: D1.1 (K), R1.1
- new net: D3.1 (K), R3.1
Other:
- note added: "Voltage divider info: Ratio Vin/Vo = 2.422 5.5Vin = 3.07Vo"
- moved on the sheet: J1

Commit message: Fixed mistakes Drew Found
Connections:
- net +3.3V is gone; now on net +3V3: Teensy4.1.3V1 (3.3V)
Other:
- note added: "Voltage divider info: Ratio Vin/Vo = 1.79 5.5Vin = 3.07Vo"
- note removed: "Voltage divider info: Ratio Vin/Vo = 2.422 5.5Vin = 3.07Vo"

Commit message: Added footprints to all components and started PCB
Parts:
- BZ1: footprint (none) -> adaafruitBuzzer:Adafruit_Buzzer
- D1, D2, D3: footprint (none) -> LED_SMD:LED_0805_2012Metric
- J1, J2: footprint (none) -> Connector_JST:JST_XH_S4B-XH-A_1x04_P2.50mm_Horizontal
- J3, J4: footprint (none) -> Connector_JST:JST_XH_S2B-XH-A_1x02_P2.50mm_Horizontal
- R1, R2, R3: footprint (none) -> Resistor_SMD:R_0805_2012Metric
- R4, R6: footprint (none) -> Resistor_SMD:R_0201_0603Metric
- Rpull1, Rpull2: footprint (none) -> Resistor_SMD:R_01005_0402Metric
Changed lines of the file:
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@@
 			)
 		)
-		(property "Footprint" ""
+		(property "Footprint" "Resistor_SMD:R_0805_2012Metric"
 			(at 90.932 128.27 90)
 			(effects
@@
 			)
 		)
-		(property "Footprint" ""
+		(property "Footprint" "Resistor_SMD:R_01005_0402Metric"
 			(at 129.54 65.278 90)
 			(effects
@@
 			)
 		)
-		(property "Footprint" ""
+		(property "Footprint" "adaafruitBuzzer:Adafruit_Buzzer"
 			(at 118.745 104.14 90)
 			(effects
@@
 			)
 		)
-		(property "Footprint" ""
+		(property "Footprint" "Resistor_SMD:R_0201_0603Metric"
 			(at 132.08 85.598 90)
 			(effects
@@
 			)
 		)
-		(property "Footprint" ""
+		(property "Footprint" "Resistor_SMD:R_0201_0603Metric"
 			(at 139.7 85.598 90)
 			(effects
@@
 			)
 		)
-		(property "Footprint" ""
+		(property "Footprint" "Resistor_SMD:R_0805_2012Metric"
 			(at 101.092 128.27 90)
 			(effects
@@
 			)
 		)
-		(property "Footprint" ""
+		(property "Footprint" "Connector_JST:JST_XH_S2B-XH-A_1x02_P2.50mm_Horizontal"
 			(at 148.59 78.74 0)
 			(effects
@@
 			)
 		)
-		(property "Footprint" ""
+		(property "Footprint" "LED_SMD:LED_0805_2012Metric"
 			(at 92.71 120.65 0)
 			(effects
@@
 			)
 		)
-		(property "Footprint" ""
+		(property "Footprint" "Connector_JST:JST_XH_S4B-XH-A_1x04_P2.50mm_Horizontal"
 			(at 148.59 134.62 0)
 			(effects
@@
 			)
 		)
-		(property "Footprint" ""
+		(property "Footprint" "Connector_JST:JST_XH_S4B-XH-A_1x04_P2.50mm_Horizontal"
 			(at 148.59 111.76 0)
 			(effects
@@
 			)
 		)
-		(property "Footprint" ""
+		(property "Footprint" "Connector_JST:JST_XH_S2B-XH-A_1x02_P2.50mm_Horizontal"
 			(at 148.59 91.44 0)
 			(effects
@@
 			)
 		)
-		(property "Footprint" ""
+		(property "Footprint" "LED_SMD:LED_0805_2012Metric"
 			(at 82.55 120.65 0)
 			(effects
@@
 			)
 		)
-		(property "Footprint" ""
+		(property "Footprint" "Resistor_SMD:R_0805_2012Metric"
 			(at 80.772 128.27 90)
 			(effects
@@
 			)
 		)
-		(property "Footprint" ""
+		(property "Footprint" "Resistor_SMD:R_01005_0402Metric"
 			(at 129.54 67.818 90)
 			(effects
@@
 			)
 		)
-		(property "Footprint" ""
+		(property "Footprint" "LED_SMD:LED_0805_2012Metric"
 			(at 102.87 120.65 0)
 			(effects

Commit message: designed PCB
Parts:
- renumbered D3 to D1, D1 to D3, J4 to J1, J3 to J2, J2 to J3, J1 to J4, R3 to R1, R1 to R3, R6 to R4, R4 to R5
Connections:
- net +3V3: now also Teensy4.1.3V (3.3V)
Changed lines of the file:
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@@
 		(dnp no)
 		(fields_autoplaced yes)
-		(property "Reference" "#PWR020"
+		(property "Reference" "#PWR01"
 			(at 82.55 138.43 0)
 			(effects
@@
 			(project "Jack_Yeulenski_Flight_Computer"
 				(path "/0e457dee-ab7a-4947-acac-685db257dbd9"
-					(reference "#PWR020")
+					(reference "#PWR01")
 					(unit 1)
 				)
@@
 		(dnp no)
 		(fields_autoplaced yes)
-		(property "Reference" "#PWR016"
+		(property "Reference" "#PWR04"
 			(at 102.87 138.43 0)
 			(effects
@@
 			(project ""
 				(path "/0e457dee-ab7a-4947-acac-685db257dbd9"
-					(reference "#PWR016")
+					(reference "#PWR04")
+					(unit 1)
+				)
+			)
+		)
+	)
+	(symbol
+		(lib_id "power:+3V3")
+		(at 91.44 81.28 90)
+		(unit 1)
+		(exclude_from_sim no)
+		(in_bom yes)
+		(on_board yes)
+		(dnp no)
+		(fields_autoplaced yes)
+		(property "Reference" "#PWR021"
+			(at 95.25 81.28 0)
+			(effects
+				(font
+					(size 1.27 1.27)
+				)
+				(hide yes)
+			)
+		)
+		(property "Value" "+3V3"
+			(at 87.63 81.2799 90)
+			(effects
+				(font
+					(size 1.27 1.27)
+				)
+				(justify left)
+			)
+		)
+		(property "Footprint" ""
+			(at 91.44 81.28 0)
+			(effects
+				(font
+					(size 1.27 1.27)
+				)
+				(hide yes)
+			)
+		)
+		(property "Datasheet" ""
+			(at 91.44 81.28 0)
+			(effects
+				(font
+					(size 1.27 1.27)
+				)
+				(hide yes)
+			)
+		)
+		(property "Description" "Power symbol creates a global label with name \"+3V3\""
+			(at 91.44 81.28 0)
+			(effects
+				(font
+					(size 1.27 1.27)
+				)
+				(hide yes)
+			)
+		)
+		(pin "1"
+		)
+		(instances
+			(project ""
+				(path "/0e457dee-ab7a-4947-acac-685db257dbd9"
+					(reference "#PWR021")
 					(unit 1)
 				)
@@
 		(dnp no)
 		(fields_autoplaced yes)
-		(property "Reference" "#PWR013"
+		(property "Reference" "#PWR010"
 			(at 143.51 100.33 0)
 			(effects
@@
 			(project ""
 				(path "/0e457dee-ab7a-4947-acac-685db257dbd9"
-					(reference "#PWR013")
+					(reference "#PWR010")
 					(unit 1)
 				)
@@
 		(dnp no)
 		(fields_autoplaced yes)
-		(property "Reference" "#PWR018"
+		(property "Reference" "#PWR02"
 			(at 92.71 138.43 0)
 			(effects
@@
 			(project "Jack_Yeulenski_Flight_Computer"
 				(path "/0e457dee-ab7a-4947-acac-685db257dbd9"
-					(reference "#PWR018")
+					(reference "#PWR02")
 					(unit 1)
 				)
@@
 		(dnp no)
 		(fields_autoplaced yes)
-		(property "Reference" "#PWR015"
+		(property "Reference" "#PWR03"
 			(at 102.87 120.65 0)
 			(effects
@@
 			(project ""
 				(path "/0e457dee-ab7a-4947-acac-685db257dbd9"
-					(reference "#PWR015")
+					(reference "#PWR03")
 					(unit 1)
 				)
@@
 		(dnp no)
 		(fields_autoplaced yes)
-		(property "Reference" "#PWR05"
+		(property "Reference" "#PWR09"
 			(at 135.89 67.31 0)
 			(effects
@@
 			(project ""
 				(path "/0e457dee-ab7a-4947-acac-685db257dbd9"
-					(reference "#PWR05")
+					(reference "#PWR09")
 					(unit 1)
 				)
@@
 		(dnp no)
 		(fields_autoplaced yes)
-		(property "Reference" "#PWR01"
+		(property "Reference" "#PWR05"
 			(at 123.19 48.26 0)
 			(effects
@@
 			(project ""
 				(path "/0e457dee-ab7a-4947-acac-685db257dbd9"
-					(reference "#PWR01")
+					(reference "#PWR05")
 					(unit 1)
 				)
@@
 		(dnp no)
 		(fields_autoplaced yes)
-		(property "Reference" "#PWR09"
+		(property "Reference" "#PWR014"
 			(at 143.51 146.05 0)
 			(effects
@@
 			(project ""
 				(path "/0e457dee-ab7a-4947-acac-685db257dbd9"
-					(reference "#PWR09")
+					(reference "#PWR014")
 					(unit 1)
 				)
@@
 		(dnp no)
 		(fields_autoplaced yes)
-		(property "Reference" "R6"
+		(property "Reference" "R4"
 			(at 132.08 77.47 90)
 			(effects
@@
 			(project ""
 				(path "/0e457dee-ab7a-4947-acac-685db257dbd9"
-					(reference "R6")
+					(reference "R4")
 					(unit 1)
 				)
@@
 		(dnp no)
 		(fields_autoplaced yes)
-		(property "Reference" "R4"
+		(property "Reference" "R5"
 			(at 139.7 77.47 90)
 			(effects
@@
 			(project ""
 				(path "/0e457dee-ab7a-4947-acac-685db257dbd9"
-					(reference "R4")
+					(reference "R5")
 					(unit 1)
 				)
@@
 		(dnp no)
 		(fields_autoplaced yes)
-		(property "Reference" "#PWR02"
+		(property "Reference" "#PWR06"
 			(at 113.03 50.8 0)
 			(effects
@@
 			(project ""
 				(path "/0e457dee-ab7a-4947-acac-685db257dbd9"
-					(reference "#PWR02")
+					(reference "#PWR06")
 					(unit 1)
 				)
@@
 		(dnp no)
 		(fields_autoplaced yes)
-		(property "Reference" "#PWR014"
+		(property "Reference" "#PWR07"
 			(at 116.84 115.57 0)
 			(effects
@@
 			(project ""
 				(path "/0e457dee-ab7a-4947-acac-685db257dbd9"
-					(reference "#PWR014")
+					(reference "#PWR07")
 					(unit 1)
 				)
@@
 		(dnp no)
 		(fields_autoplaced yes)
-		(property "Reference" "R1"
+		(property "Reference" "R3"
 			(at 105.41 126.9999 0)
 			(effects
@@
 			(project ""
 				(path "/0e457dee-ab7a-4947-acac-685db257dbd9"
-					(reference "R1")
+					(reference "R3")
 					(unit 1)
 				)
@@
 		(dnp no)
 		(fields_autoplaced yes)
-		(property "Reference" "J4"
+		(property "Reference" "J1"
 			(at 151.13 78.7399 0)
 			(effects
@@
 			(project "Jack_Yeulenski_Flight_Computer"
 				(path "/0e457dee-ab7a-4947-acac-685db257dbd9"
-					(reference "J4")
+					(reference "J1")
 					(unit 1)
 				)
@@
 		(dnp no)
 		(fields_autoplaced yes)
-		(property "Reference" "J1"
+		(property "Reference" "J4"
 			(at 151.13 134.6199 0)
 			(effects
@@
 			(project ""
 				(path "/0e457dee-ab7a-4947-acac-685db257dbd9"
-					(reference "J1")
+					(reference "J4")
 					(unit 1)
 				)
@@
 		(dnp no)
 		(fields_autoplaced yes)
-		(property "Reference" "J2"
+		(property "Reference" "J3"
 			(at 151.13 111.7599 0)
 			(effects
@@
 			(project "Jack_Yeulenski_Flight_Computer"
 				(path "/0e457dee-ab7a-4947-acac-685db257dbd9"
-					(reference "J2")
+					(reference "J3")
 					(unit 1)
 				)
@@
 		(dnp no)
 		(fields_autoplaced yes)
-		(property "Reference" "J3"
+		(property "Reference" "J2"
 			(at 151.13 91.4399 0)
 			(effects
@@
 			(project ""
 				(path "/0e457dee-ab7a-4947-acac-685db257dbd9"
-					(reference "J3")
+					(reference "J2")
 					(unit 1)
 				)
@@
 		(dnp no)
 		(fields_autoplaced yes)
-		(property "Reference" "D3"
+		(property "Reference" "D1"
 			(at 86.36 120.9674 90)
 			(effects
@@
 			(project "Jack_Yeulenski_Flight_Computer"
 				(path "/0e457dee-ab7a-4947-acac-685db257dbd9"
-					(reference "D3")
+					(reference "D1")
 					(unit 1)
 				)
@@
 		(dnp no)
 		(fields_autoplaced yes)
-		(property "Reference" "R3"
+		(property "Reference" "R1"
 			(at 85.09 126.9999 0)
 			(effects
@@
 			(project "Jack_Yeulenski_Flight_Computer"
 				(path "/0e457dee-ab7a-4947-acac-685db257dbd9"
-					(reference "R3")
+					(reference "R1")
 					(unit 1)
 				)
@@
 		(dnp no)
 		(fields_autoplaced yes)
-		(property "Reference" "D1"
+		(property "Reference" "D3"
 			(at 106.68 120.9674 90)
 			(effects
@@
 			(project ""
 				(path "/0e457dee-ab7a-4947-acac-685db257dbd9"
-					(reference "D1")
+					(reference "D3")
 					(unit 1)
 				)
@@
 		(dnp no)
 		(fields_autoplaced yes)
-		(property "Reference" "#PWR010"
+		(property "Reference" "#PWR013"
 			(at 143.51 135.89 0)
 			(effects
@@
 			(project ""
 				(path "/0e457dee-ab7a-4947-acac-685db257dbd9"
-					(reference "#PWR010")
+					(reference "#PWR013")
 					(unit 1)
 				)
@@
 		(dnp no)
 		(fields_autoplaced yes)
-		(property "Reference" "#PWR017"
+		(property "Reference" "#PWR08"
 			(at 128.27 90.17 0)
 			(effects
@@
 			(project ""
 				(path "/0e457dee-ab7a-4947-acac-685db257dbd9"
-					(reference "#PWR017")
-					(unit 1)
-				)
+					(reference "#PWR08")
+					(unit 1)
+				)

Commit message: Updated PCB according to Drew's feedback
Parts:
- added H1, H2, H3, H4: MountingHole, MountingHole:MountingHole_3.2mm_M3, symbol Mechanical:MountingHole
- R1, R3: footprint Resistor_SMD:R_0805_2012Metric -> Resistor_SMD:R_0603_1608Metric
- R2: footprint Resistor_SMD:R_0805_2012Metric -> Diode_SMD:D_0603_1608Metric
- R4, R5: footprint Resistor_SMD:R_0201_0603Metric -> Resistor_SMD:R_0603_1608Metric
- Rpull1, Rpull2: footprint Resistor_SMD:R_01005_0402Metric -> Resistor_SMD:R_0402_1005Metric
