File: Apollo/project_folder/Jack_Yeulenski_Flight_Computer/IMU.kicad_sch (KiCad schematic)
At the start: 1 part, among them U2 BNO055

Commit message: Finished updating sensors and main sheet, waiting on Drew review
Parts:
- added C1: 1uF, symbol Device:C
- added C2: 100nF, symbol Device:C
- added C3: 120nF, symbol Device:C
Connections:
- net +3V3: now reaches U2.11 (NRESET)
- net +3V3: now also U2.28 (VDDIO), U2.3 (VDD), U2.4 (NBOOT_LOAD_PIN), C2.1, C3.1
- net GND: now reaches U2.18 (COM2)
- net GND: now also U2.2 (GND), U2.25 (GNDIO), U2.5 (PS1), U2.6 (PS0), C1.1, C2.2, C3.2
- net SCL: now reaches U2.19 (COM1)
- net SDA: now reaches U2.20 (COM0)
- net at U2.9 (CAP): now also C1.2
- no-connect marks 0 -> 7
Other:
- note added: "Default I2C address: 0100101b (0x29) Alternate I2C address: 0101000b (0x28) COM3 is used to switch adress"
- note added: "Should be done, went through all pins on datasheet"

Commit message: Fixed mistakes Drew Found
Connections:
- net +3V3: now also U2.17 (COM3)
- no-connect marks 7 -> 6
Other:
- note added: "Default I2C address (COM3 HIGH): 0100101b (0x29) Alternate I2C address (COM3 LOW): 0101000b (0x28) COM3 is used to switch adress"
- note removed: "Default I2C address: 0100101b (0x29) Alternate I2C address: 0101000b (0x28) COM3 is used to switch adress"
Changed lines of the file:
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@@
 	(generator_version "9.0")
 	(paper "A4")
-	(text "Default I2C address: 0100101b (0x29)\nAlternate I2C address: 0101000b (0x28)\nCOM3 is used to switch adress"
+	(text "Default I2C address (COM3 HIGH): 0100101b (0x29)\nAlternate I2C address (COM3 LOW): 0101000b (0x28)\nCOM3 is used to switch adress"
 		(exclude_from_sim no)
 		(at 79.502 61.214 0)
@@
 		(diameter 0)
 		(color 0 0 0 0)
-	)
-	(no_connect
-		(at 101.6 100.33)
 	)
 	(no_connect
@@
 					(unit 1)
 				)
+			)
+		)
+	)
+	(symbol
+		(lib_id "power:+3V3")
+		(at 101.6 100.33 90)
+		(unit 1)
+		(exclude_from_sim no)
+		(in_bom yes)
+		(on_board yes)
+		(dnp no)
+		(fields_autoplaced yes)
+		(property "Reference" "#PWR019"
+			(at 105.41 100.33 0)
+			(effects
+				(font
+					(size 1.27 1.27)
+				)
+				(hide yes)
+			)
+		)
+		(property "Value" "+3V3"
+			(at 97.79 100.3299 90)
+			(effects
+				(font
+					(size 1.27 1.27)
+				)
+				(justify left)
+			)
+		)
+		(property "Footprint" ""
+			(at 101.6 100.33 0)
+			(effects
+				(font
+					(size 1.27 1.27)
+				)
+				(hide yes)
+			)
+		)
+		(property "Datasheet" ""
+			(at 101.6 100.33 0)
+			(effects
+				(font
+					(size 1.27 1.27)
+				)
+				(hide yes)
+			)
+		)
+		(property "Description" "Power symbol creates a global label with name \"+3V3\""
+			(at 101.6 100.33 0)
+			(effects
+				(font
+					(size 1.27 1.27)
+				)
+				(hide yes)
+			)
+		)
+		(pin "1"
+		)
+		(instances
+			(project ""
+				(path "/0e457dee-ab7a-4947-acac-685db257dbd9/ac8308a5-c176-4748-bfbf-484ade2f530b"
+					(reference "#PWR019")
+					(unit 1)
+				)

Commit message: Added footprints to all components and started PCB
Parts:
- C1, C2: footprint (none) -> Capacitor_SMD:C_0805_2012Metric
- C3: value 120nF -> 100nF; footprint (none) -> Capacitor_SMD:C_0805_2012Metric
Changed lines of the file:
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@@
 			)
 		)
-		(property "Footprint" ""
+		(property "Footprint" "Capacitor_SMD:C_0805_2012Metric"
 			(at 100.6348 105.41 0)
 			(effects
@@
 			)
 		)
-		(property "Footprint" ""
+		(property "Footprint" "Capacitor_SMD:C_0805_2012Metric"
 			(at 147.0152 85.09 0)
 			(effects
@@
 			)
 		)
-		(property "Value" "120nF"
+		(property "Value" "100nF"
 			(at 158.75 82.5499 0)
 			(effects
@@
 			)
 		)
-		(property "Footprint" ""
+		(property "Footprint" "Capacitor_SMD:C_0805_2012Metric"
 			(at 155.9052 85.09 0)
 			(effects

Commit message: designed PCB
Parts:
- U1: renamed from U2; footprint BNO055:LGA28R50P4X10_380X520X100 -> Package_LGA:LGA-28_5.2x3.8mm_P0.5mm
- renumbered C1 to C3, C2 to C4, C3 to C5
Changed lines of the file:
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@@
 		(dnp no)
 		(fields_autoplaced yes)
-		(property "Reference" "#PWR06"
+		(property "Reference" "#PWR020"
 			(at 162.56 77.47 0)
 			(effects
@@
 			(project ""
 				(path "/0e457dee-ab7a-4947-acac-685db257dbd9/ac8308a5-c176-4748-bfbf-484ade2f530b"
-					(reference "#PWR06")
+					(reference "#PWR020")
 					(unit 1)
 				)
@@
 		(dnp no)
 		(fields_autoplaced yes)
-		(property "Reference" "C1"
+		(property "Reference" "C3"
 			(at 105.41 107.9499 0)
 			(effects
@@
 			(project ""
 				(path "/0e457dee-ab7a-4947-acac-685db257dbd9/ac8308a5-c176-4748-bfbf-484ade2f530b"
-					(reference "C1")
+					(reference "C3")
 					(unit 1)
 				)
@@
 		(dnp no)
 		(fields_autoplaced yes)
-		(property "Reference" "#PWR019"
+		(property "Reference" "#PWR018"
 			(at 105.41 100.33 0)
 			(effects
@@
 			(project ""
 				(path "/0e457dee-ab7a-4947-acac-685db257dbd9/ac8308a5-c176-4748-bfbf-484ade2f530b"
-					(reference "#PWR019")
+					(reference "#PWR018")
 					(unit 1)
 				)
@@
 		(dnp no)
 		(fields_autoplaced yes)
-		(property "Reference" "C2"
+		(property "Reference" "C4"
 			(at 149.86 80.0099 0)
 			(effects
@@
 			(project ""
 				(path "/0e457dee-ab7a-4947-acac-685db257dbd9/ac8308a5-c176-4748-bfbf-484ade2f530b"
-					(reference "C2")
+					(reference "C4")
 					(unit 1)
 				)
@@
 		(dnp no)
 		(fields_autoplaced yes)
-		(property "Reference" "U2"
+		(property "Reference" "U1"
 			(at 121.92 69.85 0)
 			(effects
@@
 			)
 		)
-		(property "Footprint" "BNO055:LGA28R50P4X10_380X520X100"
+		(property "Footprint" "Package_LGA:LGA-28_5.2x3.8mm_P0.5mm"
 			(at 121.92 90.17 0)
 			(effects
@@
 			(project "Jack_Yeulenski_Flight_Computer"
 				(path "/0e457dee-ab7a-4947-acac-685db257dbd9/ac8308a5-c176-4748-bfbf-484ade2f530b"
-					(reference "U2")
+					(reference "U1")
 					(unit 1)
 				)
@@
 		(dnp no)
 		(fields_autoplaced yes)
-		(property "Reference" "#PWR07"
+		(property "Reference" "#PWR019"
 			(at 157.48 113.03 0)
 			(effects
@@
 			(project ""
 				(path "/0e457dee-ab7a-4947-acac-685db257dbd9/ac8308a5-c176-4748-bfbf-484ade2f530b"
-					(reference "#PWR07")
+					(reference "#PWR019")
 					(unit 1)
 				)
@@
 		(on_board yes)
 		(dnp no)
-		(property "Reference" "#PWR08"
+		(property "Reference" "#PWR017"
 			(at 105.41 85.09 0)
 			(effects
@@
 			(project ""
 				(path "/0e457dee-ab7a-4947-acac-685db257dbd9/ac8308a5-c176-4748-bfbf-484ade2f530b"
-					(reference "#PWR08")
+					(reference "#PWR017")
 					(unit 1)
 				)
@@
 		(dnp no)
 		(fields_autoplaced yes)
-		(property "Reference" "C3"
+		(property "Reference" "C5"
 			(at 158.75 80.0099 0)
 			(effects
@@
 			(project ""
 				(path "/0e457dee-ab7a-4947-acac-685db257dbd9/ac8308a5-c176-4748-bfbf-484ade2f530b"
-					(reference "C3")
-					(unit 1)
-				)
+					(reference "C5")
+					(unit 1)
+				)

Commit message: Replaced BNO with BMI
Parts:
- removed C5: 100nF, Capacitor_SMD:C_0805_2012Metric, symbol Device:C
- removed U1: BNO055, Package_LGA:LGA-28_5.2x3.8mm_P0.5mm, symbol SRAD:BNO055
- added U1: BMI088, BMI088 (1):PQFN50P450X300X100-16N, symbol BMI088:BMI088
- C3: value 1uF -> 100nF; footprint Capacitor_SMD:C_0805_2012Metric -> Capacitor_SMD:C_0603_1608Metric
- C4: footprint Capacitor_SMD:C_0805_2012Metric -> Capacitor_SMD:C_0603_1608Metric
Connections:
- net +3V3: now also C3.1, U1.11 (VDDIO), U1.14 (CSB1), U1.3 (VDD), U1.7 (PS)
- net GND: now also C3.2, U1.1 (INT2), U1.10 (SDO2), U1.12 (INT3), U1.13 (INT4), U1.15 (SDO1), U1.16 (INT1), U1.2 (NC), U1.4 (GNDA), U1.6 (GNDIO); no longer C3.1
- net SCL: now also U1.8 (SCL/SCK)
- net SDA: now also U1.9 (SDA/SDI)
- no-connect marks 6 -> 1
Other:
- note added: "Accelerometer: SD01 to gnd: 0011000b (0x18) SD01 to VDD(): 0011001b (0x19) Gyroscope: SD01 to gnd: 1101000b (0x68) SD01 to VDDIO: 1101001b (0x69)"
- note removed: "Default I2C address (COM3 HIGH): 0100101b (0x29) Alternate I2C address (COM3 LOW): 0101000b (0x28) COM3 is used to switch adress"
- note removed: "Should be done, went through all pins on datasheet"
