File: Apollo/project_folder/AlexFlightComputer/AlexFlightComputer.kicad_pcb (KiCad board)
At the start: 2 copper layers, 9 parts, among them IC1 WSEN-PADS_2511020213301 (Baro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, J1 BAT, J2 SW, J3 GPS, J4 Radio, U1 MLX90393SLW-ABA-011-RE (Magne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, U2 BMI270 (IMU)

Commit message: Made Board v.2
Adjusted for pin out
Connections:
- IC1 pad 3: unconnected-(IC1-Pad3) -> GND
- IC1 pad 5: unconnected-(IC1-Pad5) -> +3.3V
- IC1 pad 6: unconnected-(IC1-Pad6) -> +3.3V
- U1 pad 2: unconnected-(U1-MS/CS-Pad2) -> +3.3V
- U2 pad 1: unconnected-(U2-SDO-Pad1) -> GND
- U2 pad 12: unconnected-(U2-CSB-Pad12) -> +3.3V
Changed lines of the file:
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@@
 	(net 45 "unconnected-(Teensy4.1-TX2-Pad8)")
 	(net 46 "/Batt-Sw")
-	(net 47 "unconnected-(U1-MS{slash}CS-Pad2)")
-	(net 48 "unconnected-(U1-INT{slash}TRIG-Pad7)")
-	(net 49 "unconnected-(U1-N{slash}C__1-Pad9)")
-	(net 50 "unconnected-(U1-A0-Pad12)")
-	(net 51 "unconnected-(U1-N{slash}C__2-Pad10)")
-	(net 52 "unconnected-(U1-A1-Pad11)")
-	(net 53 "unconnected-(U1-N{slash}C-Pad4)")
-	(net 54 "unconnected-(U1-EXP-Pad17)")
-	(net 55 "unconnected-(U1-N{slash}C__3-Pad14)")
-	(net 56 "unconnected-(U1-INT-Pad1)")
-	(net 57 "unconnected-(U1-MISO-Pad6)")
-	(net 58 "unconnected-(U1-N{slash}C__4-Pad16)")
-	(net 59 "unconnected-(U2-INT1-Pad4)")
-	(net 60 "unconnected-(U2-ASCX-Pad3)")
-	(net 61 "unconnected-(U2-OSDO-Pad11)")
-	(net 62 "unconnected-(U2-OSCB-Pad10)")
-	(net 63 "unconnected-(U2-SDO-Pad1)")
-	(net 64 "unconnected-(U2-CSB-Pad12)")
-	(net 65 "unconnected-(U2-INT2-Pad9)")
-	(net 66 "unconnected-(U2-ASDX-Pad2)")
-	(net 67 "unconnected-(IC1-Pad3)")
-	(net 68 "unconnected-(IC1-Pad6)")
-	(net 69 "unconnected-(IC1-Pad7)")
-	(net 70 "unconnected-(IC1-Pad5)")
+	(net 47 "unconnected-(U1-INT{slash}TRIG-Pad7)")
+	(net 48 "unconnected-(U1-N{slash}C__1-Pad9)")
+	(net 49 "unconnected-(U1-A0-Pad12)")
+	(net 50 "unconnected-(U1-N{slash}C__2-Pad10)")
+	(net 51 "unconnected-(U1-A1-Pad11)")
+	(net 52 "unconnected-(U1-N{slash}C-Pad4)")
+	(net 53 "unconnected-(U1-EXP-Pad17)")
+	(net 54 "unconnected-(U1-N{slash}C__3-Pad14)")
+	(net 55 "unconnected-(U1-INT-Pad1)")
+	(net 56 "unconnected-(U1-MISO-Pad6)")
+	(net 57 "unconnected-(U1-N{slash}C__4-Pad16)")
+	(net 58 "unconnected-(U2-INT1-Pad4)")
+	(net 59 "unconnected-(U2-ASCX-Pad3)")
+	(net 60 "unconnected-(U2-OSDO-Pad11)")
+	(net 61 "unconnected-(U2-OSCB-Pad10)")
+	(net 62 "unconnected-(U2-INT2-Pad9)")
+	(net 63 "unconnected-(U2-ASDX-Pad2)")
+	(net 64 "unconnected-(IC1-Pad7)")
 	(footprint "Connector_JST:JST_XH_B4B-XH-A_1x04_P2.50mm_Vertical"
 		(layer "F.Cu")
@@
 			(size 0.35 0.375)
 			(layers "F.Cu")
-			(net 67 "unconnected-(IC1-Pad3)")
-			(pintype "bidirectional+no_connect")
+			(net 12 "GND")
+			(pintype "bidirectional")
 		)
 		(pad "4" smd rect
@@
 			(size 0.35 0.375)
 			(layers "F.Cu")
-			(net 70 "unconnected-(IC1-Pad5)")
-			(pintype "bidirectional+no_connect")
+			(net 26 "+3.3V")
+			(pintype "bidirectional")
 		)
 		(pad "6" smd rect
@@
 			(size 0.375 0.35)
 			(layers "F.Cu")
-			(net 68 "unconnected-(IC1-Pad6)")
-			(pintype "input+no_connect")
+			(net 26 "+3.3V")
+			(pintype "input")
 		)
 		(pad "7" smd rect
@@
 			(size 0.375 0.35)
 			(layers "F.Cu")
-			(net 69 "unconnected-(IC1-Pad7)")
+			(net 64 "unconnected-(IC1-Pad7)")
 			(pintype "output+no_connect")
 		)
@@
 			(size 0.254 0.8128)
 			(layers "F.Cu" "F.Mask" "F.Paste")
-			(net 56 "unconnected-(U1-INT-Pad1)")
+			(net 55 "unconnected-(U1-INT-Pad1)")
 			(pinfunction "INT")
 			(pintype "output+no_connect")
@@
 			(size 0.254 0.8128)
 			(layers "F.Cu" "F.Mask" "F.Paste")
-			(net 47 "unconnected-(U1-MS{slash}CS-Pad2)")
+			(net 26 "+3.3V")
 			(pinfunction "MS/CS")
-			(pintype "input+no_connect")
+			(pintype "input")
 		)
 		(pad "3" smd rect
@@
 			(size 0.254 0.8128)
 			(layers "F.Cu" "F.Mask" "F.Paste")
-			(net 53 "unconnected-(U1-N{slash}C-Pad4)")
+			(net 52 "unconnected-(U1-N{slash}C-Pad4)")
 			(pinfunction "N/C")
 			(pintype "passive+no_connect")
@@
 			(size 0.254 0.8128)
 			(layers "F.Cu" "F.Mask" "F.Paste")
-			(net 57 "unconnected-(U1-MISO-Pad6)")
+			(net 56 "unconnected-(U1-MISO-Pad6)")
 			(pinfunction "MISO")
 			(pintype "output+no_connect")
@@
 			(size 0.254 0.8128)
 			(layers "F.Cu" "F.Mask" "F.Paste")
-			(net 48 "unconnected-(U1-INT{slash}TRIG-Pad7)")
+			(net 47 "unconnected-(U1-INT{slash}TRIG-Pad7)")
 			(pinfunction "INT/TRIG")
 			(pintype "bidirectional+no_connect")
@@
 			(size 0.254 0.8128)
 			(layers "F.Cu" "F.Mask" "F.Paste")
-			(net 49 "unconnected-(U1-N{slash}C__1-Pad9)")
+			(net 48 "unconnected-(U1-N{slash}C__1-Pad9)")
 			(pinfunction "N/C__1")
 			(pintype "passive+no_connect")
@@
 			(size 0.254 0.8128)
 			(layers "F.Cu" "F.Mask" "F.Paste")
-			(net 51 "unconnected-(U1-N{slash}C__2-Pad10)")
+			(net 50 "unconnected-(U1-N{slash}C__2-Pad10)")
 			(pinfunction "N/C__2")
 			(pintype "passive+no_connect")
@@
 			(size 0.254 0.8128)
 			(layers "F.Cu" "F.Mask" "F.Paste")
-			(net 52 "unconnected-(U1-A1-Pad11)")
+			(net 51 "unconnected-(U1-A1-Pad11)")
 			(pinfunction "A1")
 			(pintype "input+no_connect")
@@
 			(size 0.254 0.8128)
 			(layers "F.Cu" "F.Mask" "F.Paste")
-			(net 50 "unconnected-(U1-A0-Pad12)")
+			(net 49 "unconnected-(U1-A0-Pad12)")
 			(pinfunction "A0")
 			(pintype "input+no_connect")
@@
 			(size 0.254 0.8128)
 			(layers "F.Cu" "F.Mask" "F.Paste")
-			(net 55 "unconnected-(U1-N{slash}C__3-Pad14)")
+			(net 54 "unconnected-(U1-N{slash}C__3-Pad14)")
 			(pinfunction "N/C__3")
 			(pintype "passive+no_connect")
@@
 			(size 0.254 0.8128)
 			(layers "F.Cu" "F.Mask" "F.Paste")
-			(net 58 "unconnected-(U1-N{slash}C__4-Pad16)")
+			(net 57 "unconnected-(U1-N{slash}C__4-Pad16)")
 			(pinfunction "N/C__4")
 			(pintype "passive+no_connect")
@@
 			(size 1.6764 1.6764)
 			(layers "F.Cu" "F.Mask" "F.Paste")
-			(net 54 "unconnected-(U1-EXP-Pad17)")
+			(net 53 "unconnected-(U1-EXP-Pad17)")
 			(pinfunction "EXP")
 			(pintype "passive+no_connect")
@@
 			(size 0.475 0.25)
 			(layers "F.Cu" "F.Mask" "F.Paste")
-			(net 63 "unconnected-(U2-SDO-Pad1)")
+			(net 12 "GND")
 			(pinfunction "SDO")
-			(pintype "bidirectional+no_connect")
+			(pintype "bidirectional")
 			(solder_mask_margin 0.102)
 		)
@@
 			(size 0.475 0.25)
 			(layers "F.Cu" "F.Mask" "F.Paste")
-			(net 66 "unconnected-(U2-ASDX-Pad2)")
+			(net 63 "unconnected-(U2-ASDX-Pad2)")
 			(pinfunction "ASDX")
 			(pintype "bidirectional+no_connect")
@@
 			(size 0.475 0.25)
 			(layers "F.Cu" "F.Mask" "F.Paste")
-			(net 60 "unconnected-(U2-ASCX-Pad3)")
+			(net 59 "unconnected-(U2-ASCX-Pad3)")
 			(pinfunction "ASCX")
 			(pintype "bidirectional+no_connect")
@@
 			(size 0.475 0.25)
 			(layers "F.Cu" "F.Mask" "F.Paste")
-			(net 59 "unconnected-(U2-INT1-Pad4)")
+			(net 58 "unconnected-(U2-INT1-Pad4)")
 			(pinfunction "INT1")
 			(pintype "bidirectional+no_connect")
@@
 			(size 0.475 0.25)
 			(layers "F.Cu" "F.Mask" "F.Paste")
-			(net 65 "unconnected-(U2-INT2-Pad9)")
+			(net 62 "unconnected-(U2-INT2-Pad9)")
 			(pinfunction "INT2")
 			(pintype "bidirectional+no_connect")
@@
 			(size 0.475 0.25)
 			(layers "F.Cu" "F.Mask" "F.Paste")
-			(net 62 "unconnected-(U2-OSCB-Pad10)")
+			(net 61 "unconnected-(U2-OSCB-Pad10)")
 			(pinfunction "OSCB")
 			(pintype "input+no_connect")
@@
 			(size 0.475 0.25)
 			(layers "F.Cu" "F.Mask" "F.Paste")
-			(net 61 "unconnected-(U2-OSDO-Pad11)")
+			(net 60 "unconnected-(U2-OSDO-Pad11)")
 			(pinfunction "OSDO")
 			(pintype "output+no_connect")
@@
 			(size 0.25 0.475)
 			(layers "F.Cu" "F.Mask" "F.Paste")
-			(net 64 "unconnected-(U2-CSB-Pad12)")
+			(net 26 "+3.3V")
 			(pinfunction "CSB")
-			(pintype "input+no_connect")
+			(pintype "input")
 			(solder_mask_margin 0.102)
 		)

Commit message: Post-Review Revisions (10/27)
Parts:
- added C1: 100nF, Capacitor_SMD:C_0603_1608Metric, F.Cu at (175.2, 64.0)
- added C2: 100nF, Capacitor_SMD:C_0603_1608Metric, F.Cu at (175.3, 69.5)
- added C3: 100nF, Capacitor_SMD:C_0603_1608Metric, F.Cu at (176.0, 55.5)
- added C4: 100nF, Capacitor_SMD:C_0603_1608Metric, F.Cu at (169.0, 72.5)
- added C5: 100nF, Capacitor_SMD:C_0603_1608Metric, F.Cu at (174.5, 60.2)
- added C6: 100nF, Capacitor_SMD:C_0603_1608Metric, F.Cu at (168.5, 49.5)
- added D1: LED, LED_SMD:LED_0805_2012Metric, F.Cu at (165.0, 37.4)
- added H1: MountingHole, MountingHole:MountingHole_3.2mm_M3, F.Cu at (142.0, 101.5)
- added H2: MountingHole, MountingHole:MountingHole_3.2mm_M3, F.Cu at (171.0, 101.5)
- added R1: 5.1kR, Resistor_SMD:R_0201_0603Metric, F.Cu at (167.0, 62.0)
- added R2: 5.1kR, Resistor_SMD:R_0201_0603Metric, F.Cu at (167.8, 65.0)
- added R3: 560, Resistor_SMD:R_0201_0603Metric, F.Cu at (165.2, 41.5)
- moved U2 1.91 mm to (168.5, 68.5)
Connections:
- U1 pad 11: unconnected-(U1-A1-Pad11) -> +3.3V
- U1 pad 12: unconnected-(U1-A0-Pad12) -> +3.3V

Commit message: Completed PCB v.1 (10/29)
Parts:
- added H3: MountingHole, MountingHole:MountingHole_3.2mm_M3, F.Cu at (176.0, 116.0)
- moved H1 71.2 mm to (157.5, 32.0)
- moved J3 36.7 mm to (178.0, 67.2)
- moved H2 36.0 mm to (138.0, 116.0)
- moved J1 30.0 mm to (142.8, 37.4)
- moved J2 28.5 mm to (172.8, 37.4)
- moved BZ1 28.3 mm to (157.5, 112.0), turned to 0 degrees
- moved C4 22.0 mm to (176.2, 51.8), turned to 180 degrees
- moved U2 17.8 mm to (179.5, 54.5), turned to 180 degrees
- moved IC1 16.3 mm to (170.0, 70.5), turned to -90 degrees
- moved D1 10.7 mm to (168.5, 47.6), turned to -90 degrees
- moved R3 9.13 mm to (168.5, 50.0), turned to 180 degrees
- moved C1 6.43 mm to (173.8, 70.3), turned to 90 degrees
- moved J4 5.25 mm to (142.0, 54.2)
- moved C3 5.24 mm to (179.7, 51.8)
- moved C6 4.95 mm to (168.8, 54.4)
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Routing:
- net +3.3V: track 0.00 -> 188.1 mm, vias 0 -> 10
- net GND: track 0.00 -> 185.8 mm, vias 0 -> 11
- net /SDA: track 0.00 -> 42.5 mm, vias 0 -> 2
- net /SCL: track 0.00 -> 32.8 mm, vias 0 -> 2
- net /Batt-Sw: track 0.00 -> 27.5 mm
- net +5V: track 0.00 -> 10.7 mm
- net Net-(BZ1-+): track 0.00 -> 10.5 mm
- net /RX: track 0.00 -> 8.67 mm
- net /TX: track 0.00 -> 8.65 mm
- net Net-(D1-A): track 0.00 -> 1.63 mm
Other:
- board outline added: 53.5 x 99 mm
