File: Apollo/project_folder/amin_flight_computer/amin_flight_computer.kicad_sch (KiCad schematic)
At the start: 0 parts

Commit message: Amin project
Parts:
- added BT1: Battery_Cell, Connector_JST:JST_JWPF_B02B-JWPF-SK-R_1x02_P2.00mm_Vertical, symbol Device:Battery_Cell
- added D1, D2: D_Schottky, Diode_SMD:D_0201_0603Metric, symbol Device:D_Schottky
- added J1: USB4105-GF-A-060, USB4105-GF-A-060:GCT_USB4105-GF-A-060, symbol Imported:USB4105-GF-A-060
- added J2: Conn_Coaxial_Small, Connector_Coaxial:U.FL_Molex_MCRF_73412-0110_Vertical, symbol Connector:Conn_Coaxial_Small
- added U1: LEA-M8T, RF_GPS:ublox_LEA, symbol RF_GPS:LEA-M8T
- added U2: ESP32-S3-MINI-1, RF_Module:ESP32-S2-MINI-1, symbol RF_Module:ESP32-S3-MINI-1
- added U3: XC6220B331MR, Package_TO_SOT_SMD:SOT-23-5, symbol Regulator_Linear:XC6220B331MR
- added U4: TPD2EUSB30, Package_TO_SOT_SMD:Texas_DRT-3, symbol Power_Protection:TPD2EUSB30
Connections:
- new net: BT1.1 (+), D2.2 (A)
- new net: U1.1 (SDA/~{SPI_CS}), U2.4 (IO0)
- new net: J2.1 (In), U1.16 (RF_IN)
- new net: U1.2 (SCL/SPI_CLK), U2.5 (IO1)
- new net: J1.A7 (DN1), U2.23 (USB_D-), U4.1 (D+)
- new net: J1.A6 (DP1), U2.24 (USB_D+), U4.2 (D-)
- new net: D1.1 (K), D2.1 (K), U3.1 (VIN)
- new net: D1.2 (A), J1.A4_B9 (VBUS), J1.B4_A9 (VBUS)
- new net GND: BT1.2 (-), J1.A1_B12 (GND), J1.B1_A12 (GND), J1.SH1 (SHELL_GND), J1.SH2 (SHELL_GND), J1.SH3 (SHELL_GND), J1.SH4 (SHELL_GND), J2.2 (Ext), U1.13 (GND), U1.14 (GND), U1.15 (GND), U1.17 (GND), U1.19 (V_ANT), U1.7 (GND), U2.1 (GND), U2.2 (GND), U2.42 (GND), U2.43 (GND), U2.46 (GND), U2.47 (GND), U2.48 (GND), U2.49 (GND), U2.50 (GND), U2.51 (GND), U2.52 (GND), U2.53 (GND), U2.54 (GND), U2.55 (GND), U2.56 (GND), U2.57 (GND), U2.58 (GND), U2.59 (GND), U2.60 (GND), U2.61 (GND), U2.62 (GND), U2.63 (GND), U2.64 (GND), U2.65 (GND), U3.2 (GND), U4.3 (GND)
- new net VCC: U1.11 (V_BCKP), U1.6 (VCC), U2.3 (3V3), U3.5 (VOUT)

Commit message: PCB Updates
Parts:
- removed BT1: Battery_Cell, Connector_JST:JST_JWPF_B02B-JWPF-SK-R_1x02_P2.00mm_Vertical, symbol Device:Battery_Cell
- added C1: 100nf, Capacitor_SMD:C_0603_1608Metric, symbol Device:C
- added D3: LED, LED_SMD:LED_0805_2012Metric, symbol Device:LED
- added H1, H2: MountingHole_Pad, TestPoint:TestPoint_Plated_Hole_D2.0mm, symbol Mechanical:MountingHole_Pad
- added J3: Battery1, Connector_JST:JST_PH_B2B-PH-K_1x02_P2.00mm_Vertical, symbol Connector_Generic:Conn_01x02
- added R1: 5.1K, Resistor_SMD:R_0603_1608Metric, symbol Device:R
- D1, D2: footprint Diode_SMD:D_0201_0603Metric -> Diode_SMD:D_0603_1608Metric
- J1: footprint USB4105-GF-A-060:GCT_USB4105-GF-A-060 -> USB4105_GF_A_060:GCT_USB4105-GF-A-060; symbol Imported:USB4105-GF-A-060 -> USB4105-GF-A-060:USB4105-GF-A-060
- U2: footprint RF_Module:ESP32-S2-MINI-1 -> ESP32_S3_MINI_1_N4R2:XCVR_ESP32-S3-MINI-1-N4R2
Connections:
- net GND: now also C1.1, D3.1 (K), H1.1, H2.1, J3.2 (Pin_2)
- net VCC: now also C1.2, R1.1
- net at D2.2 (A): now also J3.1 (Pin_1)
- net at U2.45 (EN): now also R1.2
- net at U2.6 (IO2): now also D3.2 (A)
- net at D1.1 (K), D2.1 (K), U3.1 (VIN): now also U3.3 (CE)
- net at D1.2 (A), J1.A4_B9 (VBUS): no longer J1.B4_A9 (VBUS)
- no-connect marks 0 -> 54
Other:
- moved on the sheet: D1, D2

Commit message: Update capacitor size
Parts:
- C1: footprint Capacitor_SMD:C_0603_1608Metric -> Capacitor_SMD:C_0805_2012Metric
Changed lines of the file:
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@@
 			)
 		)
-		(property "Footprint" "Capacitor_SMD:C_0603_1608Metric"
+		(property "Footprint" "Capacitor_SMD:C_0805_2012Metric"
 			(at 149.86 29.5148 0)
 			(effects

Commit message: Amin FC Updates
Parts:
- added Boot1, Reset1: SKRPABE010, footprints:SW4_SKRPABE010_ALPS, symbol 2025-11-04_22-14-40:SKRPABE010
- added C2: 10uf, Capacitor_SMD:C_0805_2012Metric, symbol Device:C
- added D4: LED_PWR, LED_SMD:LED_0805_2012Metric, symbol Device:LED
- added R2, R3, R6: 10K, Resistor_SMD:R_0603_1608Metric, symbol Device:R
- added R4, R5: 5.1K, Resistor_SMD:R_0402_1005Metric, symbol Device:R
- added SW1: CSS-1210TB, footprints:SW3_CSS-1210TB_NDC, symbol 2025-11-04_22-26-13:CSS-1210TB
- C1: value 100nf -> 22uf
- D3: value LED -> LED_GPIO
- R1: value 5.1K -> 10K
Connections:
- net GND: now also C1.2, Boot1.1, C2.2, R3.1, R4.1, R5.1, R6.1, Reset1.1, SW1.1; no longer C1.1, D3.1 (K)
- net VCC: now also C1.1, D4.2 (A), R2.1; no longer C1.2
- net at R1.2, U2.45 (EN): now also Reset1.4
- net at U1.1 (SDA/~{SPI_CS}): now also U2.12 (IO8); no longer U2.4 (IO0)
- net at U1.2 (SCL/SPI_CLK): now also U2.13 (IO9); no longer U2.5 (IO1)
- net at D3.2 (A): now also U2.15 (IO11); no longer U2.6 (IO2)
- net at J1.A7 (DN1), U4.1 (D+): now also U2.24 (USB_D+); no longer U2.23 (USB_D-)
- net at J1.A6 (DP1), U4.2 (D-): now also U2.23 (USB_D-); no longer U2.24 (USB_D+)
- net at D1.1 (K), D2.1 (K), U3.1 (VIN): now also C2.1, SW1.2; no longer U3.3 (CE)
- net at J1.A5 (CC1): now also R4.2
- net at J1.B5 (CC2): now also R5.2
- new net: D4.1 (K), R6.2
- new net: D3.1 (K), R3.2
- new net: Boot1.3, R2.2, U2.4 (IO0)
- new net: SW1.3, U3.3 (CE)
Other:
- moved on the sheet: D1, D2, D3, H1, H2, J1, J2, J3, U1, U3, U4

Commit message: Amin FC Updates
Connections:
- net SDA: now reaches U1.1 (SDA/~{SPI_CS}), U2.12 (IO8)
- net SCL: now reaches U1.2 (SCL/SPI_CLK), U2.13 (IO9)
- net DN: now reaches U2.23 (USB_D-), U4.2 (D-)
- net DN: now also J1.A7 (DN1), J1.B7 (DN2); no longer J1.A6 (DP1)
- net DP: now reaches U2.24 (USB_D+), U4.1 (D+)
- net DP: now also J1.A6 (DP1), J1.B6 (DP2); no longer J1.A7 (DN1)
- no-connect marks 54 -> 52
Other:
- moved on the sheet: D1, D3, R3, R4, R5
