File: Apollo/project_folder/Ahlinkar flights computer/rockets test.kicad_sch (KiCad schematic)
At the start: 14 parts, among them J1 switch, J2 batt, U1(Barometer)1 LPS22HH, U2(Magnetometer)1 MLX90395xLW, U3(IMU)1 BMI323

Commit message: added LEDs and organized pcb layout
Parts:
- added D1: red LED, LED_SMD:LED_0805_2012Metric, symbol Device:LED
- added D2: green LED, LED_SMD:LED_0805_2012Metric, symbol Device:LED
- added R3: ~, Resistor_SMD:R_0603_1608Metric, symbol Device:R
Connections:
- net +3.3V: now also R3.2
- net GND: now also D1.1 (K), D2.1 (K)
- new net: D1.2 (A), D2.2 (A), R3.1

Commit message: Ahlinkar update wired pcb design
Parts:
- Radio1: footprint Connector_JST:JST_XH_B4B-XH-AM_1x04_P2.50mm_Vertical -> Connector_JST:JST_XH_B4B-XH-A_1x04_P2.50mm_Vertical
Changed lines of the file:
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@@
 			)
 		)
-		(property "Footprint" "Connector_JST:JST_XH_B4B-XH-AM_1x04_P2.50mm_Vertical"
+		(property "Footprint" "Connector_JST:JST_XH_B4B-XH-A_1x04_P2.50mm_Vertical"
 			(at 107.95 175.26 0)
 			(effects

Commit message: Ahlinkar - update on pcb design and wiring connections
Parts:
- R1, R2: value 100 kOhms -> 5.1k
- R3: value ~ -> 183
Connections:
- net GND: no longer U1(Barometer)1.6 (~{CS}), U2(Magnetometer)1.2 (~{CS})
- net RX: now also Radio1.3 (Pin_3); no longer Radio1.2 (Pin_2)
- net TX: now also Radio1.2 (Pin_2); no longer Radio1.3 (Pin_3)
- removed net A0: Teensy4.1.14 (A0), U1(Barometer)1.5 (SA0), U2(Magnetometer)1.12 (A0)
- net A1: no longer names the net of Teensy4.1.15 (A1)
- net A1: no longer U2(Magnetometer)1.11 (A1)
- no-connect marks 40 -> 42
Changed lines of the file:
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@@
 	)
 	(no_connect
-		(at 134.62 161.29)
-	)
-	(no_connect
 		(at 134.62 153.67)
 	)
@@
 	)
 	(no_connect
-		(at 134.62 158.75)
-	)
-	(no_connect
 		(at 97.79 129.54)
 	)
@@
 	)
 	(no_connect
+		(at 72.39 114.3)
+	)
+	(no_connect
 		(at 97.79 93.98)
 	)
@@
 	)
 	(no_connect
+		(at 161.29 83.82)
+	)
+	(no_connect
 		(at 72.39 116.84)
 	)
@@
 	)
 	(no_connect
+		(at 114.3 43.18)
+	)
+	(no_connect
 		(at 97.79 96.52)
 	)
@@
 	)
 	(no_connect
+		(at 97.79 114.3)
+	)
+	(no_connect
 		(at 72.39 127)
 	)
 	(no_connect
+		(at 97.79 116.84)
+	)
+	(no_connect
 		(at 72.39 93.98)
 	)
@@
 		(at 72.39 119.38)
 	)
-	(no_connect
-		(at 114.3 43.18)
-	)
 	(wire
 		(pts
@@
 	(wire
 		(pts
-			(xy 162.56 146.05) (xy 160.02 146.05)
-		)
-		(stroke
-			(width 0)
-			(type default)
-		)
-	)
-	(wire
-		(pts
 			(xy 40.64 119.38) (xy 40.64 121.92)
 		)
@@
 	(wire
 		(pts
-			(xy 100.33 114.3) (xy 97.79 114.3)
-		)
-		(stroke
-			(width 0)
-			(type default)
-		)
-	)
-	(wire
-		(pts
 			(xy 147.32 66.04) (xy 154.94 66.04)
 		)
@@
 	(wire
 		(pts
-			(xy 162.56 148.59) (xy 160.02 148.59)
-		)
-		(stroke
-			(width 0)
-			(type default)
-		)
-	)
-	(wire
-		(pts
 			(xy 109.22 83.82) (xy 118.11 83.82)
 		)
@@
 	(wire
 		(pts
-			(xy 129.54 146.05) (xy 134.62 146.05)
-		)
-		(stroke
-			(width 0)
-			(type default)
-		)
-	)
-	(wire
-		(pts
 			(xy 161.29 40.64) (xy 154.94 40.64)
 		)
@@
 	(wire
 		(pts
-			(xy 68.58 114.3) (xy 72.39 114.3)
-		)
-		(stroke
-			(width 0)
-			(type default)
-		)
-	)
-	(wire
-		(pts
 			(xy 165.1 95.25) (xy 160.02 95.25)
 		)
@@
 	(wire
 		(pts
-			(xy 179.07 107.95) (xy 175.26 107.95)
-		)
-		(stroke
-			(width 0)
-			(type default)
-		)
-	)
-	(wire
-		(pts
 			(xy 154.94 35.56) (xy 156.21 35.56)
 		)
@@
 	(wire
 		(pts
-			(xy 100.33 116.84) (xy 97.79 116.84)
-		)
-		(stroke
-			(width 0)
-			(type default)
-		)
-	)
-	(wire
-		(pts
 			(xy 99.06 86.36) (xy 99.06 83.82)
 		)
@@
 	(wire
 		(pts
-			(xy 177.8 102.87) (xy 175.26 102.87)
-		)
-		(stroke
-			(width 0)
-			(type default)
-		)
-	)
-	(wire
-		(pts
 			(xy 69.85 151.13) (xy 93.98 151.13)
 		)
@@
 	(wire
 		(pts
+			(xy 99.06 175.26) (xy 102.87 175.26)
+		)
+		(stroke
+			(width 0)
+			(type default)
+		)
+	)
+	(wire
+		(pts
 			(xy 99.06 86.36) (xy 97.79 86.36)
 		)
@@
 	(wire
 		(pts
-			(xy 99.06 175.26) (xy 102.87 175.26)
-		)
-		(stroke
-			(width 0)
-			(type default)
-		)
-	)
-	(wire
-		(pts
 			(xy 129.54 151.13) (xy 134.62 151.13)
 		)
@@
 		)
 	)
-	(label "A1"
-		(at 162.56 146.05 0)
-		(effects
-			(font
-				(size 1.27 1.27)
-			)
-			(justify left bottom)
-		)
-	)
-	(label "A1"
-		(at 100.33 114.3 0)
-		(effects
-			(font
-				(size 1.27 1.27)
-			)
-			(justify left bottom)
-		)
-	)
 	(label "SDA"
 		(at 55.88 171.45 0)
@@
 		)
 	)
-	(label "CS"
-		(at 177.8 107.95 0)
+	(label "TX"
+		(at 99.06 175.26 0)
 		(effects
 			(font
@@
 		)
 	)
-	(label "A0"
-		(at 100.33 116.84 0)
-		(effects
-			(font
-				(size 1.27 1.27)
-			)
-			(justify left bottom)
-		)
-	)
 	(label "TX"
 		(at 69.85 91.44 0)
@@
 		)
 	)
-	(label "A0"
-		(at 162.56 148.59 0)
-		(effects
-			(font
-				(size 1.27 1.27)
-			)
-			(justify left bottom)
-		)
-	)
-	(label "TX"
-		(at 99.06 177.8 0)
-		(effects
-			(font
-				(size 1.27 1.27)
-			)
-			(justify left bottom)
-		)
-	)
-	(label "CS"
-		(at 129.54 146.05 0)
-		(effects
-			(font
-				(size 1.27 1.27)
-			)
-			(justify left bottom)
-		)
-	)
 	(label ""
 		(at 154.94 38.1 0)
@@
 		)
 	)
-	(label "CS"
-		(at 68.58 114.3 0)
+	(label "RX"
+		(at 99.06 177.8 0)
 		(effects
 			(font
@@
 		)
 	)
-	(label "RX"
-		(at 99.06 175.26 0)
-		(effects
-			(font
-				(size 1.27 1.27)
-			)
-			(justify left bottom)
-		)
-	)
-	(label "A0"
-		(at 177.8 102.87 0)
-		(effects
-			(font
-				(size 1.27 1.27)
-			)
-			(justify left bottom)
-		)
-	)
 	(symbol
 		(lib_id "power:GND")
@@
 			)
 		)
-		(property "Value" "100 kOhms"
+		(property "Value" "5.1k"
 			(at 120.65 17.526 90)
 			(effects
@@
 			)
 		)
-		(property "Value" "100 kOhms"
+		(property "Value" "5.1k"
 			(at 131.572 23.876 90)
 			(effects
@@
 			)
 		)
-		(property "Value" "~"
+		(property "Value" "183"
 			(at 55.88 114.3 90)
 			(effects
@@
 					(size 1.27 1.27)
 				)
-				(hide yes)
 			)
 		)

Commit message: Ahlinkar - update on pcb
Parts:
- removed R3: 183, Resistor_SMD:R_0603_1608Metric, symbol Device:R
- added D3: LED, LED_SMD:LED_0805_2012Metric, symbol Device:LED
- added H1, H2, H3, H4: MountingHole, MountingHole:MountingHole_3.2mm_M3, symbol Mechanical:MountingHole
- added R4, R5, R6: 560, Resistor_SMD:R_0603_1608Metric, symbol Device:R
Connections:
- net +3.3V: now also D3.2 (A)
- net GND: now also R4.2, R5.2, R6.2; no longer D1.1 (K), D2.1 (K)
- net at D2.2 (A): now also Teensy4.1.31 (GPIO); no longer D1.2 (A)
- net at Teensy4.1.32 (GPIO): now also D1.2 (A)
- new net: D3.1 (K), R6.1
- new net: D2.1 (K), R4.1
- new net: D1.1 (K), R5.1
- no-connect marks 42 -> 39
Other:
- moved on the sheet: D1, D2, GPS1

Commit message: ahlinkar
Connections:
- net GND: no longer GPS1.2 (Pin_2), GPS1.3 (Pin_3), R1.2, R2.2, Teensy4.1.10 (CS), Teensy4.1.18 (SDA), Teensy4.1.19 (SCL), U1(Barometer)1.2 (SCL), U1(Barometer)1.4 (SDA), U2(Magnetometer)1.3 (SCLK), U2(Magnetometer)1.5 (MOSI), U2(Magnetometer)1.7 (INT/TRG), U3(IMU)1.13 (SCX), U3(IMU)1.14 (SDX)
- new net SCL: GPS1.3 (Pin_3), R1.2, Teensy4.1.19 (SCL), U1(Barometer)1.2 (SCL), U2(Magnetometer)1.3 (SCLK), U3(IMU)1.13 (SCX)
- new net SDA: GPS1.2 (Pin_2), R2.2, Teensy4.1.18 (SDA), U1(Barometer)1.4 (SDA), U2(Magnetometer)1.5 (MOSI), U3(IMU)1.14 (SDX)

Commit message: Ahlinkar - fixed some errors
Connections:
- net +3.3V: now also U1(Barometer)1.6 (~{CS})
- net GND: now also U1(Barometer)1.5 (SA0)
- no-connect marks 39 -> 44

Commit message: final changes
Connections:
- net +3.3V: now also U2(Magnetometer)1.11 (A1), U2(Magnetometer)1.2 (~{CS})
- net GND: now also U2(Magnetometer)1.12 (A0), U2(Magnetometer)1.6 (MISO)
- no-connect marks 44 -> 40
