File: Apollo/project_folder/RyanLing_Flight_Computer/RyanLing_Flight_Computer.kicad_pcb (KiCad board)
At the start: 2 copper layers, 25 parts, among them J1 Battery, J2 Switch, U1 ICM-20948, U2 BMP390

Commit message: Update RyanLing_Flight_Computer.kicad_pcb
Parts:
- moved U1 1.12 mm to (135.5, 67.0), turned to 180 degrees
- moved H1 0.50 mm to (156.0, 31.5)
Routing:
- net +3.3V: track 79.2 -> 67.8 mm, vias 7 -> 6
- net GND: track 152.1 -> 143.4 mm, vias 8 -> 9
- net (no net): track 5.33 -> 0.00 mm, vias 2 -> 0
- net /SCL: track 50.7 -> 47.3 mm, vias 2 -> 3
- net Net-(U1-REGOUT): track 7.58 -> 4.51 mm
- net /SDA: track 34.5 -> 37.4 mm, vias 5 -> 3
- net Net-(J2-Pin_1): track 14.7 -> 16.4 mm, vias 0 -> 1
- net Net-(Teensy4.1-A17): track 44.5 -> 44.6 mm, vias 0 -> 1
Other:
- board outline added: 37 x 77.5 mm

Commit message: Ryan Ling's PCB(Final)
Parts:
- moved H1 4.50 mm to (156.0, 65.0)
- moved H1 0.50 mm to (156.0, 31.0)
Other:
- board text added: "Ryan Ling"
Changed lines of the file:
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@@
 	(footprint "MountingHole:MountingHole_3.2mm_M3"
 		(layer "F.Cu")
-		(at 156 31.5)
+		(at 156 31)
 		(descr "Mounting Hole 3.2mm, M3, no annular, generated by kicad-footprint-generator mountinghole.py")
 		(tags "mountinghole M3")
@@
 	(footprint "MountingHole:MountingHole_3.2mm_M3"
 		(layer "F.Cu")
-		(at 151.5 65)
+		(at 156 65)
 		(descr "Mounting Hole 3.2mm, M3, no annular, generated by kicad-footprint-generator mountinghole.py")
 		(tags "mountinghole M3")
@@
 		(layer "Edge.Cuts")
 	)
+	(gr_text "Ryan Ling"
+		(at 146 60 0)
+		(layer "F.SilkS")
+		(effects
+			(font
+				(size 1.5 1.5)
+				(thickness 0.3)
+				(bold yes)
+			)
+			(justify left bottom)
+		)
+	)
 	(segment
 		(start 143.34 99)
@@
 	)
 	(segment
+		(start 134.9 68.872774)
+		(end 134.696774 69.076)
+		(width 0.2)
+		(layer "F.Cu")
+		(net 2)
+	)
+	(segment
 		(start 134 74.45)
 		(end 134.55 75)
@@
 	)
 	(segment
-		(start 134.696774 69.076)
-		(end 134.901 68.871774)
-		(width 0.2)
-		(layer "F.Cu")
-		(net 2)
-	)
-	(segment
 		(start 138.45 80.435)
 		(end 141.825 77.06)
@@
 	)
 	(segment
+		(start 134.9 68.5)
+		(end 134.9 68.872774)
+		(width 0.2)
+		(layer "F.Cu")
+		(net 2)
+	)
+	(segment
 		(start 135.112599 73.6)
 		(end 135.2126 73.499999)
@@
 	(segment
 		(start 135.3 65.5)
-		(end 135.3 64.2)
+		(end 135.3 64.3)
 		(width 0.2)
 		(layer "F.Cu")
@@
 	)
 	(segment
-		(start 135.3 64.2)
-		(end 135.2 64.2)
-		(width 0.2)
-		(layer "F.Cu")
-		(net 3)
-	)
-	(segment
-		(start 135.2 64.2)
+		(start 135.3 64.3)
 		(end 133 62)
 		(width 0.2)
@@
 	)
 	(segment
-		(start 131.5 65.5)
-		(end 131.875 65.125)
-		(width 0.2)
-		(layer "F.Cu")
-		(net 4)
-	)
-	(segment
 		(start 131.875 59.5)
 		(end 132 59.5)
@@
 	)
 	(segment
-		(start 130 69.6)
-		(end 135.6 69.6)
+		(start 131.88 66)
+		(end 131.5 66)
 		(width 0.2)
 		(layer "F.Cu")
@@
 	)
 	(segment
-		(start 131.5 66)
-		(end 131.5 65.5)
+		(start 130 69.6)
+		(end 135.6 69.6)
 		(width 0.2)
 		(layer "F.Cu")
@@
 	)
 	(segment
-		(start 131.875 65.125)
-		(end 131.875 59.5)
-		(width 0.2)
-		(layer "F.Cu")
-		(net 4)
-	)
-	(segment
 		(start 131.626 81.526)
 		(end 135 81.526)
@@
 	(segment
 		(start 134 66)
-		(end 131.5 66)
+		(end 131.88 66)
 		(width 0.2)
 		(layer "F.Cu")
@@
 	)
 	(segment
+		(start 131.875 59.5)
+		(end 131.875 65.995)
+		(width 0.2)
+		(layer "F.Cu")
+		(net 4)
+	)
+	(segment
 		(start 130.6 80.5)
 		(end 131.626 81.526)
@@
 	)
 	(segment
+		(start 131.875 65.995)
+		(end 131.88 66)
+		(width 0.2)
+		(layer "F.Cu")
+		(net 4)
+	)
+	(segment
 		(start 135 80.074)
 		(end 135 81.526)
@@
 	)
 	(segment
-		(start 137.68 61.82)
-		(end 141.825 61.82)
+		(start 137.825 55.5)
+		(end 137.825 56.325)
 		(width 0.2)
 		(layer "F.Cu")
@@
 	)
 	(segment
-		(start 137.5 62)
-		(end 137.68 61.82)
+		(start 138 67.5)
+		(end 138 61.82)
 		(width 0.2)
 		(layer "F.Cu")
@@
 	)
 	(segment
-		(start 137.825 55.5)
-		(end 137.825 56.325)
+		(start 141.825 61.82)
+		(end 138 61.82)
 		(width 0.2)
 		(layer "F.Cu")
@@
 	(segment
 		(start 137.576 67.5)
-		(end 138.5 67.5)
+		(end 138 67.5)
 		(width 0.2)
 		(layer "F.Cu")
@@
 	)
 	(segment
-		(start 137.825 56.325)
-		(end 139.5 58)
+		(start 138 67.5)
+		(end 138.5 67.5)
 		(width 0.2)
 		(layer "F.Cu")
@@
 	)
 	(segment
-		(start 137.576 67.5)
-		(end 137.576 62.076)
+		(start 137.825 56.325)
+		(end 139.5 58)
 		(width 0.2)
 		(layer "F.Cu")
@@
 		(width 0.2)
 		(layer "F.Cu")
-		(net 14)
-	)
-	(segment
-		(start 137.576 62.076)
-		(end 137.5 62)
-		(width 0.2)
-		(layer "F.Cu")
