File: Spaceport/PCBs/flight-computer/flight-computer/USB-C_Port.kicad_sch (KiCad schematic)
At the start: 5 parts, among them J4 USB_C_Receptacle_USB2.0_16P

Commit message: Revert "Merge branch 'main' of https://github.com/Terrapin-Rocket-Team/SRAD-Avionics"
This reverts commit e5f68e4e525f2a5ad7eebbc917cc2807b67ca5e1, reversing
changes made to 8a40e2e341d8980ca528983581171a8bd9cc0146.
Parts:
- D9: footprint Diode_SMD:D_0805_2012Metric_Pad1.15x1.40mm_HandSolder -> (none)
- R18, R5: footprint Resistor_SMD:R_0603_1608Metric_Pad0.98x0.95mm_HandSolder -> (none)
Changed lines of the file:
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@@
 			)
 		)
-		(property "Footprint" "Diode_SMD:D_0805_2012Metric_Pad1.15x1.40mm_HandSolder"
+		(property "Footprint" ""
 			(at 132.08 68.58 0)
 			(effects
@@
 			)
 		)
-		(property "Footprint" "Resistor_SMD:R_0603_1608Metric_Pad0.98x0.95mm_HandSolder"
+		(property "Footprint" ""
 			(at 132.842 82.55 90)
 			(effects
@@
 			)
 		)
-		(property "Footprint" "Resistor_SMD:R_0603_1608Metric_Pad0.98x0.95mm_HandSolder"
+		(property "Footprint" ""
 			(at 143.002 82.55 90)
 			(effects
