File: Spaceport/PCBs/flight-computer/flight-computer/ESP32.kicad_sch (KiCad schematic)
At the start: 3 parts, among them J6 UART, U9 ESP32-S3-MINI-1-N4R2

Commit message: added more footprints to schematic, started layout (lots of work to go)
Parts:
- J6: footprint Connector_JST:JST_XH_B6B-XH-A_1x04_P2.50mm_Vertical -> Connector_JST:JST_XH_B6B-XH-A_1x06_P2.50mm_Vertical
- U9: footprint ESP32-S3-MINI-1-N4R2:XCVR_ESP32-S3-MINI-1-N4R2 -> RF_Module:ESP32-S2-MINI-1
Changed lines of the file:
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@@
 			)
 		)
-		(property "Footprint" "Connector_JST:JST_XH_B6B-XH-A_1x04_P2.50mm_Vertical"
+		(property "Footprint" "Connector_JST:JST_XH_B6B-XH-A_1x06_P2.50mm_Vertical"
 			(at 181.61 49.53 0)
 			(effects
@@
 			)
 		)
-		(property "Footprint" "ESP32-S3-MINI-1-N4R2:XCVR_ESP32-S3-MINI-1-N4R2"
+		(property "Footprint" "RF_Module:ESP32-S2-MINI-1"
 			(at 135.89 68.58 0)
 			(effects
