File: Spaceport/PCBs/flight-computer/flight-computer/GPS.kicad_sc.kicad_sch (KiCad schematic)
At the start: 2 parts, among them U1 SAM-M10Q-00B

Commit message: added stm32
Connections:
- no-connect marks 3 -> 6
Changed lines of the file:
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@@
+	)
+	(no_connect
+		(at 138.43 74.93)
 	)
 	(no_connect
@@
 	)
 	(no_connect
+		(at 138.43 90.17)
+	)
+	(no_connect
 		(at 92.71 74.93)
 	)
+	(no_connect
+		(at 138.43 87.63)
+	)
 	(wire

Commit message: added external I2C, SPI, SWD, UART connectors, cleaned up schematics, and changed STM32 schematic for one with power pins. Need to add decoupling capacitors for STM32, external clock for STM32
Connections:
- net SCL renamed I2C1_SCL
- net SDA renamed I2C1_SDA
Changed lines of the file:
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@@
 		)
 	)
-	(global_label "SCL"
+	(global_label "I2C1_SCL"
 		(shape input)
 		(at 138.43 82.55 0)
@@
 		)
 		(property "Intersheetrefs" "${INTERSHEET_REFS}"
-			(at 144.9228 82.55 0)
+			(at 150.1842 82.55 0)
 			(effects
 				(font
@@
 		)
 	)
-	(global_label "SDA"
+	(global_label "I2C1_SDA"
 		(shape bidirectional)
 		(at 138.43 80.01 0)
@@
 		)
 		(property "Intersheetrefs" "${INTERSHEET_REFS}"
-			(at 146.0946 80.01 0)
+			(at 151.356 80.01 0)
 			(effects
 				(font

Commit message: Added LEDS, Buzzer, Oscillator, decoupling capacitors, fixed 3.3 volt netclasses, reorganized main schematic page, added some annotations
Connections:
- net +3.3V renamed +3V3
Changed lines of the file:
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@@
+	(wire
+		(pts
+			(xy 148.59 69.85) (xy 153.67 69.85)
+		)
+		(stroke
+			(width 0)
+			(type default)
+		)
+	)
 	(wire
 		(pts
@@
 	(wire
 		(pts
-			(xy 148.59 69.85) (xy 148.59 95.25)
+			(xy 153.67 69.85) (xy 153.67 95.25)
 		)
 		(stroke
@@
 	(wire
 		(pts
-			(xy 148.59 95.25) (xy 142.24 95.25)
+			(xy 142.24 95.25) (xy 153.67 95.25)
 		)
 		(stroke
@@
 				(path "/b419aaf0-5349-42bc-a414-d94cafbe45e9/d5f88fd8-f77f-45f2-a5f4-fb1e7853b7c3"
 					(reference "C?")
+					(unit 1)
+				)
+			)
+		)
+	)
+	(symbol
+		(lib_id "power:+3V3")
+		(at 146.05 60.96 0)
+		(unit 1)
+		(exclude_from_sim no)
+		(in_bom yes)
+		(on_board yes)
+		(dnp no)
+		(fields_autoplaced yes)
+		(property "Reference" "#PWR049"
+			(at 146.05 64.77 0)
+			(effects
+				(font
+					(size 1.27 1.27)
+				)
+				(hide yes)
+			)
+		)
+		(property "Value" "+3V3"
+			(at 146.05 55.88 0)
+			(effects
+				(font
+					(size 1.27 1.27)
+				)
+			)
+		)
+		(property "Footprint" ""
+			(at 146.05 60.96 0)
+			(effects
+				(font
+					(size 1.27 1.27)
+				)
+				(hide yes)
+			)
+		)
+		(property "Datasheet" ""
+			(at 146.05 60.96 0)
+			(effects
+				(font
+					(size 1.27 1.27)
+				)
+				(hide yes)
+			)
+		)
+		(property "Description" "Power symbol creates a global label with name \"+3V3\""
+			(at 146.05 60.96 0)
+			(effects
+				(font
+					(size 1.27 1.27)
+				)
+				(hide yes)
+			)
+		)
+		(pin "1"
+		)
+		(instances
+			(project ""
+				(path "/b419aaf0-5349-42bc-a414-d94cafbe45e9/d5f88fd8-f77f-45f2-a5f4-fb1e7853b7c3"
+					(reference "#PWR049")
 					(unit 1)
 				)
@@
 					(unit 1)
 				)
-			)
-		)
-	)
-	(symbol
-		(lib_id "power:+3.3V")
-		(at 146.05 60.96 0)
-		(unit 1)
-		(exclude_from_sim no)
-		(in_bom yes)
-		(on_board yes)
-		(dnp no)
-		(property "Reference" "#PWR0102"
-			(at 146.05 64.77 0)
-			(effects
-				(font
-					(size 1.27 1.27)
-				)
-				(hide yes)
-			)
-		)
-		(property "Value" "+3.3V"
-			(at 146.05 55.88 0)
-			(effects
-				(font
-					(size 1.27 1.27)
-				)
-			)
-		)
-		(property "Footprint" ""
-			(at 146.05 60.96 0)
-			(effects
-				(font
-					(size 1.27 1.27)
-				)
-				(hide yes)
-			)
-		)
-		(property "Datasheet" ""
-			(at 146.05 60.96 0)
-			(effects
-				(font
-					(size 1.27 1.27)
-				)
-				(hide yes)
-			)
-		)
-		(property "Description" "Power symbol creates a global label with name \"+3.3V\""
-			(at 146.05 60.96 0)
-			(effects
-				(font
-					(size 1.27 1.27)
-				)
-				(hide yes)
-			)
-		)
-		(pin "1"
-		)
-		(instances
-			(project "GPS.kicad_sc"
-				(path "/13dbe8fb-eb72-456b-8450-e5b1c8c3b2c0"
-					(reference "#PWR03")
-					(unit 1)
-				)
-			)
-			(project "flight-computer"
-				(path "/b419aaf0-5349-42bc-a414-d94cafbe45e9/d5f88fd8-f77f-45f2-a5f4-fb1e7853b7c3"
-					(reference "#PWR0102")
-					(unit 1)
-				)

Commit message: push for schematic review
Connections:
- net +3V3 renamed +3V3A
Changed lines of the file:
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@@
 			)
 		)
-		(property "Value" "+3V3"
-			(at 146.05 55.88 0)
+		(property "Value" "+3V3A"
+			(at 148.59 59.6899 0)
 			(effects
 				(font
 					(size 1.27 1.27)
 				)
+				(justify left)
 			)
 		)

Commit message: removed SdCard
Parts:
- added C18: 100 nF, symbol Device:C
- renumbered C1 to C?
Connections:
- net +3V3A: now also C18.1
- net GND: now also C18.2

Commit message: added footprints and fixed 3.3v/gnd connector orientation
Parts:
- C18, C?: footprint (none) -> Capacitor_SMD:C_0603_1608Metric_Pad1.08x0.95mm_HandSolder
- U1: footprint SAM-M10Q-00B:XCVR_SAM-M10Q-00B -> SAM-M10Q:XCVR_SAM-M10Q-00B
Changed lines of the file:
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@@
 			)
 		)
-		(property "Footprint" ""
+		(property "Footprint" "Capacitor_SMD:C_0603_1608Metric_Pad1.08x0.95mm_HandSolder"
 			(at 169.8752 72.39 0)
 			(effects
@@
 			)
 		)
-		(property "Footprint" ""
+		(property "Footprint" "Capacitor_SMD:C_0603_1608Metric_Pad1.08x0.95mm_HandSolder"
 			(at 155.9052 72.39 0)
 			(effects
@@
 	(symbol
 		(lib_id "power:+3V3")
-		(at 176.53 64.77 270)
-		(unit 1)
-		(exclude_from_sim no)
-		(in_bom yes)
-		(on_board yes)
-		(dnp no)
-		(fields_autoplaced yes)
+		(at 176.53 64.77 0)
+		(unit 1)
+		(exclude_from_sim no)
+		(in_bom yes)
+		(on_board yes)
+		(dnp no)
 		(property "Reference" "#PWR049"
-			(at 172.72 64.77 0)
+			(at 176.53 68.58 0)
 			(effects
 				(font
@@
 		)
 		(property "Value" "+3V3A"
-			(at 180.34 64.7699 90)
+			(at 173.228 60.9599 0)
 			(effects
 				(font
@@
 			)
 		)
-		(property "Footprint" "SAM-M10Q-00B:XCVR_SAM-M10Q-00B"
+		(property "Footprint" "SAM-M10Q:XCVR_SAM-M10Q-00B"
 			(at 115.57 80.01 0)
 			(effects

Commit message: added more footprints to schematic, started layout (lots of work to go)
Parts:
- gave numbers to parts that had none: 1
- renumbered U1 to U5
Changed lines of the file:
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@@
 		(on_board yes)
 		(dnp no)
-		(property "Reference" "C?"
+		(property "Reference" "C24"
 			(at 172.72 67.3099 0)
 			(effects
@@
 			(project "flight-computer"
 				(path "/b419aaf0-5349-42bc-a414-d94cafbe45e9/d5f88fd8-f77f-45f2-a5f4-fb1e7853b7c3"
-					(reference "C?")
+					(reference "C24")
 					(unit 1)
 				)
@@
 		(dnp no)
 		(fields_autoplaced yes)
-		(property "Reference" "U?"
+		(property "Reference" "U5"
 			(at 115.57 57.15 0)
 			(effects
@@
 			(project "flight-computer"
 				(path "/b419aaf0-5349-42bc-a414-d94cafbe45e9/d5f88fd8-f77f-45f2-a5f4-fb1e7853b7c3"
-					(reference "U?")
-					(unit 1)
-				)
+					(reference "U5")
+					(unit 1)
+				)
