File: Spaceport/PCBs/flight-computer/flight-computer/Power.kicad_sch (KiCad schematic)
At the start: 25 parts, among them U5 AZ1084CD-3.3TRG1, U6 TPS62A03DRLR

Commit message: push for schematic review
Parts:
- removed C24: 22uF, symbol Device:C
- removed R10, R11: 150, symbol Device:R
- removed U5: AZ1084CD-3.3TRG1, TO-252-3_6P6X6P1_DIO, symbol SRAD-Avionics:AZ1084CD-3.3TRG1
- added IC1, IC2: AP7362-33SP-13, SOIC127P600X150-9N, symbol SRAD-Avionics:AP7362-33SP-13
- added J10, J9: Conn_01x02, symbol Connector_Generic:Conn_01x02
- added L4: 1.8uH, symbol Device:L
- C23: value 10uF -> 56pF
- L3: value L -> 1uH
- R13: value 110k -> 113k
- R16: value 649k -> 500k
Connections:
- net 5V: now also L4.2
- net GND: now also IC1.1 (GND), IC1.2 (EN), IC1.9 (EP), IC2.1 (GND), IC2.2 (EN), IC2.9 (EP), J10.1 (Pin_1), J9.1 (Pin_1)
- net 4.5V renamed 3.6V
- net 3.6V: now also IC1.3 (IN_1), IC1.4 (IN_2), IC2.3 (IN_1), IC2.4 (IN_2); no longer C23.1
- new net: C23.1, J10.2 (Pin_2), L4.1
- new net +3V3A: IC1.5 (OUT_1), IC1.6 (OUT_2), IC1.7 (OUT_3)
- new net +3V3B: IC2.5 (OUT_1), IC2.6 (OUT_2), IC2.7 (OUT_3), J9.2 (Pin_2)
- no-connect marks 1 -> 4
Other:
- note added: "CFF is optional"
- note added: "VOUT 3.6V"
- note added: "VOUT 5.04V"
- note removed: "VIN"
- note removed: "VOUT 3.3V"
- note removed: "VOUT 4.5V"
- moved on the sheet: C38, C39, C40, L3, R16, R17, U6

Commit message: removed SdCard
Parts:
- removed C23: 56pF, symbol Device:C
- removed C27, C28: 22uF, symbol Device:C
- added C20: 330uF, symbol Device:C_Polarized
- added C22: 100nF, symbol Device:C
- added C9: 22uF, symbol Device:C
- C26: value 22uF -> 100nF
- C30: value .1uF -> 10uF
- C31: value .1uF -> 100nF
- C38: value C -> DNP
- J10: value Conn_01x02 -> 5.0VOUT
- J9: value Conn_01x02 -> 3.3VOUT
- R13: value 113k -> 111k
- R14: value 28k -> 28.7k
Connections:
- net +3V3B: now also J9.1 (Pin_1); no longer J9.2 (Pin_2)
- net 3.6V: now also IC1.2 (EN), IC2.2 (EN)
- net 5V: now also J10.1 (Pin_1), C20.1, C9.2; no longer PS1.5 (VOUT), R13.1
- net GND: now also J10.2 (Pin_2), J9.2 (Pin_2), C20.2, C22.2, C9.1; no longer IC1.2 (EN), IC2.2 (EN), J10.1 (Pin_1), J9.1 (Pin_1)
- net SW: now also PS1.9 (SW__1)
- net at L4.1: now also PS1.5 (VOUT), R13.1; no longer J10.2 (Pin_2)
- net BAT+ renamed BAT_CHARGER
- net BAT_CHARGER: now also C22.1
- no-connect marks 4 -> 3
Other:
- moved on the sheet: C25, C26, C29, C30, C31, C32, C38, C39, C40, IC1, IC2, J10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

Commit message: added footprints and fixed 3.3v/gnd connector orientation
Parts:
- C20: footprint (none) -> Capacitor_SMD:C_1210_3225Metric_Pad1.33x2.70mm_HandSolder
- C22, C25, C26, C29, C30, C31, C32, C39, C40, C9: footprint (none) -> Capacitor_SMD:C_0603_1608Metric_Pad1.08x0.95mm_HandSolder
- C38: now not fitted
- J10, J9: footprint (none) -> Connector_JST:JST_XH_B2B-XH-A_1x02_P2.50mm_Vertical
- L1, L3, L4: footprint (none) -> Inductor_SMD:L_0805_2012Metric_Pad1.05x1.20mm_HandSolder
- PS1: footprint TPS61288LRQQR:CONV_TPS61288LRQQR -> Package_DFN_QFN:Texas_VQFN-HR-20_3x2.5mm_P0.5mm_RQQ0011A
- R12, R13, R14, R16, R17: footprint (none) -> Resistor_SMD:R_0603_1608Metric_Pad0.98x0.95mm_HandSolder
- U6: footprint DRL0006A-MFG -> Package_TO_SOT_SMD:SOT-563
Other:
- moved on the sheet: C20, C26, C9, J9

Commit message: added more footprints to schematic, started layout (lots of work to go)
Parts:
- IC1, IC2: footprint SOIC127P600X150-9N -> Package_SO:Diodes_SO-8EP
Changed lines of the file:
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@@
 			)
 		)
-		(property "Footprint" "SOIC127P600X150-9N"
+		(property "Footprint" "Package_SO:Diodes_SO-8EP"
 			(at 251.46 230.81 0)
 			(effects
@@
 			)
 		)
-		(property "Footprint" "SOIC127P600X150-9N"
+		(property "Footprint" "Package_SO:Diodes_SO-8EP"
 			(at 251.46 195.25 0)
 			(effects

Commit message: schematic change notes
Other:
- note added: "KV 11/25 - Made footprint DNP"
Changed lines of the file:
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@@
+	)
+	(rectangle
+		(start 97.79 120.65)
+		(end 97.79 129.54)
+		(stroke
+			(width 0)
+			(type default)
+		)
+		(fill
+			(type none)
+		)
 	)
 	(rectangle
@@
 		(effects
 			(font
+				(size 1.27 1.27)
+			)
+		)
+	)
+	(text "KV 11/25 - Made footprint DNP\n"
+		(exclude_from_sim no)
+		(at 101.092 118.364 0)
+		(effects
+			(font

Commit message: more changes for FC Board
Parts:
- C20: footprint Capacitor_SMD:C_1210_3225Metric_Pad1.33x2.70mm_HandSolder -> Capacitor_SMD:CP_Elec_10x10
Changed lines of the file:
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@@
 			)
 		)
-		(property "Footprint" "Capacitor_SMD:C_1210_3225Metric_Pad1.33x2.70mm_HandSolder"
+		(property "Footprint" "Capacitor_SMD:CP_Elec_10x10"
 			(at 171.1452 52.07 0)
 			(effects
