File: Spaceport/PCBs/flight-computer/flight-computer/flight-computer.kicad_pcb (KiCad board)
At the start: 4 copper layers, 64.5 x 48.1 mm, 108 parts, among them IC1 AP7362-33SP-13, IC2 AP7362-33SP-13, J1 10067847-001RLF, J10 5.0VOUT, J11 SWD, J12 Charge, J13 Conn_01x02, J2 Conn_01x02, J3 Conn_01x02, J4 USB_C_Receptacle_USB2.0_16P, J5 UART, J6 UART, J7 I2C, J8 SPI, J9 3.3VOUT, U1 MS5611-01BA, U2 BMI088, U3 H3LIS331DL, U4 MMC5603NJ, U5 SAM-M10Q-00B, U6 TPS62A03DRLR, U7 STM32H723VEHx, U8 BQ25606RGER, U9 ESP32-S3-MINI-1-N4R2, Y1 ECS-2520S

Commit message: more routing
Parts:
- removed J1: 10067847-001RLF, Connector_Card:microSD_HC_Wuerth_693072010801
- removed R25: 10kR, Resistor_SMD:R_0603_1608Metric_Pad0.98x0.95mm_HandSolder
- added J14: Micro_SD_Card, Connector_Card:microSD_HC_Wuerth_693072010801, B.Cu at (154.4, 89.3)
- R23, R26, R27, R28: moved to B.Cu
- moved R23 13.4 mm to (156.4, 70.4)
- moved D6 4.11 mm to (125.9, 71.8)
- moved R7 4.11 mm to (129.5, 75.8)
- moved R8 4.11 mm to (129.5, 71.8)
- moved D4 4.11 mm to (125.9, 75.8)
- moved R26 3.09 mm to (167.3, 65.0)
- moved R28 3.09 mm to (164.2, 65.0)
- moved C18 2.87 mm to (144.6, 94.1)
- moved C24 2.83 mm to (143.7, 86.7)
- moved U5 2.59 mm to (148.6, 89.4)
- moved R11 1.02 mm to (161.5, 78.6), turned to 90 degrees
- moved C11 0.76 mm to (159.2, 72.9)
- moved C15 0.76 mm to (163.9, 72.9)
- moved C1 0.12 mm to (157.1, 81.3), turned to -90 degrees
Routing:
- net LED3_PWM: track 0.00 -> 42.9 mm
- net LED1_PWM: track 0.00 -> 42.9 mm
- net ESP_RX: track 6.77 -> 49.0 mm, vias 1 -> 2
- net LED2_PWM: track 0.00 -> 42.0 mm
- net ESP_TX: track 4.25 -> 42.5 mm, vias 0 -> 1
- net SWD_DIO: track 0.00 -> 27.1 mm, vias 0 -> 1
- net EXT_I2C_SCL: track 0.00 -> 25.8 mm
- net SDMMC1_D1: track 0.00 -> 25.7 mm, vias 0 -> 1
- net SDMMC1_D0: track 0.00 -> 25.2 mm, vias 0 -> 1
- net EXT_I2C_SDA: track 0.00 -> 25.1 mm
- net SWD_CLK: track 0.00 -> 25.0 mm, vias 0 -> 1
- net NRST: track 0.00 -> 24.9 mm, vias 0 -> 2
- net EXT_SPI_CS: track 0.00 -> 22.3 mm, vias 0 -> 2
- net SDMMC1_CK: track 0.00 -> 20.9 mm, vias 0 -> 1
- net EXT_SPI_CLK: track 0.00 -> 20.8 mm, vias 0 -> 2
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- added copper zone on In1.Cu, net GND
- added copper zone on In2.Cu, net GND
Other:
- board size 64.5 x 48.1 mm -> 65.1 x 48.6 mm

Commit message: PCB V1 - Needs review
Parts:
- BZ1, C1, C18, C24, J14: moved to F.Cu
- C2, C3, C4, C5, C6, D2, R10, R11, R18, U1, U2, U3, U4, U5: moved to B.Cu
- H1, H2, H3, H4: footprint MountingHole:MountingHole_3.2mm_M3_DIN965_Pad -> MountingHole:MountingHole_3.2mm_M3_DIN965
- moved C5 21.4 mm to (172.7, 78.2), turned to 180 degrees
- moved C4 15.7 mm to (171.8, 81.2), turned to -90 degrees
- moved U3 13.1 mm to (168.8, 80.1), turned to 90 degrees
- moved C18 12.2 mm to (143.2, 82.0)
- moved R18 11.7 mm to (175.5, 52.5), turned to -90 degrees
- moved C2 9.29 mm to (159.3, 86.4), turned to 90 degrees
- moved R5 7.64 mm to (172.6, 52.6)
- moved R10 6.75 mm to (157.5, 79.8), turned to -90 degrees
- moved U2 5.54 mm to (161.9, 86.4), turned to 90 degrees
- moved C1 5.49 mm to (162.5, 80.5), turned to 0 degrees
- moved D2 4.49 mm to (174.3, 59.0)
- moved U1 4.38 mm to (163.0, 80.4), turned to -90 degrees
- moved C6 3.71 mm to (166.4, 84.3), turned to 90 degrees
- moved C10 3.39 mm to (161.0, 69.5), turned to 90 degrees
- moved R26 3.10 mm to (164.2, 65.0)
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Connections:
- U7 pad A2: SDMMC1_D10 -> unconnected-(U7-PC13-PadA2)
- U7 pad H10: unconnected-(U7-PB14-PadH10) -> LED3_PWM
- U7 pad H8: LED3_PWM -> unconnected-(U7-PD14-PadH8)
Routing:
- net +3V3A: track 57.6 -> 215.5 mm, vias 8 -> 20
- net GND: track 247.6 -> 181.0 mm, vias 65 -> 82
- net +3V3B: track 46.7 -> 101.5 mm
- net D+: track 0.49 -> 28.9 mm, vias 1 -> 3
- net D-: track 2.84 -> 30.4 mm, vias 1 -> 3
- net Net-(BZ1-+): track 0.00 -> 26.5 mm, vias 0 -> 2
- net SDMMC1_D2: track 0.63 -> 19.3 mm, vias 1 -> 2
- net SDMMC1_D3: track 1.74 -> 18.9 mm, vias 1 -> 2
- net I2C1_SCL: track 32.7 -> 45.2 mm, vias 3 -> 4
- net I2C1_SDA: track 26.5 -> 37.9 mm, vias 0 -> 1
- net Net-(D9-A): track 0.00 -> 8.62 mm, vias 0 -> 2
- net Net-(J13-Pin_2): track 1.98 -> 10.1 mm, vias 0 -> 1
- net SDMMC1_D1: track 25.7 -> 17.7 mm, vias 1 -> 2
- net SDMMC1_D0: track 25.2 -> 19.1 mm, vias 1 -> 2
- net Net-(U7-PA0): track 0.00 -> 6.00 mm, vias 0 -> 1
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Other:
- board size 65.1 x 48.6 mm -> 65.1 x 49.9 mm

Commit message: Kicad should really have an autosave feature
Routing:
- net GND: track 181.0 -> 187.1 mm, vias 82 -> 83
- net ADC: track 0.00 -> 3.11 mm
- net +3V3A: track 215.5 -> 217.8 mm
- net /Power/5V: track 27.4 -> 29.1 mm
- net Net-(J13-Pin_2): track 10.1 -> 11.5 mm
Changed lines of the file:
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@@
 		(net 6)
 	)
+	(gr_line
+		(start 157.988 69.2404)
+		(end 158.0388 69.7484)
+		(stroke
+			(width 0.2)
+			(type default)
+		)
+		(layer "B.Cu")
+		(net 61)
+	)
+	(gr_line
+		(start 158.0388 69.7484)
+		(end 158.0388 69.7992)
+		(stroke
+			(width 0.2)
+			(type default)
+		)
+		(layer "B.Cu")
+		(net 61)
+	)
+	(gr_line
+		(start 158.0388 69.7992)
+		(end 158.5976 69.7992)
+		(stroke
+			(width 0.2)
+			(type default)
+		)
+		(layer "B.Cu")
+		(net 61)
+	)
+	(gr_line
+		(start 158.0896 69.4436)
+		(end 158.0896 69.6468)
+		(stroke
+			(width 0.2)
+			(type default)
+		)
+		(layer "B.Cu")
+		(net 61)
+	)
+	(gr_line
+		(start 158.5976 69.7992)
+		(end 158.0896 69.4436)
+		(stroke
+			(width 0.2)
+			(type default)
+		)
+		(layer "B.Cu")
+		(net 61)
+	)
+	(gr_line
+		(start 158.0896 69.6468)
+		(end 158.242 69.6976)
+		(stroke
+			(width 0.2)
+			(type default)
+		)
+		(layer "B.Cu")
+		(net 61)
+	)
 	(gr_rect
 		(start 166.2176 71.8312)
@@
 	)
 	(segment
+		(start 154.3214 87.9636)
+		(end 154.3214 90.038334)
+		(width 0.4)
+		(layer "F.Cu")
+		(net 1)
+	)
+	(segment
 		(start 132.5133 63.9778)
 		(end 132.5133 62.4724)
@@
 	)
 	(segment
+		(start 154.3214 90.038334)
+		(end 153.852201 90.507533)
+		(width 0.4)
+		(layer "F.Cu")
+		(net 1)
+	)
+	(segment
 		(start 166.747 95.327831)
 		(end 167.383631 94.6912)
@@
 	)
 	(via
+		(at 170.8404 83.312)
+		(size 0.8)
+		(drill 0.4)
+		(layers "F.Cu" "B.Cu")
+		(net 1)
+	)
+	(via
 		(at 135.5392 59.7101)
 		(size 0.45)
@@
 	)
 	(segment
+		(start 171.7934 82.069168)
+		(end 171.7934 82.359)
+		(width 0.4)
+		(layer "B.Cu")
+		(net 1)
+	)
+	(segment
 		(start 128.0878 75.049)
 		(end 131.3878 75.049)
@@
 	)
 	(segment
+		(start 160.9752 68.6853)
+		(end 162.3296 68.6853)
+		(width 0.4)
+		(layer "B.Cu")
+		(net 1)
+	)
+	(segment
 		(start 163.5201 86.379468)
 		(end 163.1146 86.379468)
@@
 	)
 	(segment
+		(start 162.3296 68.6853)
+		(end 162.5645 68.4504)
+		(width 0.4)
+		(layer "B.Cu")
+		(net 1)
+	)
+	(segment
 		(start 122.7378 68.049)
 		(end 125.871 71.1822)
@@
 	)
 	(segment
+		(start 171.7934 82.359)
+		(end 170.8404 83.312)
+		(width 0.4)
+		(layer "B.Cu")
+		(net 1)
+	)
+	(segment
 		(start 124.6378 68.049)
 		(end 122.7378 68.049)
@@
 	)
 	(segment
-		(start 159.290611 89.4588)
-		(end 160.7846 87.964811)
-		(width 0.4)
-		(layer "F.Cu")
-		(net 3)
-	)
-	(segment
 		(start 145.352201 80.107533)
 		(end 144.088302 81.371432)
@@
 	)
 	(segment
-		(start 152.4666 89.4588)
-		(end 159.290611 89.4588)
+		(start 153.0604 91.3384)
+		(end 157.411011 91.3384)
 		(width 0.4)
 		(layer "F.Cu")
@@
 	)
 	(segment
-		(start 152.1214 89.1136)
-		(end 152.4666 89.4588)
-		(width 0.4)
-		(layer "F.Cu")
-		(net 3)
-	)
-	(segment
 		(start 167.0558 72.5982)
 		(end 167.0558 72.5678)
@@
 	)
 	(segment
+		(start 152.1214 90.3994)
+		(end 153.0604 91.3384)
+		(width 0.4)
+		(layer "F.Cu")
+		(net 3)
+	)
+	(segment
 		(start 164.2738 71.386)
 		(end 164.2738 71.3802)
@@
 	)
 	(segment
+		(start 160.7846 87.964811)
+		(end 160.7846 87.63)
+		(width 0.4)
+		(layer "F.Cu")
+		(net 3)
+	)
+	(segment
 		(start 166.6738 74.5802)
 		(end 167.0978 75.0042)
@@
 	)
 	(segment
-		(start 160.7846 87.964811)
-		(end 160.7846 87.63)
-		(width 0.4)
-		(layer "F.Cu")
-		(net 3)
-	)
-	(segment
 		(start 169.6814 69.7395)
 		(end 167.5145 69.7395)
@@
 	(segment
 		(start 152.1214 87.9636)
-		(end 152.1214 89.1136)
+		(end 152.1214 90.3994)
 		(width 0.4)
 		(layer "F.Cu")
@@
 	)
 	(segment
+		(start 157.411011 91.3384)
+		(end 160.7846 87.964811)
+		(width 0.4)
+		(layer "F.Cu")
+		(net 3)
+	)
+	(segment
 		(start 171.1568 75.6528)
 		(end 171.958 76.454)
@@
 	)
 	(segment
+		(start 142.5689 67.1832)
+		(end 142.5689 65.4983)
+		(width 1)
+		(layer "F.Cu")
+		(net 6)
+	)
+	(segment
 		(start 142.5504 68.7324)
 		(end 142.5504 70.4905)
@@
 	)
 	(segment
+		(start 142.5689 65.4983)
+		(end 142.5504 65.4798)
+		(width 1)
+		(layer "F.Cu")
+		(net 6)
+	)
+	(segment
 		(start 142.5504 67.1068)
 		(end 142.5504 68.0212)
@@
 	(segment
 		(start 157.3598 68.5614)
-		(end 159.9692 71.1708)
+		(end 158.3182 69.5198)
+		(width 0.15)
+		(layer "B.Cu")
+		(net 61)
+	)
+	(segment
+		(start 157.471 70.367)
+		(end 157.3479 70.367)
 		(width 0.15)
 		(layer "B.Cu")
@@
 	)
 	(segment
+		(start 158.3182 69.5198)
+		(end 159.9692 71.1708)
+		(width 0.15)
+		(layer "B.Cu")
+		(net 61)
+	)
+	(segment
 		(start 160.3756 72.1868)
 		(end 161.9504 72.1868)
@@
 	)
 	(segment
+		(start 158.3182 69.5198)
+		(end 157.471 70.367)
+		(width 0.15)
+		(layer "B.Cu")
+		(net 61)
+	)
+	(segment
 		(start 161.9504 72.1868)
 		(end 162.2552 71.882)
@@
 	)
 	(segment
+		(start 164.2316 64.0829)
+		(end 167.3396 64.0829)
+		(width 0.15)
+		(layer "B.Cu")
+		(net 76)
+	)
+	(segment

Commit message: changed SPI pins, rerouted D+/-, moved vias off pads. Silkscreen needs to be fixed still
Parts:
- moved C6 15.3 mm to (156.2, 95.7), turned to 0 degrees
- moved U4 13.1 mm to (157.1, 94.0), turned to 90 degrees
- moved H1 5.54 mm to (130.1, 53.4)
- moved J10 3.20 mm to (122.8, 61.5)
- moved J9 3.20 mm to (122.7, 53.0)
- moved H2 1.98 mm to (130.1, 95.2)
- moved H3 0.89 mm to (183.1, 53.3)
- moved H4 0.63 mm to (183.1, 95.2)
Connections:
- U7 pad A3: unconnected-(U7-PE2-PadA3) -> EXT_SPI_CLK
- U7 pad B10: EXT_SPI_CLK -> unconnected-(U7-PA12-PadB10)
- U7 pad D3: unconnected-(U7-PE5-PadD3) -> EXT_SPI_MISO
- U7 pad E2: EXT_SPI_MISO -> unconnected-(U7-PC2_C-PadE2)
- U7 pad E3: unconnected-(U7-PE6-PadE3) -> EXT_SPI_MOSI
- U7 pad F2: EXT_SPI_MOSI -> unconnected-(U7-PC1-PadF2)
Routing:
- net GND: track 187.1 -> 226.4 mm, vias 83 -> 60
- net +3V3A: track 217.8 -> 234.2 mm
- net /Power/5V: track 29.1 -> 37.7 mm, vias 3 -> 4
- net EXT_SPI_CLK: track 21.7 -> 14.4 mm, vias 0 -> 1
- net I2C1_SDA: track 37.9 -> 43.9 mm, vias 1 -> 3
- net I2C1_SCL: track 45.2 -> 51.0 mm
- net +3V3B: track 101.5 -> 103.0 mm
- net EXT_SPI_MOSI: track 15.1 -> 16.6 mm
- net EXT_SPI_MISO: track 17.1 -> 18.5 mm
- net D+: track 28.9 -> 30.0 mm
- net Net-(U8-TS): track 5.60 -> 4.61 mm
- net BAT_CHARGER: track 19.4 -> 18.8 mm, vias 5 -> 0
Other:
- board size 65.1 x 49.9 mm -> 70.1 x 49.9 mm
- board text removed: "3v3 & 5v out"
- board text removed: "3v3 Buck"
- board text removed: "ESP32"
- board text removed: "LDO"
- board text removed: "LEDS"
- board text removed: "SDCard"
- board text removed: "STM32"

Commit message: more changes
Routing:
- net +3V3B: track 103.0 -> 100.6 mm, vias 3 -> 1
Changed lines of the file:
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@@
 		(net 31)
 	)
-	(via
-		(at 156.0068 76.4032)
-		(size 0.6)
-		(drill 0.3)
-		(layers "F.Cu" "B.Cu")
+	(segment
+		(start 153.6828 76.3817)
+		(end 156.0798 76.3817)
+		(width 1)
+		(layer "F.Cu")
+		(net 33)
+	)
+	(segment
+		(start 153.0604 75.7593)
+		(end 153.6828 76.3817)
+		(width 1)
+		(layer "F.Cu")
+		(net 33)
+	)
+	(segment
+		(start 153.0604 75.0824)
+		(end 153.0604 75.7593)
+		(width 1)
+		(layer "F.Cu")
 		(net 33)
 	)
 	(via
-		(at 154.8384 76.4032)
-		(size 0.6)
+		(at 153.0604 75.0824)
+		(size 0.8)
 		(drill 0.3)
 		(layers "F.Cu" "B.Cu")
-		(net 33)
-	)
-	(via
-		(at 153.4414 76.4032)
-		(size 0.6)
-		(drill 0.3)
-		(layers "F.Cu" "B.Cu")
-		(net 33)
-	)
-	(segment
-		(start 153.0604 76.0222)
-		(end 153.4414 76.4032)
-		(width 1)
-		(layer "B.Cu")
-		(net 33)
-	)
-	(segment
-		(start 153.0604 75.0316)
-		(end 154.432 76.4032)
-		(width 1)
-		(layer "B.Cu")
 		(net 33)
 	)
@@
 	)
 	(segment
-		(start 154.432 76.4032)
-		(end 154.8384 76.4032)
+		(start 153.0604 71.2216)
+		(end 153.0604 75.0824)
 		(width 1)
 		(layer "B.Cu")
@@
 		(start 129.2 58.6)
 		(end 135.816 58.6)
-		(width 1)
-		(layer "B.Cu")
-		(net 33)
-	)
-	(segment
-		(start 153.4414 76.4032)
-		(end 156.0068 76.4032)
 		(width 1)
 		(layer "B.Cu")
@@
 	)
 	(segment
-		(start 153.0604 75.0316)
-		(end 153.0604 76.0222)
-		(width 1)
-		(layer "B.Cu")
-		(net 33)
-	)
-	(segment
 		(start 123.613 53.013)
 		(end 129.2 58.6)
@@
 		(layer "B.Cu")
 		(net 33)
-	)
-	(segment
-		(start 153.0604 71.2216)
-		(end 153.0604 75.0316)
-		(width 1)
-		(layer "B.Cu")
-		(net 33)

Commit message: more changes for FC Board
Parts:
- added C27: 100 nF, Capacitor_SMD:C_0603_1608Metric_Pad1.08x0.95mm_HandSolder, B.Cu at (172.8, 73.7)
- C20: footprint Capacitor_SMD:C_1210_3225Metric_Pad1.33x2.70mm_HandSolder -> Capacitor_SMD:CP_Elec_10x10
- C37: footprint Capacitor_SMD:C_1210_3225Metric_Pad1.33x2.70mm_HandSolder -> Capacitor_SMD:C_0805_2012Metric_Pad1.18x1.45mm_HandSolder
- D2: moved to F.Cu
- moved J9 68.2 mm to (176.8, 94.6)
- moved C20 5.61 mm to (138.0, 75.4)
- moved D2 4.16 mm to (170.7, 61.0), turned to 90 degrees
- moved C37 0.51 mm to (148.8, 61.0)
Connections:
- U8 pad 25: (no net) -> GND
Routing:
- net GND: track 226.4 -> 108.4 mm, vias 60 -> 77
- net +3V3B: track 100.6 -> 90.2 mm
- net +3V3A: track 234.2 -> 243.2 mm, vias 20 -> 18
- net /Power/5V: track 37.7 -> 30.0 mm, vias 4 -> 3
- net (no net): track 2.27 -> 0.00 mm
- net LED1_PWM: track 41.3 -> 43.5 mm
- net I2C1_SCL: track 51.0 -> 49.5 mm, vias 4 -> 3
- net LED2_PWM: track 40.2 -> 41.4 mm
- net D+: track 30.0 -> 29.0 mm, vias 3 -> 2
- net D-: track 30.0 -> 29.2 mm, vias 3 -> 2
- net NRST: track 26.4 -> 27.0 mm, vias 1 -> 2
- net EXT_SPI_MISO: track 18.5 -> 18.0 mm
- net I2C1_SDA: track 43.9 -> 43.4 mm
- added copper zone on F.Cu, net /Power/5V
- added copper zone on B.Cu, net GND
- added copper zone on F.Cu, net GND
Other:
- board size 70.1 x 49.9 mm -> 70.1 x 50.9 mm

Commit message: ofc I forgot to save
Parts:
- removed U4: MMC5603NJ, MMC5603NJ:WLP4_0P82X0P82_MEM
- added C28: 100 nF, Capacitor_SMD:C_0603_1608Metric_Pad1.08x0.95mm_HandSolder, B.Cu at (160.7, 97.2)
- added JP1: 000111X, Jumper:SolderJumper-2_P1.3mm_Open_RoundedPad1.0x1.5mm, B.Cu at (163.2, 98.5)
- added JP10: 0x18, Jumper:SolderJumper-2_P1.3mm_Open_RoundedPad1.0x1.5mm, F.Cu at (167.1, 84.8)
- added JP11: 0x76, Jumper:SolderJumper-2_P1.3mm_Open_RoundedPad1.0x1.5mm, B.Cu at (167.6, 86.9)
- added JP12: 0x77, Jumper:SolderJumper-2_P1.3mm_Open_RoundedPad1.0x1.5mm, B.Cu at (165.1, 86.9)
- added JP2: 000110X, Jumper:SolderJumper-2_P1.3mm_Open_RoundedPad1.0x1.5mm, B.Cu at (163.2, 95.9)
- added JP3: 00011X1, Jumper:SolderJumper-2_P1.3mm_Open_RoundedPad1.0x1.5mm, B.Cu at (151.6, 96.2)
- added JP4: 00011X0, Jumper:SolderJumper-2_P1.3mm_Open_RoundedPad1.0x1.5mm, B.Cu at (151.6, 98.7)
- added JP5: Accel 0x19, Jumper:SolderJumper-2_P1.3mm_Open_RoundedPad1.0x1.5mm, B.Cu at (170.6, 88.4)
- added JP6: Accel 0x18, Jumper:SolderJumper-2_P1.3mm_Open_RoundedPad1.0x1.5mm, B.Cu at (170.6, 91.0)
- added JP7: Gyro 0x69, Jumper:SolderJumper-2_P1.3mm_Open_RoundedPad1.0x1.5mm, B.Cu at (163.2, 90.8)
- added JP8: Accel 0x68, Jumper:SolderJumper-2_P1.3mm_Open_RoundedPad1.0x1.5mm, B.Cu at (163.2, 93.4)
- added JP9: 0x19, Jumper:SolderJumper-2_P1.3mm_Open_RoundedPad1.0x1.5mm, F.Cu at (169.7, 84.8)
- added U10: MLX90393ELW-ABA-xxx-xx, Package_DFN_QFN:QFN-16-1EP_3x3mm_P0.5mm_EP1.75x1.75mm, B.Cu at (157.7, 96.4)
- C6: value 100nF -> 100 nF
- moved C3 4.28 mm to (161.1, 83.7), turned to 0 degrees
- moved C2 3.09 mm to (161.3, 88.8), turned to 180 degrees
- moved C6 1.93 mm to (154.5, 96.5), turned to -90 degrees
- moved U2 0.69 mm to (161.3, 86.3), turned to 180 degrees
- moved J10 0.46 mm to (123.2, 61.5)
Connections:
- U1 pad 4: GND -> Net-(JP11-B)
- U1 pad 5: GND -> Net-(JP11-B)
- U2 pad 10: GND -> Net-(JP7-A)
- U2 pad 15: GND -> Net-(JP5-A)
- U3 pad 7: +3V3A -> Net-(JP10-B)
Routing:
- net +3V3A: track 243.2 -> 270.3 mm
- net Net-(JP5-A): track 0.00 -> 10.7 mm
- net Net-(JP11-B): track 0.00 -> 10.7 mm, vias 0 -> 2
- net Net-(JP7-A): track 0.00 -> 8.90 mm
- net Net-(JP1-A): track 0.00 -> 8.63 mm
- net Net-(JP10-B): track 0.00 -> 8.07 mm, vias 0 -> 1
- net Net-(JP3-A): track 0.00 -> 7.64 mm
- net GND: track 108.4 -> 102.6 mm, vias 77 -> 83
- net Net-(U10-Supply): track 0.00 -> 1.93 mm
- net I2C1_SCL: track 49.5 -> 50.3 mm

Commit message: forgot to add 3v3 connection to new magnetometer
Connections:
- C28 pad 2: Net-(U10-Supply) -> +3V3A
- U10 pad 8: Net-(U10-Supply) -> +3V3A
Routing:
- net +3V3A: track 270.3 -> 277.0 mm
- net Net-(U10-Supply): track 1.93 -> 0.00 mm
Changed lines of the file:
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@@
 	(net 199 "unconnected-(U10-NC-Pad4)")
 	(net 200 "unconnected-(U10-NC-Pad10)")
-	(net 201 "Net-(U10-Supply)")
-	(net 202 "Net-(JP5-A)")
+	(net 201 "Net-(JP5-A)")
 	(footprint "Capacitor_SMD:C_0603_1608Metric_Pad1.08x0.95mm_HandSolder"
 		(layer "F.Cu")
@@
 			(layers "B.Cu" "B.Mask" "B.Paste")
 			(roundrect_rratio 0.25)
-			(net 201 "Net-(U10-Supply)")
+			(net 3 "+3V3A")
 			(pintype "passive")
 		)
@@
 			(size 1 0.5)
 			(layers "B.Cu" "B.Mask")
-			(net 202 "Net-(JP5-A)")
+			(net 201 "Net-(JP5-A)")
 			(pinfunction "A")
 			(pintype "passive")
@@
 			(size 1 0.5)
 			(layers "B.Cu" "B.Mask")
-			(net 202 "Net-(JP5-A)")
+			(net 201 "Net-(JP5-A)")
 			(pinfunction "B")
 			(pintype "passive")
@@
 			(layers "B.Cu" "B.Mask" "B.Paste")
 			(roundrect_rratio 0.25)
-			(net 201 "Net-(U10-Supply)")
+			(net 3 "+3V3A")
 			(pinfunction "Supply")
 			(pintype "power_in")
@@
 			(size 0.35 0.59)
 			(layers "B.Cu" "B.Mask" "B.Paste")
-			(net 202 "Net-(JP5-A)")
+			(net 201 "Net-(JP5-A)")
 			(pinfunction "SDO1")
 			(pintype "output")
@@
 	)
 	(segment
-		(start 164.846 91.758401)
+		(start 164.846 94.7166)
 		(end 164.846 97.529595)
 		(width 0.2)
@@
 	)
 	(segment
+		(start 162.314969 94.7166)
+		(end 164.846 94.7166)
+		(width 0.2)
+		(layer "B.Cu")
+		(net 3)
+	)
+	(segment
 		(start 144.3228 74.4092)
 		(end 136.0638 66.1502)
@@
 	)
 	(segment
+		(start 160.720096 96.311473)
+		(end 162.314969 94.7166)
+		(width 0.2)
+		(layer "B.Cu")
+		(net 3)
+	)
+	(segment
 		(start 161.204944 88.0364)
 		(end 160.442402 88.798942)
@@
 	)
 	(segment
+		(start 159.123326 97.119096)
+		(end 159.912473 97.119096)
+		(width 0.2)
+		(layer "B.Cu")
+		(net 3)
+	)
+	(segment
 		(start 160.442401 88.900541)
 		(end 160.442401 88.798943)
@@
 	)
 	(segment
+		(start 159.912473 97.119096)
+		(end 160.720096 96.311473)
+		(width 0.2)
+		(layer "B.Cu")
+		(net 3)
+	)
+	(segment
 		(start 144.3228 77.5463)
 		(end 145.352201 78.575701)
@@
 	)
 	(segment
+		(start 164.846 91.758401)
+		(end 164.846 94.7166)
+		(width 0.2)
+		(layer "B.Cu")
+		(net 3)
+	)
+	(segment
 		(start 156.7906 61.7438)
 		(end 156.7906 61.2612)
@@
 	)
 	(segment
-		(start 159.123326 97.119096)
-		(end 159.912473 97.119096)
-		(width 0.2)
-		(layer "B.Cu")
-		(net 201)
-	)
-	(segment
-		(start 159.912473 97.119096)
-		(end 160.720096 96.311473)
-		(width 0.2)
-		(layer "B.Cu")
-		(net 201)
-	)
-	(segment
 		(start 169.972001 88.4428)
 		(end 169.977001 88.4478)
 		(width 0.2)
 		(layer "B.Cu")
-		(net 202)
+		(net 201)
 	)
 	(segment
@@
 		(width 0.2)
 		(layer "B.Cu")
-		(net 202)
+		(net 201)
 	)
 	(segment
@@
 		(width 0.2)
 		(layer "B.Cu")
-		(net 202)
+		(net 201)
 	)
 	(segment
@@
 		(width 0.2)
 		(layer "B.Cu")
-		(net 202)
+		(net 201)
 	)
 	(segment
@@
 		(width 0.2)
 		(layer "B.Cu")
-		(net 202)
+		(net 201)
 	)
 	(zone
