File: Spaceport/PCBs/flight-computer/Alternate layout/flight-computer.kicad_pcb (KiCad board)
At the start: 4 copper layers, 65.1 x 53 mm, 113 parts, among them IC1 AP7362-33SP-13, IC2 AP7362-33SP-13, J1 SWD, J10 5.0VOUT, J12 Charge, J13 Conn_01x02, J14 Micro_SD_Card, J2 Conn_01x02, J3 Conn_01x02, J4 USB_C_Receptacle_USB2.0_16P, J5 UART, J6 UART, J7 I2C, J8 SPI, J9 3.3VOUT, U1 MS5611-01BA, U10 MLX90393ELW-ABA-xxx-xx, U2 BMI088, U3 H3LIS331DL, U5 SAM-M10Q-00B, U6 TPS62A03DRLR, U7 STM32H723VEHx, U8 BQ25606RGER, U9 ESP32-S3-MINI-1-N4R2, Y1 ECS-2520S

Commit message: final version of the FC trust
Parts:
- added G***: LOGO, STM32-flight-computer:TRT_Logo, F.Cu at (159.7, 88.6)
- C20: value 220uF -> 220 µF
- C22, C26, C31: value 100nF -> 100 nF
- C25: value 27pF -> 27 pF
- C29: value 620pF -> 620 pF
- C30: value 10uF -> 10 µF
- C32: value 2.2uF -> 2.2 µF
- C34: value 47nF -> 47 nF
- C39, C9: value 22uF -> 22 µF
- C40: value 4.7uF -> 4.7 µF
- C41, C42, C43, C44: value 10µF -> 10 µF
- moved H2 0.10 mm to (190.1, 70.0)
- moved H3 0.10 mm to (190.1, 115.0)
Routing:
- net EXT_SPI_CS: track 27.2 -> 27.3 mm, vias 2 -> 1
Other:
- board text added: "+ CL - DIO RST"
- board text added: "- CL DA +"
- board text added: "- CS CL MISO MOSI +"
- board text added: "- EN RX TX I/O +"
- board text added: "- RX TX +"
- board text added: "Designed By Krish Vyas"
- board text added: "Device May Break If Eaten By Turtles"
- board text added: "Do not put device in contact with rocket hot propellant"
- board text added: "If Text Is Visible, Board Had An Oopsie"
- board text added: "JLCJLCJLCJLC"
- board text added: "Not For Military Use"
- board text added: "TRT FC V1.0"
- board text added: "This Side Down btw"
- board text added: "ZARATAN"
- board text added: "ooo shiny logo"
- board text removed: "+ DA CL -"
- board text removed: "+ I/O TX RX EN -"
- board text removed: "+ MOSI MOSI CL CS -"
- board text removed: "+ TX RX -"
- board text removed: "RST DIO - CL +"

Commit message: moved some silkscreen components around
Other:
- board text added: "Do not put device in contact with hot rocket propellant"
- board text removed: "Do not put device in contact with rocket hot propellant"

Commit message: Add R27 resistor to BMS and update PCB layout
This was rushed, so my solution is clapped. I do think there will be some interference between the Bat+ track and the Vset track. Uncommit these changes to change the pcb, but the schematic does need at least a 51K ohm resistor.
Parts:
- added R27: 60K, Resistor_SMD:R_0603_1608Metric_Pad0.98x0.95mm_HandSolder, F.Cu at (149.3, 78.9)
- moved C36 4.11 mm to (147.6, 82.3)
- moved R15 0.70 mm to (143.1, 77.6)
- moved D7 0.39 mm to (144.6, 82.5)
- moved R20 0.10 mm to (143.6, 79.4)
- moved R4 0.05 mm to (146.0, 78.7)
Connections:
- U8 pad 12: unconnected-(U8-VSET-Pad12) -> Net-(U8-VSET)
Routing:
- net GND: track 43.1 -> 52.5 mm
- net BAT+: track 40.0 -> 44.8 mm
- net Net-(U8-VSET): track 0.00 -> 1.78 mm
- net Net-(U8-STAT): track 2.80 -> 3.55 mm
- net Net-(D1-K): track 4.28 -> 3.70 mm

Commit message: changes
still need to fix silkscreen but removed ground traces
Routing:
- net GND: track 52.5 -> 43.1 mm
Changed lines of the file:
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@@
 		(tags "resistor handsolder")
 		(property "Reference" "R4"
-			(at -2.5908 0.094 90)
+			(at -2.62 0.29 90)
 			(layer "F.SilkS")
 			(effects
@@
 		(tags "resistor handsolder")
 		(property "Reference" "R27"
-			(at 0 -1.43 90)
+			(at 0.08 -1.25 270)
 			(layer "F.SilkS")
 			(effects
@@
 	)
 	(segment
-		(start 148.22 83.122501)
-		(end 151.6204 79.722101)
-		(width 0.2)
-		(layer "F.Cu")
-		(net 1)
-	)
-	(segment
 		(start 167.2392 100.575901)
 		(end 167.2392 99.4461)
@@
 	)
 	(segment
-		(start 151.6204 79.722101)
-		(end 151.6204 78.5607)
-		(width 0.2)
-		(layer "F.Cu")
-		(net 1)
-	)
-	(segment
 		(start 168.4031 91.3368)
 		(end 168.9624 91.3368)
@@
 	)
 	(segment
-		(start 147.61 83.122501)
-		(end 148.22 83.122501)
-		(width 0.2)
-		(layer "F.Cu")
-		(net 1)
-	)
-	(segment
 		(start 182.5624 87.6221)
 		(end 182.2704 87.330101)
@@
 	)
 	(segment
-		(start 149.28 79.8025)
-		(end 150.3786 79.8025)
-		(width 0.2)
-		(layer "F.Cu")
-		(net 1)
-	)
-	(segment
 		(start 181.61 86.6697)
 		(end 181.61 85.4701)
@@
 		(layer "F.Cu")
 		(net 1)
-	)
-	(segment
-		(start 150.3786 79.8025)
-		(end 151.6204 78.5607)
-		(width 0.2)
-		(layer "F.Cu")
-		(net 1)

Commit message: Changed silkscreen
Parts:
- moved C36 1.54 mm to (149.1, 82.1)
- moved R15 0.60 mm to (143.7, 77.6)
- moved R27 0.27 mm to (149.1, 78.7)
- moved R20 0.12 mm to (143.8, 79.4)
- moved R4 0.10 mm to (146.1, 78.7)
- turned R26 to 0 degrees
Routing:
- net BAT+: track 44.8 -> 42.0 mm
- net Net-(U7-PA2): track 16.2 -> 17.7 mm

Commit message: removed all global labels
Parts:
- moved D7 0.27 mm to (144.6, 82.2)
Connections:
- net BAT+ renamed /VSENSE
- net BAT_CHARGER renamed /Battery Charger/BAT_OUT
- net D+ renamed /USB-C_Port/D+
- net D- renamed /USB-C_Port/D-
- net ESP_RX renamed /ESP32/RX
- net ESP_TX renamed /ESP32/TX
- net EXT_I2C_SCL renamed /EXT_I2C_SCL
- net EXT_I2C_SDA renamed /EXT_I2C_SDA
- net EXT_SPI_CLK renamed /EXT_SPI_CLK
- net EXT_SPI_CS renamed /EXT_SPI_CS
- net EXT_SPI_MISO renamed /EXT_SPI_MISO
- net EXT_SPI_MOSI renamed /EXT_SPI_MOSI
- net EXT_UART_RX renamed /EXT_UART_RX
- net EXT_UART_TX renamed /EXT_UART_TX
- net I2C1_SCL renamed /Barometer/I2C_SCL
- net I2C1_SDA renamed /Barometer/I2C_SDA
- net LED1_PWM renamed /LED1_PWM
- net LED2_PWM renamed /LWD2_PWM
- net LED3_PWM renamed /LED3_PWM
- net NRST renamed /RST
- net SDMMC1_CK renamed /SDCard/SCLK
- net SDMMC1_CMD renamed /SDMMC_CMD
- net SDMMC1_D0 renamed /SDCard/D0
- net SDMMC1_D1 renamed /SDCard/D1
- net SDMMC1_D2 renamed /SDCard/D2
- net SDMMC1_D3 renamed /SDCard/D3
- net SWD_CLK renamed /SWD_CLK
- net SWD_DIO renamed /SWD_DIO
Other:
- board text added: "BAT CHARGE +"
- board text removed: "USB 5V +"

Commit message: silkscreen changes
Routing:
- net Net-(U8-~{PG}): track 4.24 -> 3.73 mm
Other:
- board text added: "DO NOT USE BAT CHARGE CONNECTOR WHEN USB IS CONNECTED"
- board text removed: "ooo shiny logo"

Commit message: started on the current sense circuitry, updated prod files
Connections:
- C22 pad 1: /Battery Charger/BAT_OUT -> /Power/BAT_IN
- C30 pad 1: /Battery Charger/BAT_OUT -> /Power/BAT_IN
- J4 pad A5: Net-(J4-CC2) -> Net-(J4-CC1)
- J4 pad B5: Net-(J4-CC1) -> Net-(J4-CC2)
- L1 pad 1: /Battery Charger/BAT_OUT -> /Power/BAT_IN
- PS1 pad 6: /Battery Charger/BAT_OUT -> /Power/BAT_IN
- PS1 pad 7: /Battery Charger/BAT_OUT -> /Power/BAT_IN
Routing:
- net /VSENSE: track 42.0 -> 42.5 mm
Changed lines of the file:
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@@
 	(net 193 "/Barometer/I2C_SCL")
 	(net 194 "/Barometer/I2C_SDA")
+	(net 195 "/Power/BAT_IN")
 	(footprint "Connector_JST:JST_XH_B2B-XH-A_1x02_P2.50mm_Vertical"
 		(layer "F.Cu")
@@
 			(layers "F.Cu" "F.Mask" "F.Paste")
 			(roundrect_rratio 0.188679)
-			(net 9 "/Battery Charger/BAT_OUT")
+			(net 195 "/Power/BAT_IN")
 			(pintype "passive")
 		)
@@
 			(layers "F.Cu" "F.Mask" "F.Paste")
 			(roundrect_rratio 0.188679)
-			(net 9 "/Battery Charger/BAT_OUT")
+			(net 195 "/Power/BAT_IN")
 			(pintype "passive")
 		)
@@
 			(layers "F.Cu" "F.Mask" "F.Paste")
 			(roundrect_rratio 0.25)
-			(net 9 "/Battery Charger/BAT_OUT")
+			(net 195 "/Power/BAT_IN")
 			(pinfunction "EN")
 			(pintype "input")
@@
 			(layers "F.Cu" "F.Mask" "F.Paste")
 			(roundrect_rratio 0.25)
-			(net 9 "/Battery Charger/BAT_OUT")
+			(net 195 "/Power/BAT_IN")
 			(pinfunction "VIN")
 			(pintype "input")
@@
 			(layers "F.Cu" "F.Mask" "F.Paste")
 			(roundrect_rratio 0.25)
-			(net 9 "/Battery Charger/BAT_OUT")
+			(net 195 "/Power/BAT_IN")
 			(pinfunction "VIN")
 			(pintype "input")
@@
 			(size 2 3.4)
 			(layers "F.Cu" "F.Mask" "F.Paste")
-			(net 9 "/Battery Charger/BAT_OUT")
+			(net 195 "/Power/BAT_IN")
 			(pinfunction "1")
 			(pintype "passive")
@@
 			(layers "F.Cu" "F.Mask" "F.Paste")
 			(roundrect_rratio 0.25)
-			(net 191 "Net-(J4-CC2)")
+			(net 43 "Net-(J4-CC1)")
 			(pinfunction "CC1")
 			(pintype "bidirectional")
@@
 			(layers "F.Cu" "F.Mask" "F.Paste")
 			(roundrect_rratio 0.25)
-			(net 43 "Net-(J4-CC1)")
+			(net 191 "Net-(J4-CC2)")
 			(pinfunction "CC2")
 			(pintype "bidirectional")
@@
 	)
 	(segment
-		(start 149.956 80.381499)
-		(end 149.14 81.197499)
-		(width 0.2)
+		(start 150.225 77.171763)
+		(end 149.717838 76.664601)
+		(width 0.7)
 		(layer "F.Cu")
 		(net 20)
@@
 	)
 	(segment
-		(start 149.956 76.902763)
-		(end 149.956 80.381499)
-		(width 0.2)
+		(start 149.14 81.197499)
+		(end 150.225 80.112499)
+		(width 0.7)
 		(layer "F.Cu")
 		(net 20)
@@
 		(net 20)
 	)
+	(segment
+		(start 150.225 80.112499)
+		(end 150.225 77.171763)
+		(width 0.7)
+		(layer "F.Cu")
+		(net 20)
+	)
 	(via
 		(at 149.606 76.0984)
@@
 	)
 	(segment
-		(start 141.465601 75.694599)
-		(end 138.5344 78.6258)
-		(width 0.7)
+		(start 138.5344 78.6258)
+		(end 141.465601 75.694599)
+		(width 2)
 		(layer "F.Cu")
 		(net 30)
 	)
 	(segment
-		(start 143.3842 75.694599)
-		(end 141.465601 75.694599)
-		(width 0.7)
+		(start 141.465601 75.694599)
+		(end 143.4858 75.694599)
+		(width 2)
 		(layer "F.Cu")
 		(net 30)
@@
 		(polygon
 			(pts
-				(xy 143.1544 71.2724) (xy 146.2024 71.2724) (xy 146.2024 71.882) (xy 146.6088 71.882) (xy 146.6088 72.898)
-				(xy 146.1008 72.898) (xy 146.1008 73.3552) (xy 144.9832 73.3552) (xy 144.9832 74.2696) (xy 143.1544 74.2696)
+				(xy 142.5044 71.2724) (xy 146.2024 71.2724) (xy 146.2024 71.882) (xy 146.6088 71.882) (xy 146.6088 72.898)
+				(xy 146.1008 72.898) (xy 146.1008 73.3552) (xy 144.9832 73.3552) (xy 144.9832 74.2696) (xy 142.5044 74.2696)
 			)
 		)
