File: Spaceport/PCBs/flight-computer/Alternate layout/flight-computer.kicad_sch (KiCad schematic)
At the start: 42 parts, among them J1 SWD, J13 Conn_01x02, J2 Conn_01x02, J3 Conn_01x02, J5 UART, J7 I2C, J8 SPI, U7 STM32H723VEHx, Y1 ECS-2520S

Commit message: Inductor changes, DRC checks, Silkscreen changes, BOM
Parts:
- C11: value 2.2uF -> 2.2 µF
- C12, C13, C14, C15, C17, C19, C21, C23, C27: value 100nF -> 100 nF
- R1, R10, R11, R2: value 10k -> 10 kΩ
- R23: value 10kR -> 10 kΩ
- R26, R27, R28: value 170R -> 170 RΩ
- R6, R7, R8, R9: value 110R -> 110 Ω

Commit message: Changes requested by Joseph
Parts:
- added NT1: NetTie_2, NetTie:NetTie-2_SMD_Pad0.5mm, symbol Device:NetTie_2
- BZ1: footprint Buzzer_Beeper:Buzzer_TDK_PS1240P02BT_D12.2mm_H6.5mm -> TRT-Avionics:Adafruit_5V_Buzzer
Connections:
- net GND: now also NT1.2; no longer R23.2, U7.F7 (PDR_ON)
- new net: NT1.1, R23.2, U7.F7 (PDR_ON)

Commit message: silkscreen changes + minor layout changes
Parts:
- removed R28: 170 RΩ, Resistor_SMD:R_0603_1608Metric_Pad0.98x0.95mm_HandSolder, symbol Device:R
- added R24: 78.7 kΩ, Resistor_SMD:R_0603_1608Metric_Pad0.98x0.95mm_HandSolder, symbol Device:R
- R10, R11: value 10 kΩ -> 5.1 kΩ
- R26: value 170 RΩ -> 47 kΩ
Connections:
- net ADC: no longer R26.2
- net BAT+: now also R26.2
- net GND: now also R24.1
- net at R26.1, U7.J2 (PA2): now also R24.2
- no-connect marks 52 -> 53
Other:
- moved on the sheet: R10, R11, R26

Commit message: removed unneded resistor
Parts:
- removed R27: 170 RΩ, Resistor_SMD:R_0603_1608Metric_Pad0.98x0.95mm_HandSolder, symbol Device:R
Connections:
- no-connect marks 53 -> 54

Commit message: starting current monitoring
 I'm thinking of creating a small circuit near where the BAT+ enters into the screw switch. I'll have two diff nets, a shunt resistor, and then a high side op amp current sensing circuit
Parts:
- added R25: R, symbol Device:R
Connections:
- net BAT+: now also R25.2; no longer J3.1 (Pin_1)
- new net BAT+_LOAD: J3.1 (Pin_1), R25.1
- no-connect marks 54 -> 53

Commit message: Add R27 resistor to BMS and update PCB layout
This was rushed, so my solution is clapped. I do think there will be some interference between the Bat+ track and the Vset track. Uncommit these changes to change the pcb, but the schematic does need at least a 51K ohm resistor.
Parts:
- removed R25: R, symbol Device:R
Connections:
- net BAT+_LOAD is gone; now on net BAT+: J3.1 (Pin_1)
- no-connect marks 53 -> 54

Commit message: removed all global labels
Parts:
- removed J2, J3: Conn_01x02, Connector_JST:JST_XH_B2B-XH-A_1x02_P2.50mm_Vertical, symbol Connector_Generic:Conn_01x02
Connections:
- net BAT+ renamed VSENSE
- net D+ renamed USB-C_Port/D+
- net D- renamed USB-C_Port/D-
- net ESP_RX renamed ESP32/RX
- net ESP_TX renamed ESP32/TX
- net I2C1_SCL renamed Barometer/I2C_SCL
- net I2C1_SDA renamed Barometer/I2C_SDA
- net LED2_PWM renamed LWD2_PWM
- net NRST renamed RST
- net SDMMC1_CK renamed SDCard/SCLK
- net SDMMC1_CMD renamed SDMMC_CMD
- net SDMMC1_D0 renamed SDCard/D0
- net SDMMC1_D1 renamed SDCard/D1
- net SDMMC1_D2 renamed SDCard/D2
- net SDMMC1_D3 renamed SDCard/D3
Other:
- sheet Barometer ports: added I2C_SCL, I2C_SDA; removed none
- sheet Battery Charger ports: added BAT_OUT, VSENSE; removed none
- sheet ESP32 ports: added RX, TX; removed none
- sheet GPS ports: added I2C_SCL, I2C_SDA; removed none
- sheet High-g-IMU ports: added I2C_SCL, I2C_SDA; removed none
- sheet IMU ports: added I2C_SCL, I2C_SDA; removed none
- sheet Magnetometer ports: added I2C_SCL, I2C_SDA; removed none
- sheet Power ports: added BAT_IN; removed none
- sheet SDCard ports: added CMD, D0, D1, D2, D3, SCLK; removed none
- sheet USB-C_Port ports: added D+, D-; removed none
- note removed: "According to datasheet, any pin with FT_ha can be changed (in code) to an analog option. For 16 bit resolution, it's recommended to use 170 ohm resistor in series"
- note removed: "BATTERY | SCREW SWITCH"
- note removed: "KV 11/25 - Changed switch to jumper"
- note removed: "KV 11/25 - Removed D10 Global label"
- moved on the sheet: NT1, R1, R2, R24, R26

Commit message: started on the current sense circuitry, updated prod files
Other:
- sheet Battery Charger ports: added BAT+; removed VSENSE
