File: Spaceport/PCBs/flight-computer/Alternate layout/Barometer.kicad_sc.kicad_sch (KiCad schematic)
At the start: 2 parts, among them U1 MS5611-01BA

Commit message: Inductor changes, DRC checks, Silkscreen changes, BOM
Parts:
- C1: value 100nF -> 100 nF
Changed lines of the file:
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@@
 			)
 		)
-		(property "Value" "100nF"
+		(property "Value" "100 nF"
 			(at 134.6263 54.61 90)
 			(effects

Commit message: removed all global labels
Connections:
- net I2C1_SCL renamed I2C_SCL
- net I2C1_SDA renamed I2C_SDA
Changed lines of the file:
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@@
 		)
 	)
-	(global_label "I2C1_SDA"
+	(hierarchical_label "I2C_SCL"
 		(shape input)
-		(at 116.84 71.12 180)
-		(fields_autoplaced yes)
+		(at 116.84 73.66 180)
 		(effects
 			(font
@@
 			(justify right)
 		)
-		(property "Intersheetrefs" "${INTERSHEET_REFS}"
-			(at 105.0253 71.12 0)
-			(effects
-				(font
-					(size 1.27 1.27)
-				)
-				(justify right)
-				(hide yes)
-			)
-		)
 	)
-	(global_label "I2C1_SCL"
-		(shape input)
-		(at 116.84 73.66 180)
-		(fields_autoplaced yes)
+	(hierarchical_label "I2C_SDA"
+		(shape bidirectional)
+		(at 116.84 71.12 180)
 		(effects
 			(font
@@
 			(justify right)
 		)
-		(property "Intersheetrefs" "${INTERSHEET_REFS}"
-			(at 105.0858 73.66 0)
-			(effects
-				(font
-					(size 1.27 1.27)
-				)
-				(justify right)
-				(hide yes)
-			)
-		)
 	)

Commit message: initial layout for V2.0
Connections:
- net +3V3A: no longer U1.4 (CSB), U1.5 (CSB)
- net GND: now also U1.4 (CSB), U1.5 (CSB)
Other:
- note added: "I2C 0x76"
- note removed: "0x76"
- note removed: "I2C 0X77"
Changed lines of the file:
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@@
 		(rev "1.0")
 	)
-	(text "I2C 0X77\n\n"
+	(text "I2C 0x76\n"
 		(exclude_from_sim no)
 		(at 133.858 83.82 0)
@@
 		)
 	)
-	(text "0x76"
-		(exclude_from_sim no)
-		(at 94.742 69.342 0)
-		(effects
-			(font
-				(size 1.27 1.27)
-			)
-		)
-	)
 	(junction
 		(at 127 58.42)
@@
 	)
 	(junction
+		(at 127 82.55)
+		(diameter 0)
+		(color 0 0 0 0)
+	)
+	(junction
 		(at 127 55.88)
 		(diameter 0)
@@
 	(wire
 		(pts
-			(xy 90.17 71.12) (xy 90.17 76.2)
-		)
-		(stroke
-			(width 0)
-			(type default)
-		)
-	)
-	(wire
-		(pts
 			(xy 127 55.88) (xy 127 58.42)
 		)
@@
 	(wire
 		(pts
-			(xy 90.17 76.2) (xy 116.84 76.2)
+			(xy 127 82.55) (xy 127 86.36)
 		)
 		(stroke
@@
 	(wire
 		(pts
+			(xy 116.84 76.2) (xy 116.84 82.55)
+		)
+		(stroke
+			(width 0)
+			(type default)
+		)
+	)
+	(wire
+		(pts
 			(xy 116.84 55.88) (xy 127 55.88)
 		)
@@
 	(wire
 		(pts
-			(xy 127 81.28) (xy 127 86.36)
+			(xy 116.84 82.55) (xy 127 82.55)
+		)
+		(stroke
+			(width 0)
+			(type default)
+		)
+	)
+	(wire
+		(pts
+			(xy 127 81.28) (xy 127 82.55)
 		)
 		(stroke
@@
 					(unit 1)
 				)
-			)
-		)
-	)
-	(symbol
-		(lib_id "power:+3V3")
-		(at 90.17 71.12 0)
-		(unit 1)
-		(exclude_from_sim no)
-		(in_bom yes)
-		(on_board yes)
-		(dnp no)
-		(property "Reference" "#PWR0114"
-			(at 90.17 74.93 0)
-			(effects
-				(font
-					(size 1.27 1.27)
-				)
-				(hide yes)
-			)
-		)
-		(property "Value" "+3V3A"
-			(at 82.042 69.596 0)
-			(effects
-				(font
-					(size 1.27 1.27)
-				)
-				(justify left)
-			)
-		)
-		(property "Footprint" ""
-			(at 90.17 71.12 0)
-			(effects
-				(font
-					(size 1.27 1.27)
-				)
-				(hide yes)
-			)
-		)
-		(property "Datasheet" ""
-			(at 90.17 71.12 0)
-			(effects
-				(font
-					(size 1.27 1.27)
-				)
-				(hide yes)
-			)
-		)
-		(property "Description" "Power symbol creates a global label with name \"+3V3\""
-			(at 90.17 71.12 0)
-			(effects
-				(font
-					(size 1.27 1.27)
-				)
-				(hide yes)
-			)
-		)
-		(pin "1"
-		)
-		(instances
-			(project "flight-computer"
-				(path "/b419aaf0-5349-42bc-a414-d94cafbe45e9/f857b9c9-761d-4a7f-a2fa-b1edff240511"
-					(reference "#PWR0114")
-					(unit 1)
-				)
