File: Spaceport/PCBs/flight-computer/Alternate layout/IMU.kicad_sc.kicad_sch (KiCad schematic)
At the start: 3 parts, among them U2 BMI088

Commit message: Inductor changes, DRC checks, Silkscreen changes, BOM
Parts:
- C2, C3: value 100nF -> 100 nF
Changed lines of the file:
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@@
 			)
 		)
-		(property "Value" "100nF"
+		(property "Value" "100 nF"
 			(at 177.8 87.6301 0)
 			(effects
@@
 			)
 		)
-		(property "Value" "100nF"
+		(property "Value" "100 nF"
 			(at 191.77 87.6301 0)
 			(effects

Commit message: silkscreen changes + minor layout changes
Parts:
- U2: footprint BMI088:PQFN50P450X300X100-16N -> Package_LGA:Bosch_LGA-16_4.5x3mm_P0.5mm_LayoutBorder7x1y_ClockwisePinNumbering
Changed lines of the file:
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@@
 			)
 		)
-		(property "Footprint" "BMI088:PQFN50P450X300X100-16N"
+		(property "Footprint" "Package_LGA:Bosch_LGA-16_4.5x3mm_P0.5mm_LayoutBorder7x1y_ClockwisePinNumbering"
 			(at 152.4 100.33 0)
 			(effects

Commit message: removed all global labels
Connections:
- net I2C1_SCL renamed I2C_SCL
- net I2C1_SDA renamed I2C_SDA
Changed lines of the file:
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@@
 		)
 	)
-	(global_label "I2C1_SCL"
+	(hierarchical_label "I2C_SCL"
 		(shape input)
 		(at 134.62 102.87 180)
-		(fields_autoplaced yes)
 		(effects
 			(font
@@
 			(justify right)
 		)
-		(property "Intersheetrefs" "${INTERSHEET_REFS}"
-			(at 122.8658 102.87 0)
-			(effects
-				(font
-					(size 1.27 1.27)
-				)
-				(justify right)
-				(hide yes)
-			)
-		)
 	)
-	(global_label "I2C1_SDA"
-		(shape input)
+	(hierarchical_label "I2C_SDA"
+		(shape bidirectional)
 		(at 134.62 105.41 180)
-		(fields_autoplaced yes)
 		(effects
 			(font
@@
 			(justify right)
 		)
-		(property "Intersheetrefs" "${INTERSHEET_REFS}"
-			(at 122.8053 105.41 0)
-			(effects
-				(font
-					(size 1.27 1.27)
-				)
-				(justify right)
-				(hide yes)
-			)
-		)
 	)

Commit message: schematic changes for V2 of flight computer
Connections:
- net INT2: now reaches U2.1 (INT2)
- net INT3: now reaches U2.12 (INT3)
- net INT4: now reaches U2.13 (INT4)
- net INT1: now reaches U2.16 (INT1)
- no-connect marks 5 -> 1
Changed lines of the file:
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@@
 	(text "accel 0x18\ngyro 0x68"
 		(exclude_from_sim no)
-		(at 181.61 104.394 0)
+		(at 163.068 72.644 0)
 		(effects
 			(font
@@
 	)
 	(no_connect
-		(at 170.18 107.95)
-	)
-	(no_connect
-		(at 170.18 102.87)
-	)
-	(no_connect
-		(at 170.18 100.33)
-	)
-	(no_connect
-		(at 170.18 105.41)
-	)
-	(no_connect
 		(at 134.62 97.79)
 	)
@@
 	(wire
 		(pts
+			(xy 170.18 102.87) (xy 184.15 102.87)
+		)
+		(stroke
+			(width 0)
+			(type default)
+		)
+	)
+	(wire
+		(pts
 			(xy 181.61 92.71) (xy 195.58 92.71)
 		)
@@
 	(wire
 		(pts
+			(xy 170.18 100.33) (xy 184.15 100.33)
+		)
+		(stroke
+			(width 0)
+			(type default)
+		)
+	)
+	(wire
+		(pts
 			(xy 134.62 110.49) (xy 132.08 110.49)
 		)
@@
 	(wire
 		(pts
+			(xy 170.18 105.41) (xy 184.15 105.41)
+		)
+		(stroke
+			(width 0)
+			(type default)
+		)
+	)
+	(wire
+		(pts
 			(xy 176.53 92.71) (xy 176.53 95.25)
 		)
@@
 		(pts
 			(xy 176.53 95.25) (xy 176.53 96.52)
+		)
+		(stroke
+			(width 0)
+			(type default)
+		)
+	)
+	(wire
+		(pts
+			(xy 170.18 107.95) (xy 184.15 107.95)
 		)
 		(stroke
@@
 		)
 	)
+	(hierarchical_label "INT1"
+		(shape output)
+		(at 184.15 100.33 0)
+		(effects
+			(font
+				(size 1.27 1.27)
+			)
+			(justify left)
+		)
+	)
+	(hierarchical_label "INT3"
+		(shape output)
+		(at 184.15 105.41 0)
+		(effects
+			(font
+				(size 1.27 1.27)
+			)
+			(justify left)
+		)
+	)
 	(hierarchical_label "I2C_SDA"
 		(shape bidirectional)
@@
 		)
 	)
+	(hierarchical_label "INT4"
+		(shape output)
+		(at 184.15 107.95 0)
+		(effects
+			(font
+				(size 1.27 1.27)
+			)
+			(justify left)
+		)
+	)
+	(hierarchical_label "INT2"
+		(shape output)
+		(at 184.15 102.87 0)
+		(effects
+			(font
+				(size 1.27 1.27)
+			)
+			(justify left)
+		)
+	)
+	(symbol
+		(lib_id "power:GND")
+		(at 201.93 92.71 0)
+		(unit 1)
+		(exclude_from_sim no)
+		(in_bom yes)
+		(on_board yes)
+		(dnp no)
+		(fields_autoplaced yes)
+		(property "Reference" "#PWR04"
+			(at 201.93 99.06 0)
+			(effects
+				(font
+					(size 1.27 1.27)
+				)
+				(hide yes)
+			)
+		)
+		(property "Value" "GND"
+			(at 201.93 97.79 0)
+			(effects
+				(font
+					(size 1.27 1.27)
+				)
+			)
+		)
+		(property "Footprint" ""
+			(at 201.93 92.71 0)
+			(effects
+				(font
+					(size 1.27 1.27)
+				)
+				(hide yes)
+			)
+		)
+		(property "Datasheet" ""
+			(at 201.93 92.71 0)
+			(effects
+				(font
+					(size 1.27 1.27)
+				)
+				(hide yes)
+			)
+		)
+		(property "Description" "Power symbol creates a global label with name \"GND\" , ground"
+			(at 201.93 92.71 0)
+			(effects
+				(font
+					(size 1.27 1.27)
+				)
+				(hide yes)
+			)
+		)
+		(pin "1"
+		)
+		(instances
+			(project ""
+				(path "/b419aaf0-5349-42bc-a414-d94cafbe45e9/759fe36f-7c9c-4239-abc1-10f13c7a223d"
+					(reference "#PWR04")
+					(unit 1)
+				)
+			)
+		)
+	)
 	(symbol
 		(lib_id "power:VDD")
@@
 			)
 		)
+		(property "SNAPEDA_PACKAGE_ID" ""
+			(at 181.61 88.9 0)
+			(effects
+				(font
+					(size 1.27 1.27)
+				)
+				(hide yes)
+			)
+		)
 		(pin "2"
 		)
@@
 			)
 		)
+		(property "SNAPEDA_PACKAGE_ID" ""
+			(at 152.4 100.33 0)
+			(effects
+				(font
+					(size 1.27 1.27)
+				)
+				(hide yes)
+			)
+		)
 		(pin "10"
 		)
@@
 				(path "/b419aaf0-5349-42bc-a414-d94cafbe45e9/759fe36f-7c9c-4239-abc1-10f13c7a223d"
 					(reference "U2")
-					(unit 1)
-				)
-			)
-		)
-	)
-	(symbol
-		(lib_id "power:GND")
-		(at 201.93 92.71 0)
-		(unit 1)
-		(exclude_from_sim no)
-		(in_bom yes)
-		(on_board yes)
-		(dnp no)
-		(fields_autoplaced yes)
-		(property "Reference" "#PWR04"
-			(at 201.93 99.06 0)
-			(effects
-				(font
-					(size 1.27 1.27)
-				)
-				(hide yes)
-			)
-		)
-		(property "Value" "GND"
-			(at 201.93 97.79 0)
-			(effects
-				(font
-					(size 1.27 1.27)
-				)
-				(hide yes)
-			)
-		)
-		(property "Footprint" ""
-			(at 201.93 92.71 0)
-			(effects
-				(font
-					(size 1.27 1.27)
-				)
-				(hide yes)
-			)
-		)
-		(property "Datasheet" ""
-			(at 201.93 92.71 0)
-			(effects
-				(font
-					(size 1.27 1.27)
-				)
-				(hide yes)
-			)
-		)
-		(property "Description" "Power symbol creates a global label with name \"GND\" , ground"
-			(at 201.93 92.71 0)
-			(effects
-				(font
-					(size 1.27 1.27)
-				)
-				(hide yes)
-			)
-		)
-		(pin "1"
-		)
-		(instances
-			(project ""
-				(path "/b419aaf0-5349-42bc-a414-d94cafbe45e9/759fe36f-7c9c-4239-abc1-10f13c7a223d"
-					(reference "#PWR04")
 					(unit 1)
 				)
@@
 			)
 		)
+		(property "SNAPEDA_PACKAGE_ID" ""
+			(at 195.58 88.9 0)
+			(effects
+				(font
+					(size 1.27 1.27)
+				)
+				(hide yes)
+			)
+		)
 		(pin "2"
 		)
@@
 		(on_board yes)
 		(dnp no)
-		(fields_autoplaced yes)
 		(property "Reference" "#PWR094"
 			(at 176.53 102.87 0)
@@
 		)
 		(property "Value" "GND"
-			(at 176.53 101.6 0)
-			(effects
-				(font
+			(at 179.832 97.536 0)
+			(effects
+				(font

Commit message: V2 finished, BOM made, Prod files ready
Parts:
- U2: DESCRIPTION Accelerometer, Gyroscope, 6 Axis Sensor I²C, SPI Output -> (none)
