File: Spaceport/PCBs/flight-computer/Alternate layout/Magnetometer.kicad_sc.kicad_sch (KiCad schematic)
At the start: 3 parts, among them U10 MLX90393ELW-ABA-xxx-xx

Commit message: Inductor changes, DRC checks, Silkscreen changes, BOM
Parts:
- C28, C6: value 100nF -> 100 nF
Changed lines of the file:
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@@
 			)
 		)
-		(property "Value" "100nF"
+		(property "Value" "100 nF"
 			(at 156.2163 105.41 90)
 			(effects
@@
 			)
 		)
-		(property "Value" "100nF"
+		(property "Value" "100 nF"
 			(at 166.3637 60.96 90)
 			(effects

Commit message: Changes requested by Joseph
Connections:
- net GND: now also U10.17 (GND)
Changed lines of the file:
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@@
+	)
+	(junction
+		(at 161.29 109.22)
+		(diameter 0)
+		(color 0 0 0 0)
 	)
 	(junction
@@
 	(wire
 		(pts
+			(xy 161.29 109.22) (xy 158.75 109.22)
+		)
+		(stroke
+			(width 0)
+			(type default)
+		)
+	)
+	(wire
+		(pts
 			(xy 158.75 99.06) (xy 158.75 101.6)
 		)
@@
 	(wire
 		(pts
-			(xy 168.91 109.22) (xy 158.75 109.22)
+			(xy 168.91 109.22) (xy 161.29 109.22)
+		)
+		(stroke
+			(width 0)
+			(type default)
+		)
+	)
+	(wire
+		(pts
+			(xy 161.29 99.06) (xy 161.29 109.22)
 		)
 		(stroke
@@
 		(pin "12"
 		)
+		(pin "17"
+		)
 		(instances

Commit message: removed all global labels
Connections:
- net I2C1_SCL renamed I2C_SCL
- net I2C1_SDA renamed I2C_SDA
Changed lines of the file:
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@@
 		)
 	)
-	(global_label "I2C1_SDA"
+	(hierarchical_label "I2C_SCL"
 		(shape input)
+		(at 140.97 86.36 180)
+		(effects
+			(font
+				(size 1.27 1.27)
+			)
+			(justify right)
+		)
+	)
+	(hierarchical_label "I2C_SDA"
+		(shape bidirectional)
 		(at 151.13 73.66 90)
-		(fields_autoplaced yes)
 		(effects
 			(font
@@
 			(justify left)
 		)
-		(property "Intersheetrefs" "${INTERSHEET_REFS}"
-			(at 151.13 61.8453 90)
-			(effects
-				(font
-					(size 1.27 1.27)
-				)
-				(justify left)
-				(hide yes)
-			)
-		)
 	)
-	(global_label "I2C1_SCL"
-		(shape input)
-		(at 140.97 86.36 180)
-		(fields_autoplaced yes)
-		(effects
-			(font
-				(size 1.27 1.27)
-			)
-			(justify right)
-		)
-		(property "Intersheetrefs" "${INTERSHEET_REFS}"
-			(at 129.2158 86.36 0)
-			(effects
-				(font
-					(size 1.27 1.27)
-				)
-				(justify right)
-				(hide yes)
-			)
-		)
-	)

Commit message: schematic changes for V2 of flight computer
Connections:
- net INT1: now reaches U10.1 (INT)
- net INT2: now reaches U10.7 (INT/TRIG)
- no-connect marks 3 -> 1
Other:
- moved on the sheet: C6
Changed lines of the file:
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@@
+	)
+	(junction
+		(at 129.54 88.9)
+		(diameter 0)
+		(color 0 0 0 0)
 	)
 	(junction
@@
 	)
 	(junction
-		(at 138.43 88.9)
+		(at 161.29 101.6)
 		(diameter 0)
 		(color 0 0 0 0)
@@
 		(color 0 0 0 0)
 	)
-	(junction
-		(at 158.75 109.22)
-		(diameter 0)
-		(color 0 0 0 0)
-	)
-	(no_connect
-		(at 140.97 91.44)
-	)
-	(no_connect
-		(at 156.21 73.66)
-	)
 	(no_connect
 		(at 153.67 73.66)
@@
 	(wire
 		(pts
-			(xy 138.43 88.9) (xy 140.97 88.9)
+			(xy 158.75 102.87) (xy 158.75 101.6)
+		)
+		(stroke
+			(width 0)
+			(type default)
+		)
+	)
+	(wire
+		(pts
+			(xy 153.67 102.87) (xy 153.67 101.6)
 		)
 		(stroke
@@
 	(wire
 		(pts
-			(xy 125.73 88.9) (xy 138.43 88.9)
+			(xy 161.29 101.6) (xy 158.75 101.6)
 		)
 		(stroke
@@
 	(wire
 		(pts
-			(xy 138.43 88.9) (xy 138.43 102.87)
-		)
-		(stroke
-			(width 0)
-			(type default)
-		)
-	)
-	(wire
-		(pts
-			(xy 157.48 64.77) (xy 158.75 64.77)
-		)
-		(stroke
-			(width 0)
-			(type default)
-		)
-	)
-	(wire
-		(pts
-			(xy 138.43 102.87) (xy 153.67 102.87)
+			(xy 129.54 88.9) (xy 129.54 101.6)
+		)
+		(stroke
+			(width 0)
+			(type default)
+		)
+	)
+	(wire
+		(pts
+			(xy 129.54 101.6) (xy 153.67 101.6)
 		)
 		(stroke
@@
 	(wire
 		(pts
-			(xy 161.29 99.06) (xy 161.29 109.22)
+			(xy 161.29 99.06) (xy 161.29 101.6)
 		)
 		(stroke
@@
 	(wire
 		(pts
-			(xy 158.75 101.6) (xy 158.75 109.22)
+			(xy 161.29 101.6) (xy 161.29 109.22)
 		)
 		(stroke
@@
 	(wire
 		(pts
-			(xy 153.67 102.87) (xy 153.67 101.6)
-		)
-		(stroke
-			(width 0)
-			(type default)
+			(xy 129.54 88.9) (xy 140.97 88.9)
+		)
+		(stroke
+			(width 0)
+			(type default)
+		)
+	)
+	(hierarchical_label "INT1"
+		(shape output)
+		(at 140.97 91.44 180)
+		(effects
+			(font
+				(size 1.27 1.27)
+			)
+			(justify right)
 		)
 	)
@@
 		)
 	)
+	(hierarchical_label "INT2"
+		(shape output)
+		(at 156.21 73.66 90)
+		(effects
+			(font
+				(size 1.27 1.27)
+			)
+			(justify left)
+		)
+	)
 	(hierarchical_label "I2C_SDA"
 		(shape bidirectional)
@@
 	(symbol
 		(lib_id "Device:C_Small")
-		(at 156.21 101.6 90)
+		(at 156.21 102.87 90)
 		(mirror x)
 		(unit 1)
@@
 		(dnp no)
 		(property "Reference" "C6"
-			(at 156.2163 107.95 90)
+			(at 156.2163 109.22 90)
 			(effects
 				(font
@@
 		)
 		(property "Value" "100 nF"
-			(at 156.2163 105.41 90)
+			(at 156.2163 106.68 90)
 			(effects
 				(font
@@
 		)
 		(property "Footprint" "Capacitor_SMD:C_0603_1608Metric_Pad1.08x0.95mm_HandSolder"
-			(at 156.21 101.6 0)
+			(at 156.21 102.87 0)
 			(effects
 				(font
@@
 		)
 		(property "Datasheet" "~"
-			(at 156.21 101.6 0)
+			(at 156.21 102.87 0)
 			(effects
 				(font
@@
 		)
 		(property "Description" "Unpolarized capacitor, small symbol"
-			(at 156.21 101.6 0)
+			(at 156.21 102.87 0)
+			(effects
+				(font
+					(size 1.27 1.27)
+				)
+				(hide yes)
+			)
+		)
+		(property "SNAPEDA_PACKAGE_ID" ""
+			(at 156.21 102.87 90)
 			(effects
 				(font
@@
 	(symbol
 		(lib_id "power:+3V3")
-		(at 125.73 88.9 0)
+		(at 129.54 88.9 0)
 		(unit 1)
 		(exclude_from_sim no)
@@
 		(fields_autoplaced yes)
 		(property "Reference" "#PWR010"
-			(at 125.73 92.71 0)
+			(at 129.54 92.71 0)
 			(effects
 				(font
@@
 		)
 		(property "Value" "+3V3A"
-			(at 125.73 83.82 0)
+			(at 129.54 83.82 0)
 			(effects
 				(font
@@
 		)
 		(property "Footprint" ""
-			(at 125.73 88.9 0)
+			(at 129.54 88.9 0)
 			(effects
 				(font
@@
 		)
 		(property "Datasheet" ""
-			(at 125.73 88.9 0)
+			(at 129.54 88.9 0)
 			(effects
 				(font
@@
 		)
 		(property "Description" "Power symbol creates a global label with name \"+3V3\""
-			(at 125.73 88.9 0)
+			(at 129.54 88.9 0)
 			(effects
 				(font
@@
 			)
 		)
+		(property "SNAPEDA_PACKAGE_ID" ""
+			(at 166.37 64.77 90)
+			(effects
+				(font
+					(size 1.27 1.27)
+				)
+				(hide yes)
+			)
+		)
 		(pin "1"
 		)
@@
 			)
 		)
+		(property "SNAPEDA_PACKAGE_ID" ""
+			(at 140.97 91.44 0)
+			(effects
+				(font
+					(size 1.27 1.27)
+				)
+				(hide yes)
+			)
+		)
 		(pin "3"
 		)
@@
 	(symbol
 		(lib_id "power:+3V3")
-		(at 157.48 64.77 0)
+		(at 158.75 64.77 0)
 		(unit 1)
 		(exclude_from_sim no)
@@
 		(dnp no)
 		(property "Reference" "#PWR012"
-			(at 157.48 68.58 0)
+			(at 158.75 68.58 0)
 			(effects
 				(font
@@
 		)
 		(property "Value" "+3V3A"
-			(at 154.178 60.4519 0)
+			(at 155.448 60.4519 0)
 			(effects
 				(font
@@
 		)
 		(property "Footprint" ""
-			(at 157.48 64.77 0)
+			(at 158.75 64.77 0)
 			(effects
 				(font
@@
 		)
 		(property "Datasheet" ""
-			(at 157.48 64.77 0)
+			(at 158.75 64.77 0)
 			(effects
 				(font
@@
 		)
 		(property "Description" "Power symbol creates a global label with name \"+3V3\""
-			(at 157.48 64.77 0)
-			(effects
-				(font
+			(at 158.75 64.77 0)
+			(effects
+				(font

Commit message: initial layout for V2.0
Connections:
- net GND: now also U10.10 (NC), U10.14 (NC), U10.16 (NC), U10.4 (NC), U10.9 (NC)
Changed lines of the file:
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@@
+	(wire
+		(pts
+			(xy 151.13 99.06) (xy 142.24 99.06)
+		)
+		(stroke
+			(width 0)
+			(type default)
+		)
+	)
 	(wire
 		(pts
@@
 	(wire
 		(pts
+			(xy 137.16 96.52) (xy 142.24 96.52)
+		)
+		(stroke
+			(width 0)
+			(type default)
+		)
+	)
+	(wire
+		(pts
 			(xy 153.67 101.6) (xy 153.67 99.06)
 		)
@@
 		(pts
 			(xy 158.75 64.77) (xy 163.83 64.77)
+		)
+		(stroke
+			(width 0)
+			(type default)
+		)
+	)
+	(wire
+		(pts
+			(xy 142.24 99.06) (xy 142.24 96.52)
 		)
 		(stroke
@@
 					(unit 1)
 				)
+			)
+		)
+	)
+	(symbol
+		(lib_id "power:GND")
+		(at 137.16 96.52 0)
+		(unit 1)
+		(exclude_from_sim no)
+		(in_bom yes)
+		(on_board yes)
+		(dnp no)
+		(property "Reference" "#PWR074"
+			(at 137.16 102.87 0)
+			(effects
+				(font
+					(size 1.27 1.27)
+				)
+				(hide yes)
+			)
+		)
+		(property "Value" "GND"
+			(at 137.16 100.838 0)
+			(effects
+				(font
+					(size 1.27 1.27)
+				)
+			)
+		)
+		(property "Footprint" ""
+			(at 137.16 96.52 0)
+			(effects
+				(font
+					(size 1.27 1.27)
+				)
+				(hide yes)
+			)
+		)
+		(property "Datasheet" ""
+			(at 137.16 96.52 0)
+			(effects
+				(font
+					(size 1.27 1.27)
+				)
+				(hide yes)
+			)
+		)
+		(property "Description" "Power symbol creates a global label with name \"GND\" , ground"
+			(at 137.16 96.52 0)
+			(effects
+				(font
+					(size 1.27 1.27)
+				)
+				(hide yes)
+			)
+		)
+		(pin "1"
+		)
+		(instances
+			(project ""
+				(path "/b419aaf0-5349-42bc-a414-d94cafbe45e9/59137cc8-27c9-41ae-9820-03727e90c02e"
+					(reference "#PWR074")
+					(unit 1)
+				)
