File: Spaceport/PCBs/Radios/medium-power-module-telemetry/medium-power-module-telemetry.kicad_pcb (KiCad board)
At the start: 4 copper layers, 27.4 x 45.2 mm, 80 parts, among them J2 SMA, J5 Conn_01x04_Pin, J7 UART, U3 LDL212PVR, U4 TLV61048DBVR, U6 LDL212PVR

Commit message: final for first radio board
Parts:
- moved C7 2.47 mm to (148.8, 103.9), turned to 180 degrees
- moved CD1 0.58 mm to (151.1, 128.0)
- moved TCXO1 0.57 mm to (151.2, 126.0)
- moved C20 0.10 mm to (152.1, 118.3)
- renumbered LChoke1 to LC1
Routing:
- net GND: track 0.00 -> 56.7 mm, vias 0 -> 186
- net 3V3_LDO: track 33.5 -> 70.7 mm, vias 1 -> 3
- net 8V_LDO: track 20.7 -> 38.5 mm, vias 0 -> 2
- net 3V3_IN: track 37.6 -> 48.0 mm
- net GNDX: track 0.00 -> 7.11 mm
- net 8V_TO_LDO: track 0.00 -> 5.46 mm
- net RXp: track 0.00 -> 5.15 mm
- net GPIO0: track 41.4 -> 46.1 mm
- net Net-(C0-Pad2): track 0.00 -> 4.53 mm
- net Net-(U3-ADJ/SENSE): track 0.00 -> 4.43 mm
- net Net-(U6-ADJ/SENSE): track 0.00 -> 4.21 mm
- net Net-(U7-V_EN): track 0.00 -> 4.13 mm, vias 0 -> 1
- net Net-(U4-FB): track 0.00 -> 3.69 mm
- net LNA_IN: track 0.00 -> 3.62 mm
- net TX: track 0.00 -> 3.24 mm
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- added copper zone on F.Cu, net 3V3_IN
- added copper zone on B.Cu, net 3V3_LDO
- added copper zone on F.Cu, net 3V3_LDO
- added copper zone on F.Cu, net 8V_LDO
- added copper zone on F.Cu, net 8V_TO_LDO
- added copper zone on B.Cu, net GND
- added copper zone on F.Cu, net GND
- added copper zone on B.Cu, net Net-(C11-Pad1)
- added copper zone on B.Cu, net Net-(C16-Pad2)
- added copper zone on B.Cu, net Net-(C18-Pad1)
- added copper zone on B.Cu, net Net-(C8-Pad2)
- added copper zone on F.Cu, net Net-(D1-A)
