File: Spaceport/PCBs/Radios/medium-power-module-telemetry-2/medium-power-module-telemetry-2.kicad_sch (KiCad schematic)
At the start: 80 parts, among them J1 Conn_01x05_Pin, J2 SMA, J7 UART, U3 LDL212PVR, U4 TLV61048DBVR, U6 LDL212PVR

Commit message: gerbers
Parts:
- removed C16, C18: 100p, Capacitor_SMD:C_0603_1608Metric, symbol Device:C
- removed C17: 0.1u, Capacitor_SMD:C_0603_1608Metric, symbol Device:C
- removed L10, L11: 100n, Inductor_SMD:L_0603_1608Metric, symbol Device:L
- removed R11: 2.61k, Resistor_SMD:R_0603_1608Metric, symbol Device:R
- removed U7: ~, Avionics:GRF5010, symbol Avionics:GRF5010
- added U7, U9: ~, Avionics:BGS12P2L6, symbol Avionics:BGS12P2L6
Connections:
- net 3V3_LDO: now also U7.4 (VDD), U9.4 (VDD)
- net GND: now also U7.2 (GND), U9.2 (GND)
- net GPIO0: now also U7.6 (CTRL), U9.6 (CTRL)
- net LNA_IN: now also U8.1 (RF_2), U9.1 (RF_2); no longer U8.3 (RF_1)
- net LNA_OUT: now also U7.1 (RF_2)
- net PA_IN: now also U8.3 (RF_1); no longer C8.1, L3.1
- net PA_OUT: now also U7.3 (RF_1), U9.3 (RF_1); no longer C11.2, U8.1 (RF_2)
- net SW_OUT: now also U9.5 (RF_IN); no longer U8.5 (RF_IN)
- new net AMP_IN: C8.1, L3.1, U8.5 (RF_IN)
- new net AMP_OUT: C11.2, U7.5 (RF_IN)
Other:
- note added: "PA/LNA"
- note added: "Set GPIO0 to high in RX mode"
- note removed: "LNA"
- note removed: "PA"
- note removed: "Set GPIO0 to high in TX mode"
- moved on the sheet: C11, C12, C8, L3, L4, R7, U5

Commit message: component change from making BOM
Parts:
- C1, C20, C21: value 100n -> 0.1u
- CB3: value 10nF -> 10n
- CD1: value 10uF -> 10u
- R3: value 13.7k -> 16.5k
- R7: value 2.61k -> 2.49k
- R8: value 10.2k -> 10.7k
- R9: value 59k -> 61.9k
Changed lines of the file:
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@@
 			)
 		)
-		(property "Value" "10.2k"
+		(property "Value" "10.7k"
 			(at 85.09 71.1199 0)
 			(effects
@@
 			)
 		)
-		(property "Value" "10uF"
+		(property "Value" "10u"
 			(at 13.462 83.058 0)
 			(effects
@@
 			)
 		)
-		(property "Value" "59k"
+		(property "Value" "61.9k"
 			(at 85.09 78.7399 0)
 			(effects
@@
 			)
 		)
-		(property "Value" "100n"
+		(property "Value" "0.1u"
 			(at 45.72 161.2899 0)
 			(effects
@@
 			)
 		)
-		(property "Value" "13.7k"
+		(property "Value" "16.5k"
 			(at 77.47 33.0199 0)
 			(effects
@@
 			)
 		)
-		(property "Value" "10nF"
+		(property "Value" "10n"
 			(at 60.96 71.882 90)
 			(effects
@@
 			)
 		)
-		(property "Value" "2.61k"
+		(property "Value" "2.49k"
 			(at 226.06 134.6199 0)
 			(effects
@@
 			)
 		)
-		(property "Value" "100n"
+		(property "Value" "0.1u"
 			(at 35.56 161.2899 0)
 			(effects
@@
 			)
 		)
-		(property "Value" "100n"
+		(property "Value" "0.1u"
 			(at 25.4 161.2899 0)
 			(effects

Commit message: forgot to update component values
Parts:
- L2: value 10u -> 4.7u
Changed lines of the file:
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@@
 			)
 		)
-		(property "Value" "10u"
+		(property "Value" "4.7u"
 			(at 189.23 21.59 90)
 			(effects

Commit message: mpm-telemetry v1.1
Parts:
- added D2: D_Schottky, Avionics:DIO_MSS1P4-M3_89A, symbol Device:D_Schottky
Connections:
- net 3V3_IN: no longer C1.1, C20.1, C21.1, U2.1 (VDD), U2.17 (VDD), U2.5 (VDDA)
- net 3V3_LDO: now also D2.2 (A)
- net SRX: now also U2.20 (PA10); no longer U2.19 (PA9)
- net STX: now also U2.19 (PA9); no longer U2.18 (PA8)
- new net 3V3_MCU: C1.1, C20.1, C21.1, D2.1 (K), U2.1 (VDD), U2.17 (VDD), U2.5 (VDDA)
Other:
- moved on the sheet: C1, C20, C21

Commit message: fix LDO
Parts:
- R3: value 16.5k -> 19.1k
Other:
- note added: "3.3V 500mA"
- note removed: "2.8V 500mA"
Changed lines of the file:
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@@
 		)
 	)
-	(text "2.8V 500mA"
+	(text "3.3V 500mA"
 		(exclude_from_sim no)
 		(at 70.358 40.894 0)
@@
 			)
 		)
-		(property "Value" "16.5k"
+		(property "Value" "19.1k"
 			(at 77.47 33.0199 0)
 			(effects
