File: Spaceport/PCBs/ARCH-Mega/current.kicad_sch (KiCad schematic)
At the start: 18 parts, among them U13 INA3221, U14 INA3221

Commit message: Added footprints and 3d models for missing components
Parts:
- C39, C40: footprint Package_DFN_QFN:Texas_RGV0016A_VQFN-16-1EP_4x4mm_P0.65mm_EP2.1x2.1mm -> Capacitor_SMD:C_0603_1608Metric
- U13, U14: footprint Package_DFN_QFN:Texas_RGV0016A_VQFN-16-1EP_4x4mm_P0.65mm_EP2.1x2.1mm -> custom_footprints:QFN65P400X400X100-17N
Changed lines of the file:
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@@
 			)
 		)
-		(property "Footprint" "Package_DFN_QFN:Texas_RGV0016A_VQFN-16-1EP_4x4mm_P0.65mm_EP2.1x2.1mm"
+		(property "Footprint" "Capacitor_SMD:C_0603_1608Metric"
 			(at 176.53 87.3252 0)
 			(hide yes)
@@
 			)
 		)
-		(property "Footprint" "Package_DFN_QFN:Texas_RGV0016A_VQFN-16-1EP_4x4mm_P0.65mm_EP2.1x2.1mm"
+		(property "Footprint" "Capacitor_SMD:C_0603_1608Metric"
 			(at 96.52 87.3252 0)
 			(hide yes)
@@
 			)
 		)
-		(property "Footprint" "Package_DFN_QFN:Texas_RGV0016A_VQFN-16-1EP_4x4mm_P0.65mm_EP2.1x2.1mm"
+		(property "Footprint" "custom_footprints:QFN65P400X400X100-17N"
 			(at 106.68 80.01 0)
 			(hide yes)
@@
 			)
 		)
-		(property "Footprint" "Package_DFN_QFN:Texas_RGV0016A_VQFN-16-1EP_4x4mm_P0.65mm_EP2.1x2.1mm"
+		(property "Footprint" "custom_footprints:QFN65P400X400X100-17N"
 			(at 186.69 80.01 0)
 			(hide yes)
