File: Spaceport/PCBs/STM32-flight-computer/STM32-flight-computer.kicad_sch (KiCad schematic)
At the start: 49 parts, among them J1 SMA, J2 Conn_01x06, J3 UART, J4 SW, J5 >5V, J6 USB_C_Receptacle_USB2.0_16P, U1 LBAA0XV2GT-001, U2 SAM-M8Q, U3 DPS310XTSA1, U4 STM32H723VEHx, U5 H3LIS331DLTR, U6 MMC5633NJL, U7 BMI088, U8 AMS1117-3.3

Commit message: Added all ICs to schematic
Parts:
- removed U8: AMS1117-3.3, Package_TO_SOT_SMD:SOT-223-3_TabPin2, symbol Regulator_Linear:AMS1117-3.3
- added C12, C13, C24: 100n, Capacitor_SMD:C_0603_1608Metric, symbol Device:C
- added C25: 1n, Capacitor_SMD:C_0603_1608Metric, symbol Device:C
- added D5, D?: D_Schottky, symbol Device:D_Schottky
- added L?: 1u, symbol Device:L
- added Q1, Q?: MCM3400A-TP, DFN2020-6L_MCE, symbol 2025-10-09_15-16-18:MCM3400A-TP
- added R10, R11, R12, R13, R16, R8, R9: DNP, Resistor_SMD:R_0603_1608Metric, symbol Device:R
- added R14, R15: 5k1, Resistor_SMD:R_0402_1005Metric, symbol Device:R
- added R17: 120k, Resistor_SMD:R_0603_1608Metric, symbol Device:R
- added R18, R20: 24k9, Resistor_SMD:R_0603_1608Metric, symbol Device:R
- added R19, R22, R23: 78k7, Resistor_SMD:R_0603_1608Metric, symbol Device:R
- added R21: 10k, Resistor_SMD:R_0603_1608Metric, symbol Device:R
- added U?: TPD2EUSB30A, Package_TO_SOT_SMD:Texas_DRT-3, symbol Power_Protection:TPD2EUSB30A
- added U?: TPS62902RPJR, TPS62902RPJR:IC_TPS62902RPJR, symbol TPS62902RPJR:TPS62902RPJR
- added U?: FSC-BT691, FSC-BT691:FSC-BT691, symbol FSC-BT691:FSC-BT691
- added U?: APX803L, symbol APX803L:APX803L
- added U?: NCP186AMX330TAG, NCP186AMX330TAG:PSON40P160X120X45-9N, symbol NCP186AMX330TAG:NCP186AMX330TAG
- added U?: 74LVC08ABQ115, Package_DFN_QFN:DHVQFN-14-1EP_2.5x3mm_P0.5mm_EP1x1.5mm, symbol 74LVC08ABQ115:74LVC08ABQ115
- C22: value 2u2 -> 22u
- C23: value 2u2 -> 10u
- D4: footprint Diode_SMD:D_0603_1608Metric -> (none)
- J5: value >5V -> >3.5V
- U2: value SAM-M8Q -> SAM-M10Q
- U?: value ~ -> FEMC004GSTE9-T14-17
Connections:
- net +3V3: now also U?.C6 (VCCQ), U?.E6 (VCC), U?.F5 (VCC), U?.J10 (VCC), U?.K5 (~{RST}), U?.K9 (VCC), U?.M4 (VCCQ), U?.N4 (VCCQ), U?.P3 (VCCQ), U?.P5 (VCCQ), C12.2, C13.1, C25.2, R10.2, R11.2, R12.2, R13.2, R16.2, R19.2, R9.2, U?.1 (OUT), U?.2 (OUT__1), U?.6 (~{RESET}), U?.7 (VDD); no longer D4.1 (K)
- net GND: now also C22.1, C23.1, J6.A1 (GND), J6.A12 (GND), J6.B1 (GND), J6.B12 (GND), J6.S1 (SHIELD), U?.A6 (VSS), U?.C4 (VSSQ), U?.E7 (VSS), U?.G5 (VSS), U?.H10 (VSS), U?.J5 (VSS), U?.K8 (VSS), U?.N2 (VSSQ), U?.N5 (VSSQ), U?.P4 (VSSQ), U?.P6 (VSSQ), C12.1, C13.2, C24.1, R14.2, R15.2, R18.2, R20.2, R8.2, U?.19 (GND), U?.3 (GND), U?.4 (GND), U?.5 (GND), U?.7 (MODE/S-CONF), U?.8 (GND), U?.9 (EPAD); no longer C22.2, C23.2
- net RX: no longer U4.A5 (PB7)
- net TX: no longer U4.B5 (PB6)
- net at D4.2 (A): now also J4.1 (Pin_1), D5.2 (A); no longer C23.1
- net MEM_DAT0: now reaches U?.A3 (DAT0)
- net MEM_DAT0: now also R10.1
- net MEM_DAT1: now reaches U?.A4 (DAT1)
- net MEM_DAT1: now also R11.1
- net MEM_DAT2: now reaches U?.A5 (DAT2)
- net MEM_DAT2: now also R12.1
- net MEM_DAT3: now reaches U?.B2 (DAT3)
- net MEM_DAT3: now also R13.1
- net at U?.C2 (VDDi): now also C24.2
- net at U?.H5 (DS): now also R8.1
- net MEM_CMD: now reaches U?.M5 (CMD)
- net MEM_CMD: now also R9.1
- net MEM_CLK: now reaches U?.M6 (CLK)
- net MEM_CLK: now also R16.1
- net VBUS: now reaches J6.A4 (VBUS), J6.A9 (VBUS), J6.B4 (VBUS), J6.B9 (VBUS)
- net VBUS: now also D?.2 (A)
- net at J6.A5 (CC1): now also R14.1
- net USB_D+: now reaches J6.A6 (D+)
- net USB_D+: now also J6.B6 (D+), U?.1 (D+)
- net USB_D-: now reaches J6.A7 (D-)
- net USB_D-: now also J6.B7 (D-), U?.2 (D-)
- net at J6.B5 (CC2): now also R15.1
- new net: L?.1, U?.2 (SW)
- new net: C23.2, L?.2, R17.1, R21.2, U?.3 (VOS), U?.7 (IN), U?.8 (IN__1)
- new net: R17.2, R18.1, U?.9 (FB/VSET)
- new net: C25.1, R19.1, R20.1, U?.4 (FB/ADJ)
- new net: R21.1, U?.1 (PG), U?.6 (EN)
- new net: R22.1, R23.2, U?.3 (VCC)
- new net: C22.2, D4.1 (K), D?.1 (K), U?.5 (EN), U?.6 (VIN)
- new net: U?.10 (PIO2/ADC1), U?.14 (PIO2/ADC1)
- new net: U?.11 (NC), U?.12 (NC)
- new net: U?.13 (NC), U?.9 (NC)
- new net BT_RX: U?.2 (PIO9/RX)
- new net BT_TX: U?.1 (PIO8/TX)
- new net CONN_RX: U4.A5 (PB7)
- new net CONN_TX: U4.B5 (PB6)
- new net PYRO: D5.1 (K)
- no-connect marks 87 -> 101
Other:
- note added: "0805 rec."
- note added: "0x30"
- note added: "Bluetooth Module"
- note added: "DNP = 10k if needed"
- note added: "Power"
- note added: "eMMC Storage"
- moved on the sheet: C11, C8, D2, D3, J1, J2, J3, J4, J5, J6, L1, R4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

Commit message: Finished first pass of Pyro Schem
Parts:
- removed R22, R23: 78k7, Resistor_SMD:R_0603_1608Metric, symbol Device:R
- removed U?: APX803L, symbol APX803L:APX803L
- added C12: 10u, Capacitor_SMD:C_0603_1608Metric, symbol Device:C
- added J5: Conn_01x08, symbol Connector_Generic:Conn_01x08
- added R8: 422k, Resistor_SMD:R_0603_1608Metric, symbol Device:R
- added R9: 102k, Resistor_SMD:R_0603_1608Metric, symbol Device:R
- added U6: TPS3842, symbol TPS3842:TPS3842
- gave numbers to parts that had none: 9
- renumbered C12 to C10, C13 to C11, C22 to C13, C25 to C14, C23 to C15, C24 to C16, C14 to C17, C15 to C18, C16 to C19, C17 to C20, C18 to C21, C6 to C22, C7 to C23, C9 to C24, C10 to C25, C19 to C26, C8 to C6, C11 to C7, C20 to C8, C21 to C9, D4 to D5, D5 to D6, J2 to J1, J3 to J2, J6 to J3, J1 to J4, J4 to J6, J5 to J7, Q1 to Q2, R14 to R1, R19 to R10, R9 to R11, R10 to R12, R17 to R13, R16 to R14, R11 to R15, R18 to R16, R21 to R17, R12 to R18, R13 to R19, R15 to R2, R8 to R21, U6 to U10, U5 to U11, U2 to U12, U3 to U13, U7 to U14, U4 to U3
Connections:
- net RX is gone; now on net CONN_RX: J2.3 (Pin_3)
- net TX is gone; now on net CONN_TX: J2.2 (Pin_2)
- net +3V3: now also U4.14 (VCC), C12.2
- net GND: now also U4.7 (GND), C12.1, J5.2 (Pin_2), J5.4 (Pin_4), J5.6 (Pin_6), J5.8 (Pin_8), R9.2, U6.4 (CTS), U6.5 (GND), U6.6 (CTR)
- net PYRO: now also Q1.3, Q1.6, Q2.3, Q2.6
- net PYRO_2: now reaches Q2.1
- net PYRO_2: now also J5.3 (Pin_3)
- net GATE_2: now reaches Q2.2
- net GATE_2: now also U4.6 (2Y)
- net PYRO_4: now reaches Q2.4
- net PYRO_4: now also J5.7 (Pin_7)
- net GATE_4: now reaches Q2.5
- net GATE_4: now also U4.11 (4Y)
- net V_SENSE: now reaches C13.2, D4.1 (K), D5.1 (K), U7.5 (EN), U7.6 (VIN)
- net V_SENSE: now also R8.1, U6.1 (VDD)
- net PYRO_1: now reaches Q1.1
- net PYRO_1: now also J5.1 (Pin_1)
- net GATE_1: now reaches Q1.2
- net GATE_1: now also U4.3 (1Y)
- net PYRO_3: now reaches Q1.4
- net PYRO_3: now also J5.5 (Pin_5)
- net GATE_3: now reaches Q1.5
- net GATE_3: now also U4.8 (3Y)
- net ARM: now reaches U4.1 (1A)
- net ARM: now also U4.12 (4A), U4.4 (2A), U4.9 (3A), U6.3 (~{RST})
- net FIRE_3: now reaches U4.10 (3B)
- net FIRE_4: now reaches U4.13 (4B)
- net FIRE_1: now reaches U4.2 (1B)
- net FIRE_2: now reaches U4.5 (2B)
- net GPS_D: no longer names the net of D3.2 (A), R7.2
- net SENS_D: no longer names the net of D2.2 (A), R6.2
- new net: R8.2, R9.1, U6.2 (SENSE)
- no-connect marks 101 -> 102
Other:
- moved on the sheet: D4, J2, Q1, Q2, U4

Commit message: redid pyro schematic
Parts:
- added R22, R23, R24, R25, R39: 10k, Resistor_SMD:R_0603_1608Metric, symbol Device:R
- added R26, R28, R30, R32: 24k9, Resistor_SMD:R_0603_1608Metric, symbol Device:R
- added R27, R29, R31, R33: 100k, Resistor_SMD:R_0603_1608Metric, symbol Device:R
- added R38: 300, Resistor_SMD:R_0603_1608Metric, symbol Device:R
Connections:
- net ARM: now also R38.1, R39.2
- net FIRE_1: now also R22.2
- net FIRE_2: now also R23.2
- net FIRE_3: now also R24.2
- net FIRE_4: now also R25.2
- net GND: now also Q1.1, Q1.4, Q2.1, Q2.4, R22.1, R23.1, R24.1, R25.1, R26.2, R28.2, R30.2, R32.2, R39.1; no longer J5.2 (Pin_2), J5.4 (Pin_4), J5.6 (Pin_6), J5.8 (Pin_8)
- net PYRO: now also J5.2 (Pin_2), J5.4 (Pin_4), J5.6 (Pin_6), J5.8 (Pin_8); no longer Q1.3, Q1.6, Q2.3, Q2.6
- net PYRO_1: now also Q1.6, R33.1; no longer Q1.1
- net PYRO_2: now also Q2.6, R31.1; no longer Q2.1
- net PYRO_3: now also Q1.3, R29.1; no longer Q1.4
- net PYRO_4: now also Q2.3, R27.1; no longer Q2.4
- new net SENS_1: R32.1, R33.2
- new net SENS_2: R30.1, R31.2
- new net SENS_3: R28.1, R29.2
- new net SENS_4: R26.1, R27.2
Other:
- moved on the sheet: J5, Q1, Q2, R8, R9, U4, U6

Commit message: Finished. Need BOM and Review.
Parts:
- removed J1: Conn_01x06, Connector_PinHeader_2.54mm:PinHeader_1x06_P2.54mm_Vertical, symbol Connector_Generic:Conn_01x06
- removed U1: LBAA0XV2GT-001, External Libraries:Murata-Type-2GT, symbol LBAA0XV2GT-001:LBAA0XV2GT-001
- added D1: D_Schottky, Diode_SMD:D_0603_1608Metric, symbol Device:D_Schottky
- added D8: 5V, LED_SMD:LED_0805_2012Metric, symbol Device:LED
- added J5: PRGM, Connector_PinHeader_2.54mm:PinHeader_1x05_P2.54mm_Vertical, symbol Connector_Generic:Conn_01x05
- added R26: 422k, Resistor_SMD:R_0603_1608Metric, symbol Device:R
- added R27: 102k, Resistor_SMD:R_0603_1608Metric, symbol Device:R
- added R38: 2k, Resistor_SMD:R_0603_1608Metric, symbol Device:R
- added U1: LBAA0XV2GT-001, External Libraries:Murata-Type-2GT, symbol Murata-Type-2GT:LBAA0XV2GT-001
- C10: renamed from C13; footprint Capacitor_SMD:C_0603_1608Metric -> Capacitor_SMD:C_0805_2012Metric
- C11: renamed from C15; footprint Capacitor_SMD:C_0603_1608Metric -> Capacitor_SMD:C_0805_2012Metric
- C8: renamed from C12; footprint Capacitor_SMD:C_0603_1608Metric -> Capacitor_SMD:C_0805_2012Metric
- D2: renamed from D4; footprint (none) -> Diode_SMD:D_0603_1608Metric
- D3: renamed from D5; footprint (none) -> Diode_SMD:D_0603_1608Metric
- D4: renamed from D6; footprint (none) -> Diode_SMD:D_0805_2012Metric
- J1: renamed from J5; value Conn_01x08 -> PYRO; footprint (none) -> TerminalBlock_Phoenix:TerminalBlock_Phoenix_MPT-0,5-8-2.54_1x08_P2.54mm_Horizontal
- J2: renamed from J4; footprint Connector_Coaxial:SMA_Amphenol_132289_EdgeMount -> Connector_Coaxial:SMA_Molex_73251-1153_EdgeMount_Horizontal
- L2: footprint (none) -> Inductor_SMD:L_1008_2520Metric
- Q1, Q2: footprint DFN2020-6L_MCE -> footprints:DFN2020-6L_MCE
- R24: renamed from R38; value 300 -> 1k
- U2: renamed from U6; footprint (none) -> Package_TO_SOT_SMD:SOT-563
- renumbered C6 to C1, C10 to C12, C11 to C13, C8 to C14, C9 to C15, C7 to C2, C1 to C3, C2 to C4, C3 to C5, C4 to C6, C5 to C7, C14 to C9, D2 to D5, D3 to D6, D1 to D7, J6 to J3, J7 to J4, J2 to J6, J3 to J7, R8 to R1, R27 to R10, R22 to R11, R23 to R12, R24 to R13, R25 to R14, R10 to R15, R4 to R16, R13 to R17, R17 to R18, R5 to R19, R9 to R2, R16 to R20, R20 to R21, R6 to R22, R7 to R23, R39 to R25, R1 to R28, R2 to R29, R32 to R3, R11 to R30, R12 to R31, R14 to R32, R15 to R33, R18 to R34, R19 to R35, R21 to R36, R3 to R37, R33 to R4, R30 to R5, R31 to R6, R28 to R7, R29 to R8, R26 to R9, U4 to U3, U5 to U4, U3 to U5, U7 to U6, U8 to U7, U9 to U8, U2 to U9
Connections:
- net +3V3: now also D1.1 (K), J5.1 (Pin_1), U1.28 (VDD_1), U1.29 (VDD_2); no longer C8.2, C9.2, R15.2, U7.1 (OUT), U7.2 (OUT__1)
- net ANT: now also U1.19 (ANT_LORA_SUB_G_)
- net ARM: now also R24.2, U5.J2 (PA2); no longer R24.1, R25.2
- net BT_RX: now also U5.F10 (PC6)
- net BT_TX: now also U5.E10 (PC7)
- net BZ+: now also U5.K10 (PD12); no longer U5.D9 (PA8)
- net CONN_RX: now also U5.J8 (PB13); no longer U5.A5 (PB7)
- net CONN_TX: now also U5.K8 (PB12); no longer U5.B5 (PB6)
- net DCC: now also U1.6 (DCC_SW)
- net FIRE_1: now also U5.K4 (PB1)
- net FIRE_2: now also U5.K3 (PA7)
- net FIRE_3: now also U5.K6 (PE13)
- net FIRE_4: now also U5.K5 (PE9)
- net GATE_2: now also Q1.5; no longer Q2.2
- net GATE_3: now also Q2.2; no longer Q1.5
- net GPS_R: now also U5.F2 (PC1); no longer U5.K8 (PB12)
- net MEM_CLK: now also U5.C8 (PC12)
- net MEM_CMD: now also U5.B7 (PD2)
- net MEM_DAT0: now also U5.F9 (PC8)
- net MEM_DAT1: now also U5.E9 (PC9)
- net MEM_DAT2: now also U5.B9 (PC10)
- net MEM_DAT3: now also U5.B8 (PC11)
- net MISO: now also U1.11 (LR_MISO)
- net MOSI: now also U1.12 (LR_MOSI)
- net NCS: now also U1.10 (LR_NSS)
- net NRST: now also J5.5 (Pin_5)
- net PYRO: now also J1.1 (Pin_1), J1.3 (Pin_3), J1.5 (Pin_5), J1.7 (Pin_7); no longer J1.2 (Pin_2), J1.4 (Pin_4), J1.6 (Pin_6), J1.8 (Pin_8)
- net PYRO_1: now also J1.8 (Pin_8); no longer J1.1 (Pin_1)
- net PYRO_2: now also J1.6 (Pin_6), Q1.3; no longer J1.3 (Pin_3), Q2.6
- net PYRO_3: now also J1.4 (Pin_4), Q2.6; no longer J1.5 (Pin_5), Q1.3
- net PYRO_4: now also J1.2 (Pin_2); no longer J1.7 (Pin_7)
- net RAD_BUSY: now also U5.B3 (PE3), U1.9 (LR_BUSY); no longer U5.K3 (PA7)
- net RAD_IO9: now also U5.A3 (PE2), U1.1 (DIO9); no longer U5.J2 (PA2)
- net RAD_NRST: now also U5.A2 (PC13), U1.35 (LR_NRST); no longer U5.J3 (PA6)
- net SCK: now also U1.13 (LR_SCK)
- net SENS_1: now also U5.J4 (PB0)
- net SENS_2: now also U5.J3 (PA6)
- net SENS_3: now also U5.J5 (PE8)
- net SENS_4: now also U5.J6 (PE12)
- net SENS_R: now also U5.F1 (PC0); no longer U5.K7 (PB11)
- net SWCK: now also J5.2 (Pin_2)
- net SWD: now also J5.4 (Pin_4)
- net USB_D+: now also U5.B10 (PA12)
- net USB_D-: now also U5.C10 (PA11)
- net VBUS: now also R38.1
- net VREG: now also U1.4 (VREG)
- net V_SENSE: now also R26.1
- net at U5.E2 (PC2_C): now also R26.2, R27.1
- net at U5.K2 (PA3): now also R24.1, R25.2
- net GND renamed EPAD
- net EPAD: now also U3.15 (EPAD), D8.1 (K), J5.3 (Pin_3), R27.2, U1.14 (GND_5), U1.16 (GND_6), U1.18 (GND_7), U1.20 (GND_8), U1.22 (GND_9), U1.26 (GND_10), U1.27 (GND_11), U1.3 (GND_1), U1.30 (GND_12), U1.31 (GND_13), U1.32 (GND_14), U1.33 (GND_15), U1.34 (GND_16), U1.36 (GND_17), U1.37 (GND_18), U1.38 (GND_19), U1.39 (GND_20), U1.40 (GND_21), U1.41 (GND_22), U1.42 (GND_23), U1.43 (GND_24), U1.44 (GND_25), U1.45 (GND_26), U1.46 (GND_27), U1.47 (GND_28), U1.48 (GND_29), U1.5 (GND_2), U1.7 (GND_3), U1.8 (GND_4)
- new net: C8.2, C9.2, D1.2 (A), R15.2, U7.1 (OUT), U7.2 (OUT__1)
- new net: D8.2 (A), R38.2
- no-connect marks 102 -> 80
Other:
- note added: "ADC3 IN0"
- note added: "Connectors"
- note added: "Extras"
- note added: "I2C1"
- note added: "Microcontroller"
- note added: "Pyro"
- note added: "Read ARM"
- note added: "SDMMC1"
- note added: "TIM4 CH1"
- note added: "UART5"
- note added: "USART6"
- moved on the sheet: BZ1, C1, C10, C11, C12, C13, C14, C15, C16, C2, C3, C4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

Commit message: Revised after sourcing BOM
Parts:
- C21: footprint Capacitor_SMD:C_0603_1608Metric -> Capacitor_SMD:C_0805_2012Metric
- D4: footprint Diode_SMD:D_0805_2012Metric -> Diode_SMD:D_SMA
- R16, R19: footprint Resistor_SMD:R_0603_1608Metric -> Resistor_SMD:R_0402_1005Metric
- R22, R23, R37, R38: value 2k -> 1k

Commit message: after Louie Review
Parts:
- removed H1, H2: MountingHole, MountingHole:MountingHole_3.2mm_M3, symbol Mechanical:MountingHole
- added H1, H2: MountingHole_Pad, MountingHole:MountingHole_3.2mm_M3_Pad, symbol Mechanical:MountingHole_Pad
- J4: value >3.5V -> >3.6V
Connections:
- net EPAD: now also H1.1, H2.1

Commit message: Update Screw Switch PCB and schematic files
- Increased pad dimensions in Screw Switch PCB from 3.8mm to 9.0mm for improved soldering and stability.
- Added a new mounting hole symbol in the Screw Switch schematic with properties for reference, value, footprint, datasheet, and description.
- Created an auto-saved file entry for the STM32 flight computer project to ensure recovery of recent changes.
Parts:
- removed C24: 100n, Capacitor_SMD:C_0603_1608Metric, symbol Device:C
- removed U13: DPS310XTSA1, External Libraries:XDCR_DPS310XTSA1, symbol DPS310XTSA1:DPS310XTSA1
- added D9: BT, LED_SMD:LED_0805_2012Metric, symbol Device:LED
- added R39: 100R, Resistor_SMD:R_0603_1608Metric, symbol Device:R
- added U15: MS5611-01BA, Package_LGA:LGA-8_3x5mm_P1.25mm, symbol Sensor_Pressure:MS5611-01BA
- BZ1: footprint Buzzer_Beeper:Buzzer_TDK_PS1240P02BT_D12.2mm_H6.5mm -> Buzzer_Beeper:Buzzer_Murata_PKMCS0909E
- J2: footprint Connector_Coaxial:SMA_Molex_73251-1153_EdgeMount_Horizontal -> Connector_Coaxial:SMA_Samtec_SMA-J-P-H-ST-EM1_EdgeMount
- R30, R31, R32, R33, R34, R35: value DNP -> 10k
- R36: value DNP -> 1k
Connections:
- net +3V3: now also U15.1 (VDD), U15.2 (PS), U15.4 (CSB), U15.5 (CSB)
- net BZ+: now also R39.2; no longer U5.K10 (PD12)
- net EPAD: now also U8.H5 (DS), D9.1 (K), U15.3 (GND); no longer R36.2
- net GPS_R: now also U5.E3 (PE6); no longer U5.F2 (PC1)
- net SCL: now also U15.8 (SCLK)
- net SDA: now also U15.7 (SDI/SDA)
- net SENS_R: now also U5.D3 (PE5); no longer U5.F1 (PC0)
- net V_SENSE: now also D3.2 (A), D4.2 (A), J3.1 (Pin_1); no longer C10.2, D2.1 (K), D3.1 (K), U6.5 (EN), U6.6 (VIN)
- net BT_R: now reaches R36.1
- net BT_R: now also U5.G2 (PA0); no longer U8.H5 (DS)
- new net: D9.2 (A), R36.2
- new net: C10.2, D2.1 (K), D3.1 (K), U6.5 (EN), U6.6 (VIN)
- new net R_BZ: R39.1, U5.K10 (PD12)
- no-connect marks 80 -> 77
Other:
- note added: "0x76"
- note added: "Acc: 0x18 Gyr: 0x68"
- note added: "TIM15 CH1"
- note added: "TIM15 CH2"
- note added: "TIM2 CH1"
- note removed: "0x77"
- note removed: "DNP = 10k if needed"
- note removed: "I2C: Acc: 0x18 Gyr: 0x68"
- moved on the sheet: BZ1, C25, D2, D3, D5, D6, D7, D8, H1, H2, R22, R23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

Commit message: Refactor code structure for improved readability and maintainability
Parts:
- removed J1: PYRO, TerminalBlock_Phoenix:TerminalBlock_Phoenix_MPT-0,5-8-2.54_1x08_P2.54mm_Horizontal, symbol Connector_Generic:Conn_01x08
- removed Q2: MCM3400A-TP, footprints:DFN2020-6L_MCE, symbol 2025-10-09_15-16-18:MCM3400A-TP
- removed R10, R8: 100k, Resistor_SMD:R_0603_1608Metric, symbol Device:R
- removed R13, R14: 10k, Resistor_SMD:R_0603_1608Metric, symbol Device:R
- removed R7, R9: 24k9, Resistor_SMD:R_0603_1608Metric, symbol Device:R
- added J1: PYRO, TerminalBlock_Phoenix:TerminalBlock_Phoenix_MPT-0,5-4-2.54_1x04_P2.54mm_Horizontal, symbol Connector_Generic:Conn_01x04
Connections:
- net ARM: no longer U3.12 (4A), U3.9 (3A)
- net EPAD: now also J7.SH (SHIELD); no longer J7.S1 (SHIELD), U2.4 (CTS), U2.6 (CTR)
- net PYRO: now also J1.1 (Pin_1), J1.3 (Pin_3)
- net PYRO_1: now also J1.4 (Pin_4)
- net PYRO_2: now also J1.2 (Pin_2)
- net FIRE_3: no longer names the net of U5.K6 (PE13)
- net FIRE_3: no longer U3.10 (3B)
- net FIRE_4: no longer names the net of U5.K5 (PE9)
- net FIRE_4: no longer U3.13 (4B)
- net GATE_3: no longer names the net of U3.8 (3Y)
- net GATE_4: no longer names the net of U3.11 (4Y)
- net SENS_3: no longer names the net of U5.J5 (PE8)
- net SENS_4: no longer names the net of U5.J6 (PE12)
- no-connect marks 77 -> 91
Other:
- moved on the sheet: Q1, R1, R11, R12, R2, R26, R27, R3, R4, R5, R6, U2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
Changed lines of the file:
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@@
 (kicad_sch
-	(version 20250114)
+	(version 20260306)
 	(generator "eeschema")
-	(generator_version "9.0")
+	(generator_version "10.0")
 	(paper "A3")
