File: Spaceport/PCBs/dipole-breakout/dipole-breakout.kicad_pcb (KiCad board)
At the start: 2 copper layers, 15.8 x 9 mm, 7 parts, among them J1 Conn_Coaxial, J2 Conn_01x01_Pin, J3 Conn_01x01_Pin

Commit message: small changes and add dipole board gerbers
Changed lines of the file:
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@@
 			(plot_on_all_layers_selection 0x0000000_00000000)
 			(disableapertmacros no)
-			(usegerberextensions no)
+			(usegerberextensions yes)
 			(usegerberattributes yes)
 			(usegerberadvancedattributes yes)
@@
 			(outputformat 1)
 			(mirror no)
-			(drillshape 1)
+			(drillshape 0)
 			(scaleselection 1)
-			(outputdirectory "")
+			(outputdirectory "../Gerbers/dipole-breakout/")
 		)
 	)
@@
 		(pad "1" smd rect
 			(at 0 0 90)
-			(size 1.27 4.064)
+			(size 1.5 4.064)
 			(layers "F.Cu" "F.Mask")
 			(net 2 "GND")
@@
 			(zone_connect 2)
 			(thermal_bridge_angle 0)
+			(teardrops
+				(best_length_ratio 0.5)
+				(max_length 1)
+				(best_width_ratio 1)
+				(max_width 2)
+				(curve_points 0)
+				(filter_ratio 0.9)
+				(enabled yes)
+				(allow_two_segments yes)
+				(prefer_zone_connections yes)
+			)
 		)
 	)
@@
 		(pad "1" smd rect
 			(at 0 0 90)
-			(size 1.27 4.064)
+			(size 1.5 4.064)
 			(layers "F.Cu" "F.Mask")
 			(net 1 "Net-(J1-In)")
@@
 			(zone_connect 2)
 			(thermal_bridge_angle 0)
+			(teardrops
+				(best_length_ratio 0.5)
+				(max_length 1)
+				(best_width_ratio 1)
+				(max_width 2)
+				(curve_points 0)
+				(filter_ratio 0.9)
+				(enabled yes)
+				(allow_two_segments yes)
+				(prefer_zone_connections yes)
+			)
 		)
 	)
@@
 		(net 2)
 	)
+	(zone
+		(net 1)
+		(net_name "Net-(J1-In)")
+		(layer "F.Cu")
+		(name "$teardrop_padvia$")
+		(hatch full 0.1)
+		(priority 30000)
+		(attr
+			(teardrop
+				(type padvia)
+			)
+		)
+		(connect_pads yes
+			(clearance 0)
+		)
+		(min_thickness 0.0254)
+		(filled_areas_thickness no)
+		(fill yes
+			(thermal_gap 0.5)
+			(thermal_bridge_width 0.5)
+			(island_removal_mode 1)
+			(island_area_min 10)
+		)
+		(polygon
+			(pts
+				(xy 171.618 81.45) (xy 171.618 82.55) (xy 172.368 82.75) (xy 174.401 82) (xy 172.368 81.25)
+			)
+		)
+	)
+	(zone
+		(net 2)
+		(net_name "GND")
+		(layer "F.Cu")
+		(name "$teardrop_padvia$")
+		(hatch full 0.1)
+		(priority 30000)
+		(attr
+			(teardrop
+				(type padvia)
+			)
+		)
+		(connect_pads yes
+			(clearance 0)
+		)
+		(min_thickness 0.0254)
+		(filled_areas_thickness no)
+		(fill yes
+			(thermal_gap 0.5)
+			(thermal_bridge_width 0.5)
+			(island_removal_mode 1)
+			(island_area_min 10)
+		)
+		(polygon
+			(pts
+				(xy 168.882 82.55) (xy 168.882 81.45) (xy 168.132 81.25) (xy 166.099 82) (xy 168.132 82.75)
+			)
+		)
+	)
 )
