File: Spaceport/PCBs/Sensor Boards/SensorBoardAirbrake/SensorBoardNoMCU.kicad_sch (KiCad schematic)
At the start: 14 parts, among them J2 I2C, U1 BMI088, U5 MMC5633NJL, U6 MS5611-01BA

Commit message: updates
Parts:
- removed C5: 100n, Capacitor_SMD:C_0603_1608Metric, symbol Device:C
- removed U5: MMC5633NJL, Package_BGA:WLP-4_0.86x0.86mm_P0.4mm, symbol Sensor_Magnetic:MMC5633NJL
- added C3, C4: 100n, Capacitor_SMD:C_0603_1608Metric, symbol Device:C
- added U2: MLX90393ELW-ABA-014-RE, Package_DFN_QFN:QFN-16-1EP_3x3mm_P0.5mm_EP1.75x1.75mm, symbol easyeda2kicad:MLX90393ELW-ABA-014-RE
- renumbered C2 to C1, C3 to C2, C6 to C5
Connections:
- net +3.3V: now also C3.1, C4.1, U2.12 (A0), U2.15 (VDD), U2.2 (SENB/CS), U2.8 (VDD_IO)
- net GND: now also C3.2, C4.2, U2.10 (N/C), U2.11 (A1), U2.13 (VSS), U2.14 (N/C), U2.16 (N/C), U2.17 (EP), U2.4 (N/C), U2.9 (N/C)
- net SCL1: now also U2.3 (SCL/SCLK)
- net SDA1: now also U2.5 (SDA/MOSI)
- no-connect marks 6 -> 9
Other:
- note added: "I2C: 0x19"
- note removed: "I2C: 0x30"
- moved on the sheet: C5, U6
