File: Spaceport/PCBs/flight-computer/flight-computer-2026-2027/gps.kicad_sch (KiCad schematic)
At the start: 1 part

Commit message: gps + hihg g accel done
Parts:
- added C10, C11, C8, C9: 100nF, symbol Device:C_Small
Connections:
- net GND: now reaches ANT1.1 (GND_1)
- net GND: now also ANT1.10 (GND_5), ANT1.11 (GND_6), ANT1.15 (GND_7), ANT1.16 (GND_8), ANT1.20 (GND_9), ANT1.4 (GND_2), ANT1.5 (GND_3), ANT1.6 (GND_4), C10.2, C11.2, C8.2, C9.2
- net i2c_scl: now reaches ANT1.12 (SCL)
- net +3.3VA: now reaches ANT1.17 (VCC)
- net +3.3VA: now also ANT1.2 (V_IO), ANT1.3 (V_BCKP), C10.1, C11.1, C8.1, C9.1
- net i2c_sda: now reaches ANT1.9 (SDA)
- no-connect marks 0 -> 6
Other:
- note added: "Followed the exact same breakout as last years and the Sam M10Q breakout board in the archive repository"

Commit message: removed imu, need imu stuff
also, decided to use ldo + shared everythgin 3.3VA rail. SD card looks good, found gps i2c address and implemented i2c bus based on bus capciatance.
Other:
- note added: "To poll or set the I2C address, use the CFG-I2C-ADDRESS configuration item (see the u-blox M10 interface description [3]). The CFG-I2C-ADDRESS configuration item is an 8-bit value containing the I2C address in the 7 most significant bits plus a 0 as the least significant bit. Thus, the default address becomes 0x84(1000 0100)"
Changed lines of the file:
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@@
 	(generator_version "10.0")
 	(paper "A4")
+	(text "To poll or set the I2C address, use the CFG-I2C-ADDRESS configuration item (see the u-blox M10\ninterface description [3]). The CFG-I2C-ADDRESS configuration item is an 8-bit value containing\nthe I2C address in the 7 most significant bits plus a 0 as the least significant bit. Thus, the default\naddress becomes 0x84(1000 0100)"
+		(exclude_from_sim no)
+		(at 160.782 133.604 0)
+		(effects
+			(font
+				(size 1.27 1.27)
+			)
+			(justify left)
+		)
+	)
 	(text "Followed the exact same breakout as last years\nand the Sam M10Q breakout board in the archive \nrepository\n"
 		(exclude_from_sim no)
