File: Spaceport/PCBs/flight-computer/flight-computer-2026-2027/9-dof-imu.kicad_sch (KiCad schematic)
At the start: 1 part, among them U1 ICM-20948

Commit message: imu
need to find imu that is spi + 9 DoF + in stock
Parts:
- removed U1: ICM-20948, Sensor_Motion:InvenSense_QFN-24_3x3mm_P0.4mm, symbol Sensor_Motion:ICM-20948
- added C19, C21, C22: 100nF, symbol Device:C_Small
- added C20: 10uF, symbol Device:C_Small
- added C24: 10nF, symbol Device:C_Small
- added IC3: LSM9DS1, LSM9DS1, symbol Symbols:LSM9DS1
Connections:
- new net: C24.1, IC3.21 (CAP)
- new net: C22.1, IC3.24 (C1)
- new net +3.3VA: C19.1, C20.1, C21.1, IC3.1 (VDDIO_1), IC3.22 (VDD_1), IC3.23 (VDD_2), IC3.3 (VDDIO_2)
- new net GND: C19.2, C20.2, C21.2, C22.2, C24.2, IC3.14 (RES_1), IC3.15 (RES_2), IC3.16 (RES_3), IC3.17 (RES_4), IC3.18 (RES_5), IC3.19 (GND_1), IC3.20 (GND_2)
- new net int_1: IC3.11 (INT1_A/G)
- new net int_2: IC3.12 (INT2_A/G)
- new net int_m: IC3.10 (INT_M)
- new net spi_mosi: IC3.4 (SDA/SDI/SDO)
- new net spi_sck: IC3.2 (SCL/SPC)
Other:
- note added: "Chose this imu becuase supports spi + logic voltage level can be covered by 3.3V DO NOT USE, IS NOT IN STOCK"

Commit message: remove imu
Parts:
- removed C19, C21, C22: 100nF, symbol Device:C_Small
- removed C20: 10uF, symbol Device:C_Small
- removed C24: 10nF, symbol Device:C_Small
- removed IC3: LSM9DS1, LSM9DS1, symbol Symbols:LSM9DS1

Commit message: 6-dof imu implemented, updated datacheets
changelog:
- changed 9-dof-imu sheet to 6-dof-imu and added BMI088 imu to it
- added imu sheet symbol to fc schem and connected it to spi
- marked unused interrupt pins as nc
- made pins 34-37 gpio output to use as spi cs pins (pins 34 & 35 are used for the 6 dof imu's accelerometer and gyro, respectively

- connected SD card to spi bus, uses gpio pin 36
- updated datasheets folder to reflect components in fc schem
Parts:
- added U1: BMI088, Package_LGA:Bosch_LGA-16_4.5x3mm_P0.5mm_LayoutBorder7x1y_ClockwisePinNumbering, symbol Sensor_Motion:BMI088
Connections:
- new net: U1.2 (GNDA), U1.4 (GNDA)
Other:
- note removed: "Chose this imu becuase supports spi + logic voltage level can be covered by 3.3V DO NOT USE, IS NOT IN STOCK"
Changed lines of the file:
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@@
 	(generator_version "10.0")
 	(paper "A4")
-	(text "Chose this imu becuase supports spi + logic voltage level can be covered by 3.3V\n\nDO NOT USE, IS NOT IN STOCK"
+	(symbol
+		(lib_id "Sensor_Motion:BMI088")
+		(at 140.97 95.25 0)
+		(unit 1)
+		(body_style 1)
 		(exclude_from_sim no)
-		(at 167.6088 32.24 0)
-		(effects
-			(font
-				(size 1.27 1.27)
+		(in_bom yes)
+		(on_board yes)
+		(in_pos_files yes)
+		(dnp no)
+		(fields_autoplaced yes)
+		(property "Reference" "U1"
+			(at 145.6533 77.47 0)
+			(show_name no)
+			(do_not_autoplace no)
+			(effects
+				(font
+					(size 1.27 1.27)
+				)
+				(justify left)
 			)
-			(justify left)
+		)
+		(property "Value" "BMI088"
+			(at 145.6533 80.01 0)
+			(show_name no)
+			(do_not_autoplace no)
+			(effects
+				(font
+					(size 1.27 1.27)
+				)
+				(justify left)
+			)
+		)
+		(property "Footprint" "Package_LGA:Bosch_LGA-16_4.5x3mm_P0.5mm_LayoutBorder7x1y_ClockwisePinNumbering"
+			(at 124.46 96.52 0)
+			(hide yes)
+			(show_name no)
+			(do_not_autoplace no)
+			(effects
+				(font
+					(size 1.27 1.27)
+				)
+			)
+		)
+		(property "Datasheet" "https://www.bosch-sensortec.com/media/boschsensortec/downloads/datasheets/bst-bmi088-ds001.pdf"
+			(at 124.46 96.52 0)
+			(hide yes)
+			(show_name no)
+			(do_not_autoplace no)
+			(effects
+				(font
+					(size 1.27 1.27)
+				)
+			)
+		)
+		(property "Description" "Accelerometer, Gyroscope, 6-Axis Sensor, I2C / SPI interface, LGA-16"
+			(at 140.97 95.25 0)
+			(hide yes)
+			(show_name no)
+			(do_not_autoplace no)
+			(effects
+				(font
+					(size 1.27 1.27)
+				)
+			)
+		)
+		(pin "7"
+		)
+		(pin "5"
+		)
+		(pin "14"
+		)
+		(pin "3"
+		)
+		(pin "13"
+		)
+		(pin "8"
+		)
+		(pin "12"
+		)
+		(pin "16"
+		)
+		(pin "15"
+		)
+		(pin "9"
+		)
+		(pin "2"
+		)
+		(pin "6"
+		)
+		(pin "10"
+		)
+		(pin "1"
+		)
+		(pin "11"
+		)
+		(pin "4"
+		)
+		(instances
+			(project "flight_computer_26_27"
+				(path "/4fd124df-e0d9-445f-9973-04852ab50770/a14f8403-15fe-4bfa-a826-a892b2271dab"
+					(reference "U1")
+					(unit 1)
+				)
+			)
 		)
 	)
